Commit message: added gazebo plugins for the sensors

File: robotino_description/urdf/camera.urdf.xacro (robot description, xacro)
@@ -1,5 +1,5 @@
 <?xml version="1.0"?>
 <root xmlns:xacro="http://www.ros.org/wiki/xacro">
-  <xacro:macro name="camera" params="parent name *origin">
+  <xacro:macro name="webcam" params="parent name *origin">
     <joint name="${name}_joint" type="fixed">
       <insert_block name="origin" />

File: robotino_description/urdf/hokuyo.urdf.xacro (robot description, xacro)
@@ -28,4 +28,42 @@
       </collision>
     </link>
+    <!-- gazebo extensions -->
+    <xacro:hokuyo_gazebo name="${name}" ros_topic="scan" update_rate="10" min_angle="-2.3562" max_angle="2.3562"/>
+  </xacro:macro>
+  <!--GAZEBO PLUGIN-->
+  <xacro:macro name="hokuyo_gazebo" params="name ros_topic update_rate min_angle max_angle">
+    <gazebo reference="${name}_link">
+      <sensor name="${name}" type="ray">
+        <always_on>true</always_on>
+        <update_rate>${update_rate}</update_rate>
+        <pose>0 0 0 0 0 0</pose>
+        <visualize>false</visualize>
+        <ray>
+          <scan>
+            <horizontal>
+              <samples>640</samples>
+              <resolution>1.0</resolution>
+              <min_angle>${min_angle}</min_angle>
+              <max_angle>${max_angle}</max_angle>
+            </horizontal>
+          </scan>
+          <range>
+            <min>0.05</min>
+            <max>10.0</max>
+            <resolution>0.01</resolution>
+          </range>
+          <noise>
+            <type>gaussian</type>
+            <mean>0.0</mean>
+            <stddev>0.005</stddev>
+          </noise>
+        </ray>
+        <plugin name="gazebo_ros_${name}_controller" filename="libgazebo_ros_laser.so">
+          <topicName>${ros_topic}</topicName>
+          <frameName>${name}_link</frameName>
+        </plugin>
+      </sensor>
+      <material>Gazebo/White</material>
+    </gazebo>
   </xacro:macro>
 </root>

File: robotino_description/urdf/kinect.urdf.xacro (robot description, xacro)
@@ -29,4 +29,61 @@
       </collision>
     </link>
+    <joint name="${name}_frame_joint" type="fixed">
+      <origin xyz="0 0 0" rpy="${M_PI/2} -${M_PI/2} 0" />
+      <parent link="${name}_link"/>
+      <child link="${name}_frame"/>
+    </joint>
+    <link name="${name}_frame"/>
+    <!-- gazebo extensions -->
+    <xacro:kinect_gazebo name="kinect" ros_topic="kinect" />
+  </xacro:macro>
+  <!-- GAZEBO OPENNI PLUGIN -->
+  <xacro:macro name="kinect_gazebo" params="name ros_topic">
+    <gazebo reference="${name}_frame">
+      <sensor type="depth" name="${name}_frame_sensor">
+        <always_on>true</always_on>
+        <update_rate>20.0</update_rate>
+        <camera>
+          <horizontal_fov>${62.0*M_PI/180.0}</horizontal_fov>
+          <image>
+            <format>R8G8B8</format>
+            <width>640</width>
+            <height>480</height>
+          </image>
+          <clip>
+            <near>0.1</near>
+            <far>100</far>
+          </clip>
+          <noise>
+            <type>gaussian</type>
+            <mean>0.0</mean>
+            <stddev>0.0</stddev>
+          </noise>
+        </camera>
+        <plugin name="${name}_controller" filename="libgazebo_ros_openni_kinect.so">
+          <updateRate>20.0</updateRate>
+          <cameraName>${ros_topic}</cameraName>
+          <frameName>${name}_link</frameName>
+          <imageTopicName>rgb/image_raw</imageTopicName>
+          <depthImageTopicName>depth/image_raw</depthImageTopicName>
+          <pointCloudTopicName>depth_registered/points</pointCloudTopicName>
+          <cameraInfoTopicName>rgb/camera_info</cameraInfoTopicName>
+          <depthImageCameraInfoTopicName>depth_registered/camera_info</depthImageCameraInfoTopicName>
+          <pointCloudCutoff>0.5</pointCloudCutoff>
+          <baseline>0.2</baseline>
+          <hackBaseline>0.0</hackBaseline>
+          <distortionK1>0.0</distortionK1>
+          <distortionK2>0.0</distortionK2>
+          <distortionK3>0.0</distortionK3>
+          <distortionT1>0.0</distortionT1>
+          <distortionT2>0.0</distortionT2>
+          <CxPrime>0.0</CxPrime>
+          <Cx>0.0</Cx>
+          <Cy>0.0</Cy>
+          <focalLength>0.0</focalLength>
+        </plugin>
+      </sensor>
+      <material>Gazebo/White</material>
+    </gazebo>
   </xacro:macro>
 </root>

File: robotino_description/urdf/properties.urdf.xacro (robot description, xacro)
@@ -11,7 +11,7 @@
   <property name="HOKUYO_RADIUS" value="0.02"/>
   <property name="HOKUYO_LENGTH" value="0.07"/>
-  <property name="KINECT_LENGTH" value="0.064"/>
-  <property name="KINECT_WIDTH" value="0.121"/>
-  <property name="KINECT_HEIGHT" value="0.0381"/>
+  <property name="KINECT_LENGTH" value="0.05"/>
+  <property name="KINECT_WIDTH" value="0.035"/>
+  <property name="KINECT_HEIGHT" value="0.18"/>
   <!-- camera mount positions | handeye calibration | relative to base_link -->
   <property name="camera_x" value="0.0"/>
@@ -32,7 +32,7 @@
   <property name="kinect_y" value="0.0"/>
   <property name="kinect_z" value="0.6"/>
-  <property name="kinect_roll" value="0.0"/>
+  <property name="kinect_roll" value="-${M_PI/2}"/>
   <property name="kinect_pitch" value="0.0"/>
-  <property name="kinect_yaw" value="0.0"/>
+  <property name="kinect_yaw" value="0"/>
   <!-- anglebracketusb mount positions | handeye calibration | relative to base_link -->
   <property name="anglebracketusb_x" value="0.008"/>

File: robotino_description/urdf/robotino.urdf.xacro (robot description, xacro)
@@ -9,7 +9,7 @@
   <xacro:include filename="$(find robotino_description)/urdf/kinect.urdf.xacro" />
   <xacro:body name="base"/>
-  <camera name="camera" parent="base_link">
+  <webcam name="camera" parent="base_link">
     <origin xyz="${camera_x} ${camera_y} ${camera_z}" rpy="${camera_roll} ${camera_pitch} ${camera_yaw}"/>
-  </camera>
+  </webcam>
   <hokuyo name="hokuyo" parent="base_link">
     <origin xyz="${hokuyo_x} ${hokuyo_y} ${hokuyo_z}" rpy="${hokuyo_roll} ${hokuyo_pitch} ${hokuyo_yaw}"/>
