Commit message: New description structure

File: robotino_description/urdf/robotino.urdf.xacro (robot description, xacro)
@@ -1,7 +1,23 @@
 <?xml version="1.0"?>
-<robot name="robotino">
-  <!-- Include files -->
-  <include filename="$(find robotino_description)/urdf/robotino_body.xacro"/>
-  <include filename="$(find robotino_description)/urdf/robotino_hardware.xacro"/>
-  <robotino_body />
+<robot xmlns:xacro="http://www.ros.org/wiki/xacro"
+  name="robotino">
+  <xacro:include filename="$(find robotino_description)/urdf/properties.urdf.xacro" />
+  <xacro:include filename="$(find robotino_description)/urdf/robotino_body.urdf.xacro" />
+  <xacro:include filename="$(find robotino_description)/urdf/hokuyo.urdf.xacro" />
+  <xacro:include filename="$(find robotino_description)/urdf/camera.urdf.xacro" />
+  <xacro:include filename="$(find robotino_description)/urdf/angle_bracket.urdf.xacro" />
+  <xacro:include filename="$(find robotino_description)/urdf/kinect.urdf.xacro" />
+  <xacro:body name="base"/>
+  <camera name="camera" parent="base_link">
+    <origin xyz="${camera_x} ${camera_y} ${camera_z}" rpy="${camera_roll} ${camera_pitch} ${camera_yaw}"/>
+  </camera>
+  <hokuyo name="hokuyo" parent="base_link">
+    <origin xyz="${hokuyo_x} ${hokuyo_y} ${hokuyo_z}" rpy="${hokuyo_roll} ${hokuyo_pitch} ${hokuyo_yaw}"/>
+  </hokuyo>
+  <kinect name="kinect" parent="base_link">
+    <origin xyz="${kinect_x} ${kinect_y} ${kinect_z}" rpy="${kinect_roll} ${kinect_pitch} ${kinect_yaw}"/>
+  </kinect>
+  <!--anglebracketusb name="anglebracketusb" parent="base_link">
+    <origin xyz="${anglebracketusb_x} ${anglebracketusb_y} ${anglebracketusb_z}" rpy="${anglebracketusb_roll} ${anglebracketusb_pitch} ${anglebracketusb_yaw}"/>
+  </anglebracketusb-->
 </robot>

File: robotino_description/urdf/robotino_body.urdf.xacro (robot description, xacro)
@@ -1,11 +1,42 @@
 <?xml version="1.0"?>
 <root xmlns:xacro="http://www.ros.org/wiki/xacro">
-  <property name="M_PI" value="3.14159"/>
-  <property name="M_SCALE" value="0.01"/>
-  <property name="HOKUYO_RADIUS" value="0.02"/>
-  <property name="HOKUYO_LENGTH" value="0.07"/>
-  <property name="KINECT_LENGTH" value="0.064"/>
-  <property name="KINECT_WIDTH" value="0.121"/>
-  <property name="KINECT_HEIGHT" value="0.0381"/>
+  <xacro:macro name="body" params="name">
+   <link name="${name}_link">
+      <inertial>
+        <mass value="${BASE_MASS}" />
+        <origin xyz="0 0 0" />
+        <inertia ixx="1.0" ixy="0.0" ixz="0.0"
+          iyy="1.0" iyz="0.0"
+          izz="1.0" />
+      </inertial>
+      <visual>
+        <origin xyz="0.01 0 0" rpy="0 0 ${M_PI/2}"/>
+        <geometry>
+          <mesh filename="package://robotino_description/meshes/RobotinoBody.dae" scale="${M_SCALE} ${M_SCALE} ${M_SCALE}"/>
+        </geometry>
+      </visual>
+      <collision>
+        <origin xyz="0 0 ${BASE_HEIGHT/2}" rpy="0 0 0" />
+        <geometry>
+          <cylinder radius="${BASE_RADIUS}" length="${BASE_HEIGHT}"/>
+        </geometry>
+      </collision>
+    </link>
+    <wheel name="wheel0" parent="base_link">
+      <origin xyz="0.065 0.11 0.04" rpy="0 0 ${M_PI/3}"/>
+      <axis xyz="-1 0 0"/>
+    </wheel>
+    <wheel name="wheel1" parent="base_link">
+      <origin xyz="-0.13 0 0.04" rpy="0 0 0"/>
+      <axis xyz="1 0 0"/>
+    </wheel>
+    <wheel name="wheel2" parent="base_link">
+      <origin xyz="0.065 -0.11 0.04" rpy="0 0 -${M_PI/3}"/>
+      <axis xyz="-1 0 0"/>
+    </wheel>
+    <command_bridge name="command_bridge" parent="base_link">
+      <origin xyz="-0.05 0 0.13" rpy="0 0 ${M_PI/2}"/>
+    </command_bridge>
+  </xacro:macro>
   <!-- WHEEL -->
   <xacro:macro name="wheel" params="parent name *origin *axis">
@@ -55,28 +86,4 @@
     </link>
   </xacro:macro>
-  <!-- Camera -->
-  <xacro:macro name="camera" params="parent name *origin">
-    <joint name="${name}_joint" type="fixed">
-      <insert_block name="origin" />
-      <parent link="${parent}"/>
-      <child link="${name}_link" />
-    </joint>
-    <link name="${name}_link">
-      <inertial>
-        <mass value="0.00001" />
-        <origin xyz="0 0 0" />
-        <inertia ixx="1.0" ixy="0.0" ixz="0.0"
-          iyy="1.0" iyz="0.0"
-          izz="1.0" />
-      </inertial>
-      <visual>
-        <origin xyz="0 0 0" rpy="0 0 0" />
-        <geometry>
-          <mesh filename="package://robotino_description/meshes/RobotinoCamera.dae" scale="${M_SCALE} ${M_SCALE} ${M_SCALE}"/>
-        </geometry>
-      </visual>
-    </link>
-  </xacro:macro>
-  <!-- AngleBracket With USB Hub -->
   <xacro:macro name="anglebracketusb" params="parent name *origin">
     <joint name="${name}_joint" type="fixed">

Commit message: complete frames' tree

File: robotino_description/urdf/robotino.urdf.xacro (robot description, xacro)
@@ -17,11 +17,14 @@
     </plugin>
   </gazebo>
-  <!--webcam name="camera" parent="base_link">
+  <webcam name="camera" parent="base_link">
     <origin xyz="${camera_x} ${camera_y} ${camera_z}" rpy="${camera_roll} ${camera_pitch} ${camera_yaw}"/>
-  </webcam-->
+  </webcam>
   <hokuyo name="hokuyo" parent="base_link">
     <origin xyz="${hokuyo_x} ${hokuyo_y} ${hokuyo_z}" rpy="${hokuyo_roll} ${hokuyo_pitch} ${hokuyo_yaw}"/>
   </hokuyo>
-  <kinect name="kinect" parent="tilt_link">
+  <!-- <tilt_axis name="tilt" parent="base_link"> -->
+  <!--   <origin xyz="${tilt_x} ${tilt_y} ${tilt_z}" rpy="${tilt_roll} ${tilt_pitch} ${tilt_yaw}"/> -->
+  <!-- </tilt_axis> -->
+  <kinect name="kinect" parent="base_link">
     <origin xyz="${kinect_x} ${kinect_y} ${kinect_z}" rpy="${kinect_roll} ${kinect_pitch} ${kinect_yaw}"/>
   </kinect>
@@ -32,7 +35,4 @@
     </plugin>
   </gazebo>
-  <tilt_axis name="tilt" parent="base_link">
-    <origin xyz="${tilt_x} ${tilt_y} ${tilt_z}" rpy="${tilt_roll} ${tilt_pitch} ${tilt_yaw}"/>
-  </tilt_axis>
   <!--anglebracketusb name="anglebracketusb" parent="base_link">
     <origin xyz="${anglebracketusb_x} ${anglebracketusb_y} ${anglebracketusb_z}" rpy="${anglebracketusb_roll} ${anglebracketusb_pitch} ${anglebracketusb_yaw}"/>

Commit message: added gazebo controllers

File: robotino_description/urdf/robotino.urdf.xacro (robot description, xacro)
@@ -37,11 +37,11 @@
       <commandTopic>cmd_vel</commandTopic>
       <odometryTopic>odom</odometryTopic>
-      <odometryFrame>odom</odometryFrame>
+      <odometryFrame>odom</odometryFrame> -->
       <odometryRate>20.0</odometryRate>
-      <robotBaseFrame>base_footprint</robotBaseFrame>
+      <robotBaseFrame>base_footprint</robotBaseFrame> -->
     </plugin>
   </gazebo>
   <!--anglebracketusb name="anglebracketusb" parent="base_link">
-    <origin xyz="${anglebracketusb_x} ${anglebracketusb_y} ${anglebracketusb_z}" rpy="${anglebracketusb_roll} ${anglebracketusb_pitch} ${anglebracketusb_yaw}"/>
+      <origin xyz="${anglebracketusb_x} ${anglebracketusb_y} ${anglebracketusb_z}" rpy="${anglebracketusb_roll} ${anglebracketusb_pitch} ${anglebracketusb_yaw}"/>
   </anglebracketusb-->
 </robot>
