Commit message: fixed laser frame

File: robotino_description/urdf/hokuyo.urdf.xacro (robot description, xacro)
@@ -16,5 +16,5 @@
       </inertial>
       <visual>
-        <origin xyz="0 0 0" rpy="0 0 ${M_PI/2}" />
+        <origin xyz="0 0 -0.05" rpy="0 0 ${M_PI/2}" />
         <geometry>
           <mesh filename="package://robotino_description/meshes/RobotinoLaserScanner.dae" scale="${M_SCALE} ${M_SCALE} ${M_SCALE}"/>

File: robotino_description/urdf/properties.urdf.xacro (robot description, xacro)
@@ -24,5 +24,5 @@
   <property name="hokuyo_x" value="0.024"/>
   <property name="hokuyo_y" value="0.0"/>
-  <property name="hokuyo_z" value="0.11"/>
+  <property name="hokuyo_z" value="0.16"/>
   <property name="hokuyo_roll" value="0.0"/>
   <property name="hokuyo_pitch" value="0.0"/>
