Commit message: tabs vs spaces

File: robotino_description/urdf/properties.urdf.xacro (robot description, xacro)
@@ -1,7 +1,7 @@
 <?xml version="1.0" ?>
 <robot xmlns:xacro="http://www.ros.org/wiki/xacro">
-	<!-- ****************** -->
-	<!-- ***** COMMON ***** -->
-	<!-- ****************** -->
+  <!-- ****************** -->
+  <!-- ***** COMMON ***** -->
+  <!-- ****************** -->
   <property name="M_PI" value="3.14159"/>
   <property name="M_SCALE" value="0.01"/>
@@ -14,31 +14,31 @@
   <property name="KINECT_WIDTH" value="0.121"/>
   <property name="KINECT_HEIGHT" value="0.0381"/>
-	<!-- camera mount positions | handeye calibration | relative to base_link -->
-	<property name="camera_x" value="0.044"/>
-	<property name="camera_y" value="0.0"/>
-	<property name="camera_z" value="0.2"/>
-	<property name="camera_roll" value="0.0"/>
-	<property name="camera_pitch" value="0.0"/>
-	<property name="camera_yaw" value="${M_PI/2}"/>
-	<!-- hokuyo mount positions | relative to base_link -->
-	<property name="hokuyo_x" value="0.024"/>
-	<property name="hokuyo_y" value="0.0"/>
-	<property name="hokuyo_z" value="0.11"/>
-	<property name="hokuyo_roll" value="0.0"/>
-	<property name="hokuyo_pitch" value="0.0"/>
-	<property name="hokuyo_yaw" value="0.0"/>
-	<!-- kinect mount positions | handeye calibration | relative to base_link -->
-	<property name="kinect_x" value="-0.022"/>
-	<property name="kinect_y" value="0.0"/>
-	<property name="kinect_z" value="0.6"/>
-	<property name="kinect_roll" value="0.0"/>
-	<property name="kinect_pitch" value="0.0"/>
-	<property name="kinect_yaw" value="0.0"/>
-	<!-- anglebracketusb mount positions | handeye calibration | relative to base_link -->
-	<property name="anglebracketusb_x" value="0.008"/>
-	<property name="anglebracketusb_y" value="0.0"/>
-	<property name="anglebracketusb_z" value="0.137"/>
-	<property name="anglebracketusb_roll" value="0.0"/>
-	<property name="anglebracketusb_pitch" value="0.0"/>
-	<property name="anglebracketusb_yaw" value="0.0"/>
+  <!-- camera mount positions | handeye calibration | relative to base_link -->
+  <property name="camera_x" value="0.044"/>
+  <property name="camera_y" value="0.0"/>
+  <property name="camera_z" value="0.2"/>
+  <property name="camera_roll" value="0.0"/>
+  <property name="camera_pitch" value="0.0"/>
+  <property name="camera_yaw" value="${M_PI/2}"/>
+  <!-- hokuyo mount positions | relative to base_link -->
+  <property name="hokuyo_x" value="0.024"/>
+  <property name="hokuyo_y" value="0.0"/>
+  <property name="hokuyo_z" value="0.11"/>
+  <property name="hokuyo_roll" value="0.0"/>
+  <property name="hokuyo_pitch" value="0.0"/>
+  <property name="hokuyo_yaw" value="0.0"/>
+  <!-- kinect mount positions | handeye calibration | relative to base_link -->
+  <property name="kinect_x" value="-0.022"/>
+  <property name="kinect_y" value="0.0"/>
+  <property name="kinect_z" value="0.6"/>
+  <property name="kinect_roll" value="0.0"/>
+  <property name="kinect_pitch" value="0.0"/>
+  <property name="kinect_yaw" value="0.0"/>
+  <!-- anglebracketusb mount positions | handeye calibration | relative to base_link -->
+  <property name="anglebracketusb_x" value="0.008"/>
+  <property name="anglebracketusb_y" value="0.0"/>
+  <property name="anglebracketusb_z" value="0.137"/>
+  <property name="anglebracketusb_roll" value="0.0"/>
+  <property name="anglebracketusb_pitch" value="0.0"/>
+  <property name="anglebracketusb_yaw" value="0.0"/>
 </robot>

File: robotino_description/urdf/robotino_body.urdf.xacro (robot description, xacro)
@@ -86,25 +86,3 @@
     </link>
   </xacro:macro>
-  <xacro:macro name="anglebracketusb" params="parent name *origin">
-    <joint name="${name}_joint" type="fixed">
-      <insert_block name="origin" />
-      <parent link="${parent}"/>
-      <child link="${name}_link" />
-    </joint>
-    <link name="${name}_link">
-      <inertial>
-        <mass value="0.00001" />
-        <origin xyz="0 0 0" />
-        <inertia ixx="1.0" ixy="0.0" ixz="0.0"
-          iyy="1.0" iyz="0.0"
-          izz="1.0" />
-      </inertial>
-      <visual>
-        <origin xyz="0 0 0" rpy="0 0 0" />
-        <geometry>
-          <mesh filename="package://robotino_description/meshes/AngleBracketUSBHub.dae" scale="${M_SCALE} ${M_SCALE} ${M_SCALE}"/>
-        </geometry>
-      </visual>
-    </link>
-  </xacro:macro>
 </root>

Commit message: merge robotino current version

File: robotino_description/urdf/properties.urdf.xacro (robot description, xacro)
@@ -24,15 +24,22 @@
   <property name="hokuyo_x" value="0.024"/>
   <property name="hokuyo_y" value="0.0"/>
-  <property name="hokuyo_z" value="0.11"/>
+  <property name="hokuyo_z" value="0.135"/>
   <property name="hokuyo_roll" value="0.0"/>
   <property name="hokuyo_pitch" value="0.0"/>
   <property name="hokuyo_yaw" value="0.0"/>
-  <!-- kinect mount positions | handeye calibration | relative to base_link -->
-  <property name="kinect_x" value="-0.01"/>
+   <!-- tilt mount positions | handeye calibration | relative to base_link -->
+  <property name="tilt_x" value="-0.01"/>
+  <property name="tilt_y" value="0.0"/>
+  <property name="tilt_z" value="0.47"/>
+  <property name="tilt_roll" value="0"/>
+  <property name="tilt_pitch" value="${M_PI/2}"/>
+  <property name="tilt_yaw" value="0"/>
+  <!-- kinect mount positions | handeye calibration | relative to tilt_link -->
+  <property name="kinect_x" value="-0.03"/>
   <property name="kinect_y" value="0.0"/>
-  <property name="kinect_z" value="0.3"/>
-  <property name="kinect_roll" value="0"/>
-  <property name="kinect_pitch" value="${M_PI/2}"/>
-  <property name="kinect_yaw" value="0"/>
+  <property name="kinect_z" value="0.0"/>
+  <property name="kinect_roll" value="0.0"/>
+  <property name="kinect_pitch" value="0.0"/>
+  <property name="kinect_yaw" value="0.0"/>
   <!-- anglebracketusb mount positions | handeye calibration | relative to base_link -->
   <property name="anglebracketusb_x" value="0.008"/>

File: robotino_description/urdf/robotino.urdf.xacro (robot description, xacro)
@@ -9,16 +9,20 @@
   <xacro:include filename="$(find robotino_description)/urdf/angle_bracket.urdf.xacro" />
   <xacro:include filename="$(find robotino_description)/urdf/kinect.urdf.xacro" />
+  <xacro:include filename="$(find robotino_description)/urdf/tilt_axis.urdf.xacro" />
   <xacro:body name="base"/>
-  <!--webcam name="camera" parent="base_link">
-    <origin xyz="${camera_x} ${camera_y} ${camera_z}" rpy="${camera_roll} ${camera_pitch} ${camera_yaw}"/>
-  </webcam-->
   <hokuyo name="hokuyo" parent="base_link">
     <origin xyz="${hokuyo_x} ${hokuyo_y} ${hokuyo_z}" rpy="${hokuyo_roll} ${hokuyo_pitch} ${hokuyo_yaw}"/>
   </hokuyo>
-  <kinect name="kinect" parent="base_link">
+  <!--kinect name="kinect" parent="base_link">
     <origin xyz="${kinect_x} ${kinect_y} ${kinect_z}" rpy="${kinect_roll} ${kinect_pitch} ${kinect_yaw}"/>
-  </kinect>
+  </kinect-->
   <!--anglebracketusb name="anglebracketusb" parent="base_link">
     <origin xyz="${anglebracketusb_x} ${anglebracketusb_y} ${anglebracketusb_z}" rpy="${anglebracketusb_roll} ${anglebracketusb_pitch} ${anglebracketusb_yaw}"/>
   </anglebracketusb-->
+  <tilt_axis name="tilt" parent="base_link">
+    <origin xyz="${tilt_x} ${tilt_y} ${tilt_z}" rpy="${tilt_roll} ${tilt_pitch} ${tilt_yaw}"/>
+  </tilt_axis>
+  <kinect name="kinect" parent="tilt_link">
+    <origin xyz="${kinect_x} ${kinect_y} ${kinect_z}" rpy="${kinect_roll} ${kinect_pitch} ${kinect_yaw}"/>
+  </kinect>
 </robot>
