Commit message: removed unnecesary files

File: robotino_description/urdf/kinect.urdf.xacro (robot description, xacro)
@@ -2,8 +2,12 @@
 <root xmlns:xacro="http://www.ros.org/wiki/xacro">
   <xacro:macro name="kinect" params="parent name *origin">
-    <joint name="${name}_joint" type="fixed">
+    <joint name="${name}_joint" type="revolute">
       <insert_block name="origin" />
       <parent link="${parent}"/>
       <child link="${name}_link" />
+      <axis xyz="0 1 0" />
+      <dynamics damping="0.1" />
+      <calibration rising="0"/>
+      <limit effort="100" lower="-1.57" upper="1.57" velocity="1.4"/>
     </joint>
     <link name="${name}_link">

File: robotino_description/urdf/properties.urdf.xacro (robot description, xacro)
@@ -29,7 +29,7 @@
   <property name="hokuyo_yaw" value="0.0"/>
   <!-- kinect mount positions | handeye calibration | relative to base_link -->
-  <property name="kinect_x" value="-0.022"/>
+  <property name="kinect_x" value="-0.01"/>
   <property name="kinect_y" value="0.0"/>
-  <property name="kinect_z" value="0.6"/>
+  <property name="kinect_z" value="0.3"/>
   <property name="kinect_roll" value="0"/>
   <property name="kinect_pitch" value="${M_PI/2}"/>

File: robotino_description/urdf/robotino.urdf.xacro (robot description, xacro)
@@ -9,7 +9,7 @@
   <xacro:include filename="$(find robotino_description)/urdf/kinect.urdf.xacro" />
   <xacro:body name="base"/>
-  <webcam name="camera" parent="base_link">
+  <!--webcam name="camera" parent="base_link">
     <origin xyz="${camera_x} ${camera_y} ${camera_z}" rpy="${camera_roll} ${camera_pitch} ${camera_yaw}"/>
-  </webcam>
+  </webcam-->
   <hokuyo name="hokuyo" parent="base_link">
     <origin xyz="${hokuyo_x} ${hokuyo_y} ${hokuyo_z}" rpy="${hokuyo_roll} ${hokuyo_pitch} ${hokuyo_yaw}"/>

Commit message: configuration for rviz

File: robotino_description/urdf/kinect.urdf.xacro (robot description, xacro)
@@ -2,12 +2,13 @@
 <root xmlns:xacro="http://www.ros.org/wiki/xacro">
   <xacro:macro name="kinect" params="parent name *origin">
-    <joint name="${name}_joint" type="revolute">
+      <!--joint name="${name}_joint" type="revolute"-->
+      <joint name="${name}_joint" type="fixed">
       <insert_block name="origin" />
       <parent link="${parent}"/>
       <child link="${name}_link" />
       <axis xyz="0 1 0" />
-      <dynamics damping="0.1" />
+      <!--dynamics damping="0.1" />
       <calibration rising="0"/>
-      <limit effort="100" lower="-1.57" upper="1.57" velocity="1.4"/>
+      <limit effort="100" lower="-1.57" upper="1.57" velocity="1.4"/-->
     </joint>
     <link name="${name}_link">
@@ -41,4 +42,5 @@
     <!-- gazebo extensions -->
     <xacro:kinect_gazebo name="kinect" ros_topic="kinect" />
+    <xacro:kinect_transmission name="kinect" />
   </xacro:macro>
   <!-- GAZEBO OPENNI PLUGIN -->
@@ -88,6 +90,17 @@
         </plugin>
       </sensor>
-      <material>Gazebo/White</material>
+      <material>Gazebo/Black</material>
     </gazebo>
   </xacro:macro>
+  <!--xacro:macro name="kinect_transmission" params="name">
+    <transmission name="${name}_trans">
+      <type>transmission_interface/SimpleTransmission</type>
+      <joint name="${name}_joint">
+        <hardwareInterface>EffortJointInterface</hardwareInterface>
+      </joint>
+      <actuator name="${name}_motor">
+        <mechanicalReduction>1</mechanicalReduction>
+      </actuator>
+    </transmission>
+  </xacro:macro-->
 </root>

File: robotino_description/urdf/robotino.urdf.xacro (robot description, xacro)
@@ -3,4 +3,5 @@
   name="robotino">
   <xacro:include filename="$(find robotino_description)/urdf/properties.urdf.xacro" />
+  <xacro:include filename="$(find robotino_description)/urdf/gazebo.urdf.xacro" />
   <xacro:include filename="$(find robotino_description)/urdf/robotino_body.urdf.xacro" />
   <xacro:include filename="$(find robotino_description)/urdf/hokuyo.urdf.xacro" />

Commit message: renamed point_cloud topic, adapted namesapces and new collision modle for wheels

File: robotino_description/urdf/kinect.urdf.xacro (robot description, xacro)
@@ -67,5 +67,6 @@
           <imageTopicName>rgb/image_raw</imageTopicName>
           <depthImageTopicName>depth/image_raw</depthImageTopicName>
-          <pointCloudTopicName>depth_registered/points</pointCloudTopicName>
+          <!--pointCloudTopicName>depth_registered/points</pointCloudTopicName-->
+          <pointCloudTopicName>depth/points</pointCloudTopicName>
           <cameraInfoTopicName>rgb/camera_info</cameraInfoTopicName>
           <depthImageCameraInfoTopicName>depth_registered/camera_info</depthImageCameraInfoTopicName>

File: robotino_description/urdf/robotino_body.urdf.xacro (robot description, xacro)
@@ -75,7 +75,8 @@
       </visual>
       <collision>
-        <origin xyz="0 0 0" rpy="0 0 0" />
+        <origin xyz="0 0 0" rpy="0 ${M_PI/2} 0" />
         <geometry>
-          <mesh filename="package://robotino_description/meshes/RobotinoWheel.dae" scale="${M_SCALE} ${M_SCALE} ${M_SCALE}"/>
+          <!--mesh filename="package://robotino_description/meshes/RobotinoWheel.dae" scale="${M_SCALE} ${M_SCALE} ${M_SCALE}"/-->
+          <cylinder length="0.04" radius="0.04"/>
         </geometry>
       </collision>

Commit message: current robot version

File: robotino_description/urdf/kinect.urdf.xacro (robot description, xacro)
@@ -29,10 +29,10 @@
       </collision>
     </link>
-    <joint name="${name}_frame_joint" type="fixed">
-      <origin xyz="0 0 0" rpy="${M_PI/2} -${M_PI/2} 0" />
-      <parent link="${name}_link"/>
-      <child link="${name}_frame"/>
-    </joint>
-    <link name="${name}_frame"/>
+    <!-- <joint name="${name}_frame_joint" type="fixed"> -->
+    <!--   <origin xyz="0 0 0" rpy="${M_PI/2} -${M_PI/2} 0" />  -->
+    <!--   <parent link="${name}_link"/> -->
+    <!--   <child link="${name}_frame"/> -->
+    <!-- </joint> -->
+    <!-- <link name="${name}_frame"/> -->
     <!-- gazebo extensions -->
     <xacro:kinect_gazebo name="kinect" ros_topic="kinect" />

File: robotino_description/urdf/properties.urdf.xacro (robot description, xacro)
@@ -20,5 +20,5 @@
   <property name="camera_roll" value="0.0"/>
   <property name="camera_pitch" value="0.0"/>
-  <property name="camera_yaw" value="${M_PI/2}"/>
+  <property name="camera_yaw" value="-${M_PI/2}"/>
   <!-- hokuyo mount positions | relative to base_link -->
   <property name="hokuyo_x" value="0.024"/>
@@ -31,6 +31,6 @@
   <property name="tilt_x" value="-0.01"/>
   <property name="tilt_y" value="0.0"/>
-  <property name="tilt_z" value="0.47"/>
-  <property name="tilt_roll" value="0"/>
+  <property name="tilt_z" value="0.45"/>
+  <property name="tilt_roll" value="-0.05"/>
   <property name="tilt_pitch" value="${M_PI/2}"/>
   <property name="tilt_yaw" value="0"/>
@@ -39,6 +39,6 @@
   <property name="kinect_y" value="0.0"/>
   <property name="kinect_z" value="0.0"/>
-  <property name="kinect_roll" value="0.0"/>
-  <property name="kinect_pitch" value="0.0"/>
+  <property name="kinect_roll" value="-0.02"/>
+  <property name="kinect_pitch" value="-1.45"/>
   <property name="kinect_yaw" value="0.0"/>
   <!-- anglebracketusb mount positions | handeye calibration | relative to base_link -->

File: robotino_description/urdf/robotino.urdf.xacro (robot description, xacro)
@@ -32,10 +32,10 @@
     <origin xyz="${kinect_x} ${kinect_y} ${kinect_z}" rpy="${kinect_roll} ${kinect_pitch} ${kinect_yaw}"/>
   </kinect>
-  <gazebo>
+  <!--gazebo>
     <plugin name="ros_control" filename="libmulti_hw_interface_gazebo_ros_control.so">
       <robotNamespace>tilt_controller</robotNamespace>
       <filterJointsParam>joint_names</filterJointsParam>
     </plugin>
-  </gazebo>
+  </gazebo-->
   <!--anglebracketusb name="anglebracketusb" parent="base_link">
       <origin xyz="${anglebracketusb_x} ${anglebracketusb_y} ${anglebracketusb_z}" rpy="${anglebracketusb_roll} ${anglebracketusb_pitch} ${anglebracketusb_yaw}"/>

File: robotino_description/urdf/robotino_body.urdf.xacro (robot description, xacro)
@@ -2,10 +2,10 @@
 <root xmlns:xacro="http://www.ros.org/wiki/xacro">
   <xacro:macro name="body" params="name">
-    <link name="${name}_footprint"/>
-	<joint name="${name}_footprint_joint" type="fixed">
-		<origin xyz="0 0 0" rpy="0 0 0" />
-		<child link="${name}_link" />
-		<parent link="${name}_footprint"/>
-	</joint>
+    <!-- <link name="${name}_footprint"/> -->
+	  <!-- <joint name="${name}_footprint_joint" type="fixed"> -->
+		<!--   <origin xyz="0 0 0" rpy="0 0 0" /> -->
+		<!--   <child link="${name}_link" /> -->
+		<!--   <parent link="${name}_footprint"/> -->
+	  <!-- </joint> -->
    <link name="${name}_link">
       <inertial>
