Commit message: implemented controllers

File: robotino_description/urdf/gazebo.urdf.xacro (robot description, xacro)
@@ -3,7 +3,45 @@
   <gazebo>
     <plugin name="gazebo_ros_control" filename="libgazebo_ros_control.so">
-      <robotNamespace>/tilt_controller</robotNamespace>
-      <!--robotSimType>gazebo_ros_control/DefaultRobotHWSim</robotSimType-->
+      <robotNamespace>/robotino</robotNamespace>
     </plugin>
   </gazebo>
+  <xacro:macro name="wheel_gazebo" params="name">
+    <gazebo reference="${name}_link">
+      <mu1 value="100.0" />
+      <mu2 value="100.0" />
+      <kp  value="1000000.0" />
+      <kd  value="1.0" />
+    </gazebo>
+  </xacro:macro>
+  <xacro:macro name="base_gazebo" params="name">
+    <gazebo reference="${name}_link">
+      <gravity>true</gravity>
+      <self_collide>false</self_collide>
+      <sensor name='${name}_contact_sensor' type='contact'>
+        <always_on>true</always_on>
+        <update_rate>100.0</update_rate>
+        <contact>
+          <collision>${name}_link_collision</collision>
+          <topic>${name}_bumper</topic>
+        </contact>
+        <plugin name="${name}_gazebo_ros_bumper_controller" filename="libgazebo_ros_bumper.so">
+          <frameName>world</frameName>
+          <bumperTopicName>${name}_bumper</bumperTopicName>
+        </plugin>
+      </sensor>
+    </gazebo>
+   <gazebo>
+      <plugin name="p3d_base_controller" filename="libgazebo_ros_p3d.so">
+        <alwaysOn>true</alwaysOn>
+        <updateRate>100.0</updateRate>
+        <bodyName>${name}_link</bodyName>
+        <topicName>${name}_pose_ground_truth</topicName>
+        <frameName>map</frameName>
+        <xyzOffsets>25.7 25.7 0</xyzOffsets> <!-- initialize odometry for fake localization-->
+        <rpyOffsets>0 0 0</rpyOffsets>
+        <gaussianNoise>0.01</gaussianNoise>
+      </plugin>
+      <canonicalBody>${name}_footprint</canonicalBody>
+    </gazebo>
+  </xacro:macro>
 </robot>

File: robotino_description/urdf/kinect.urdf.xacro (robot description, xacro)
@@ -2,13 +2,8 @@
 <root xmlns:xacro="http://www.ros.org/wiki/xacro">
   <xacro:macro name="kinect" params="parent name *origin">
-      <!--joint name="${name}_joint" type="revolute"-->
-      <joint name="${name}_joint" type="fixed">
+    <joint name="${name}_joint" type="fixed">
       <insert_block name="origin" />
       <parent link="${parent}"/>
       <child link="${name}_link" />
-      <axis xyz="0 1 0" />
-      <!--dynamics damping="0.1" />
-      <calibration rising="0"/>
-      <limit effort="100" lower="-1.57" upper="1.57" velocity="1.4"/-->
     </joint>
     <link name="${name}_link">
@@ -42,5 +37,4 @@
     <!-- gazebo extensions -->
     <xacro:kinect_gazebo name="kinect" ros_topic="kinect" />
-    <xacro:kinect_transmission name="kinect" />
   </xacro:macro>
   <!-- GAZEBO OPENNI PLUGIN -->
@@ -93,14 +87,3 @@
     </gazebo>
   </xacro:macro>
-  <!--xacro:macro name="kinect_transmission" params="name">
-    <transmission name="${name}_trans">
-      <type>transmission_interface/SimpleTransmission</type>
-      <joint name="${name}_joint">
-        <hardwareInterface>EffortJointInterface</hardwareInterface>
-      </joint>
-      <actuator name="${name}_motor">
-        <mechanicalReduction>1</mechanicalReduction>
-      </actuator>
-    </transmission>
-  </xacro:macro-->
 </root>

File: robotino_description/urdf/properties.urdf.xacro (robot description, xacro)
@@ -28,11 +28,18 @@
   <property name="hokuyo_pitch" value="0.0"/>
   <property name="hokuyo_yaw" value="0.0"/>
-  <!-- kinect mount positions | handeye calibration | relative to base_link -->
-  <property name="kinect_x" value="-0.01"/>
+  <!-- tilt mount positions | handeye calibration | relative to base_link -->
+  <property name="tilt_x" value="-0.01"/>
+  <property name="tilt_y" value="0.0"/>
+  <property name="tilt_z" value="0.3"/>
+  <property name="tilt_roll" value="0"/>
+  <property name="tilt_pitch" value="${M_PI/2}"/>
+  <property name="tilt_yaw" value="0"/>
+  <!-- kinect mount positions | handeye calibration | relative to tilt_link -->
+  <property name="kinect_x" value="0.0"/>
   <property name="kinect_y" value="0.0"/>
-  <property name="kinect_z" value="0.3"/>
-  <property name="kinect_roll" value="0"/>
-  <property name="kinect_pitch" value="${M_PI/2}"/>
-  <property name="kinect_yaw" value="0"/>
+  <property name="kinect_z" value="0.0"/>
+  <property name="kinect_roll" value="0.0"/>
+  <property name="kinect_pitch" value="0.0"/>
+  <property name="kinect_yaw" value="0.0"/>
   <!-- anglebracketusb mount positions | handeye calibration | relative to base_link -->
   <property name="anglebracketusb_x" value="0.008"/>

File: robotino_description/urdf/robotino.urdf.xacro (robot description, xacro)
@@ -9,4 +9,5 @@
   <xacro:include filename="$(find robotino_description)/urdf/angle_bracket.urdf.xacro" />
   <xacro:include filename="$(find robotino_description)/urdf/kinect.urdf.xacro" />
+  <xacro:include filename="$(find robotino_description)/urdf/tilt_axis.urdf.xacro" />
   <xacro:body name="base"/>
   <!--webcam name="camera" parent="base_link">
@@ -16,7 +17,10 @@
     <origin xyz="${hokuyo_x} ${hokuyo_y} ${hokuyo_z}" rpy="${hokuyo_roll} ${hokuyo_pitch} ${hokuyo_yaw}"/>
   </hokuyo>
-  <kinect name="kinect" parent="base_link">
+  <kinect name="kinect" parent="tilt_link">
     <origin xyz="${kinect_x} ${kinect_y} ${kinect_z}" rpy="${kinect_roll} ${kinect_pitch} ${kinect_yaw}"/>
   </kinect>
+  <tilt_axis name="tilt" parent="base_link">
+    <origin xyz="${tilt_x} ${tilt_y} ${tilt_z}" rpy="${tilt_roll} ${tilt_pitch} ${tilt_yaw}"/>
+  </tilt_axis>
   <!--anglebracketusb name="anglebracketusb" parent="base_link">
     <origin xyz="${anglebracketusb_x} ${anglebracketusb_y} ${anglebracketusb_z}" rpy="${anglebracketusb_roll} ${anglebracketusb_pitch} ${anglebracketusb_yaw}"/>

File: robotino_description/urdf/robotino_body.urdf.xacro (robot description, xacro)
@@ -2,4 +2,10 @@
 <root xmlns:xacro="http://www.ros.org/wiki/xacro">
   <xacro:macro name="body" params="name">
+    <link name="${name}_footprint"/>
+    <joint name="${name}_footprint_joint" type="fixed">
+      <origin xyz="0 0 0" rpy="0 0 0" />
+      <child link="${name}_link" />
+      <parent link="${name}_footprint"/>
+    </joint>
    <link name="${name}_link">
       <inertial>
@@ -17,22 +23,29 @@
       </visual>
       <collision>
-        <origin xyz="0 0 ${BASE_HEIGHT/2}" rpy="0 0 0" />
+        <origin xyz="0.01 0 0" rpy="0 0 ${M_PI/2}"/>
         <geometry>
-          <cylinder radius="${BASE_RADIUS}" length="${BASE_HEIGHT}"/>
+          <mesh filename="package://robotino_description/meshes/RobotinoBody.dae" scale="${M_SCALE} ${M_SCALE} ${M_SCALE}"/>
         </geometry>
       </collision>
     </link>
+    <base_gazebo name="base" />
     <wheel name="wheel0" parent="base_link">
       <origin xyz="0.065 0.11 0.04" rpy="0 0 ${M_PI/3}"/>
       <axis xyz="-1 0 0"/>
     </wheel>
+    <wheel_transmission name="wheel0" />
+    <wheel_gazebo name="wheel0" />
     <wheel name="wheel1" parent="base_link">
       <origin xyz="-0.13 0 0.04" rpy="0 0 0"/>
       <axis xyz="1 0 0"/>
     </wheel>
+    <wheel_transmission name="wheel1" />
+    <wheel_gazebo name="wheel1" />
     <wheel name="wheel2" parent="base_link">
       <origin xyz="0.065 -0.11 0.04" rpy="0 0 -${M_PI/3}"/>
       <axis xyz="-1 0 0"/>
     </wheel>
+    <wheel_transmission name="wheel2" />
+    <wheel_gazebo name="wheel2" />
     <command_bridge name="command_bridge" parent="base_link">
       <origin xyz="-0.05 0 0.13" rpy="0 0 ${M_PI/2}"/>
@@ -49,5 +62,5 @@
     <link name="${name}_link">
       <inertial>
-        <mass value="0.00001" />
+        <mass value="2" />
         <origin xyz="0 0 0" />
         <inertia ixx="1.0" ixy="0.0" ixz="0.0"
@@ -61,5 +74,23 @@
         </geometry>
       </visual>
+      <collision>
+        <origin xyz="0 0 0" rpy="0 0 0" />
+        <geometry>
+          <mesh filename="package://robotino_description/meshes/RobotinoWheel.dae" scale="${M_SCALE} ${M_SCALE} ${M_SCALE}"/>
+        </geometry>
+      </collision>
     </link>
+  </xacro:macro>
+  <!-- Wheel transmission   -->
+  <xacro:macro name="wheel_transmission" params="name">
+    <transmission name="${name}_trans">
+      <type>transmission_interface/SimpleTransmission</type>
+      <joint name="${name}_joint" >
+        <hardwareInterface>VelocityJointInterface</hardwareInterface>
+      </joint>
+      <actuator name="${name}_motor">
+        <mechanicalReduction>${624/35 * 80/18}</mechanicalReduction>
+      </actuator>
+    </transmission>
   </xacro:macro>
   <!-- COMMAND BRIDGE -->

Commit message: the robot can now move smoothly in simulation, wheels are turning visually

File: robotino_description/urdf/gazebo.urdf.xacro (robot description, xacro)
@@ -8,8 +8,10 @@
   <xacro:macro name="wheel_gazebo" params="name">
     <gazebo reference="${name}_link">
-      <mu1 value="100.0" />
-      <mu2 value="100.0" />
+      <mu1 value="0.0" /> <!-- 100 -->
+      <mu2 value="0.0" /> <!-- 100 , http://ode-wiki.org/wiki/index.php?title=FAQ-->
       <kp  value="1000000.0" />
       <kd  value="1.0" />
+      <!--fdir1>0 1 0</fdir1>
+      <maxContacts>1</maxContacts-->
     </gazebo>
   </xacro:macro>
@@ -31,5 +33,5 @@
       </sensor>
     </gazebo>
-   <gazebo>
+   <!--gazebo>
       <plugin name="p3d_base_controller" filename="libgazebo_ros_p3d.so">
         <alwaysOn>true</alwaysOn>
@@ -38,10 +40,20 @@
         <topicName>${name}_pose_ground_truth</topicName>
         <frameName>map</frameName>
-        <xyzOffsets>25.7 25.7 0</xyzOffsets> <!-- initialize odometry for fake localization-->
-        <rpyOffsets>0 0 0</rpyOffsets>
+        <xyzOffsets>25.7 25.7 0</xyzOffsets--> <!-- initialize odometry for fake localization-->
+        <!--rpyOffsets>0 0 0</rpyOffsets>
         <gaussianNoise>0.01</gaussianNoise>
       </plugin>
       <canonicalBody>${name}_footprint</canonicalBody>
-    </gazebo>
+    </gazebo-->
+	<!-- position controller -->
+	<gazebo>
+		<plugin name="base_controller" filename="libgazebo_ros_planar_move.so">
+			<commandTopic>cmd_vel</commandTopic>
+			<odometryTopic>odom</odometryTopic>
+			<odometryFrame>odom</odometryFrame>
+			<odometryRate>100.0</odometryRate>
+			<robotBaseFrame>base_footprint</robotBaseFrame>
+		</plugin>
+	</gazebo>
   </xacro:macro>
 </robot>

File: robotino_description/urdf/robotino_body.urdf.xacro (robot description, xacro)
@@ -2,10 +2,10 @@
 <root xmlns:xacro="http://www.ros.org/wiki/xacro">
   <xacro:macro name="body" params="name">
-    <!-- <link name="${name}_footprint"/> -->
-    <!-- <joint name="${name}_footprint_joint" type="fixed"> -->
-    <!--   <origin xyz="0 0 0" rpy="0 0 0" /> -->
-    <!--   <child link="${name}_link" /> -->
-    <!--   <parent link="${name}_footprint"/> -->
-    <!-- </joint> -->
+    <link name="${name}_footprint"/>
+	<joint name="${name}_footprint_joint" type="fixed">
+		<origin xyz="0 0 0" rpy="0 0 0" />
+		<child link="${name}_link" />
+		<parent link="${name}_footprint"/>
+	</joint>
    <link name="${name}_link">
       <inertial>
@@ -55,20 +55,19 @@
   <xacro:macro name="wheel" params="parent name *origin *axis">
     <joint name="${name}_joint" type="continuous">
+      <parent link="${parent}"/>
+      <child link="${name}_link" />
       <insert_block name="origin" />
       <insert_block name="axis" />
-      <parent link="${parent}"/>
-      <child link="${name}_link" />
     </joint>
     <link name="${name}_link">
       <inertial>
-        <mass value="2" />
+        <mass value="0.4" />
         <origin xyz="0 0 0" />
-        <inertia ixx="1.0" ixy="0.0" ixz="0.0"
-          iyy="1.0" iyz="0.0"
-          izz="1.0" />
+        <inertia ixx="0.012411765597" ixy="-0.000711733678" ixz="0.00050272983" iyy="0.015218160428" iyz="-0.000004273467" izz="0.011763977943"/>
       </inertial>
       <visual>
         <origin xyz="0 0 0" rpy="0 0 0" />
         <geometry>
+		  <!--cylinder length="0.04" radius="0.04"/-->
           <mesh filename="package://robotino_description/meshes/RobotinoWheel.dae" scale="${M_SCALE} ${M_SCALE} ${M_SCALE}"/>
         </geometry>
@@ -91,4 +90,5 @@
       </joint>
       <actuator name="${name}_motor">
+        <hardwareInterface>VelocityJointInterface</hardwareInterface>
         <mechanicalReduction>${624/35 * 80/18}</mechanicalReduction>
       </actuator>

Commit message: reset kinect position , add /joint_states controller and fix hokuyo position

File: robotino_description/urdf/gazebo.urdf.xacro (robot description, xacro)
@@ -52,5 +52,5 @@
 			<odometryTopic>odom</odometryTopic>
 			<odometryFrame>odom</odometryFrame>
-			<odometryRate>100.0</odometryRate>
+			<odometryRate>20.0</odometryRate>
 			<robotBaseFrame>base_footprint</robotBaseFrame>
 		</plugin>

File: robotino_description/urdf/properties.urdf.xacro (robot description, xacro)
@@ -31,5 +31,5 @@
   <property name="tilt_x" value="-0.01"/>
   <property name="tilt_y" value="0.0"/>
-  <property name="tilt_z" value="0.3"/>
+  <property name="tilt_z" value="0.5"/>
   <property name="tilt_roll" value="0"/>
   <property name="tilt_pitch" value="${M_PI/2}"/>

File: robotino_description/urdf/robotino.urdf.xacro (robot description, xacro)
@@ -11,10 +11,10 @@
   <xacro:include filename="$(find robotino_description)/urdf/tilt_axis.urdf.xacro" />
   <xacro:body name="base"/>
-  <gazebo>
+  <!--gazebo>
     <plugin name="ros_control" filename="libmulti_hw_interface_gazebo_ros_control.so">
       <robotNamespace>base_controller</robotNamespace>
       <filterJointsParam>joint_names</filterJointsParam>
     </plugin>
-  </gazebo>
+  </gazebo-->
   <webcam name="camera" parent="base_link">
     <origin xyz="${camera_x} ${camera_y} ${camera_z}" rpy="${camera_roll} ${camera_pitch} ${camera_yaw}"/>
@@ -23,8 +23,8 @@
     <origin xyz="${hokuyo_x} ${hokuyo_y} ${hokuyo_z}" rpy="${hokuyo_roll} ${hokuyo_pitch} ${hokuyo_yaw}"/>
   </hokuyo>
-  <!-- <tilt_axis name="tilt" parent="base_link"> -->
-  <!--   <origin xyz="${tilt_x} ${tilt_y} ${tilt_z}" rpy="${tilt_roll} ${tilt_pitch} ${tilt_yaw}"/> -->
-  <!-- </tilt_axis> -->
-  <kinect name="kinect" parent="base_link">
+  <tilt_axis name="tilt" parent="base_link">
+    <origin xyz="${tilt_x} ${tilt_y} ${tilt_z}" rpy="${tilt_roll} ${tilt_pitch} ${tilt_yaw}"/>
+  </tilt_axis>
+  <kinect name="kinect" parent="tilt_link">
     <origin xyz="${kinect_x} ${kinect_y} ${kinect_z}" rpy="${kinect_roll} ${kinect_pitch} ${kinect_yaw}"/>
   </kinect>
@@ -34,11 +34,4 @@
       <filterJointsParam>joint_names</filterJointsParam>
     </plugin>
-    <plugin name="base_controller" filename="libgazebo_ros_planar_move.so">
-      <commandTopic>cmd_vel</commandTopic>
-      <odometryTopic>odom</odometryTopic>
-      <odometryFrame>odom</odometryFrame>
-      <odometryRate>20.0</odometryRate>
-      <robotBaseFrame>base_footprint</robotBaseFrame>
-    </plugin>
   </gazebo>
   <!--anglebracketusb name="anglebracketusb" parent="base_link">

Commit message: update hydro simulation

File: robotino_description/urdf/gazebo.urdf.xacro (robot description, xacro)
@@ -1,9 +1,8 @@
 <?xml version="1.0"?>
 <robot xmlns:xacro="http://www.ros.org/wiki/xacro">
-  <gazebo>
-    <plugin name="gazebo_ros_control" filename="libgazebo_ros_control.so">
-      <robotNamespace>/robotino</robotNamespace>
+  <!--gazebo>
+    <plugin name="ros_control" filename="libgazebo_ros_control.so">
     </plugin>
-  </gazebo>
+  </gazebo-->
   <xacro:macro name="wheel_gazebo" params="name">
     <gazebo reference="${name}_link">
@@ -33,27 +32,14 @@
       </sensor>
     </gazebo>
-   <!--gazebo>
-      <plugin name="p3d_base_controller" filename="libgazebo_ros_p3d.so">
-        <alwaysOn>true</alwaysOn>
-        <updateRate>100.0</updateRate>
-        <bodyName>${name}_link</bodyName>
-        <topicName>${name}_pose_ground_truth</topicName>
-        <frameName>map</frameName>
-        <xyzOffsets>25.7 25.7 0</xyzOffsets--> <!-- initialize odometry for fake localization-->
-        <!--rpyOffsets>0 0 0</rpyOffsets>
-        <gaussianNoise>0.01</gaussianNoise>
+	<!-- position controller -->
+    <gazebo>
+      <plugin name="base_controller" filename="libgazebo_ros_planar_move.so">
+          <commandTopic>cmd_vel</commandTopic>
+          <odometryTopic>odom</odometryTopic>
+          <odometryFrame>odom</odometryFrame>
+          <odometryRate>20.0</odometryRate>
+          <robotBaseFrame>base_footprint</robotBaseFrame>
       </plugin>
-      <canonicalBody>${name}_footprint</canonicalBody>
-    </gazebo-->
-	<!-- position controller -->
-	<gazebo>
-		<plugin name="base_controller" filename="libgazebo_ros_planar_move.so">
-			<commandTopic>cmd_vel</commandTopic>
-			<odometryTopic>odom</odometryTopic>
-			<odometryFrame>odom</odometryFrame>
-			<odometryRate>20.0</odometryRate>
-			<robotBaseFrame>base_footprint</robotBaseFrame>
-		</plugin>
-	</gazebo>
+    </gazebo>
   </xacro:macro>
 </robot>

File: robotino_description/urdf/robotino.urdf.xacro (robot description, xacro)
@@ -11,19 +11,7 @@
   <xacro:include filename="$(find robotino_description)/urdf/tilt_axis.urdf.xacro" />
   <xacro:body name="base"/>
-  <!--gazebo>
-    <plugin name="ros_control" filename="libmulti_hw_interface_gazebo_ros_control.so">
-      <robotNamespace>base_controller</robotNamespace>
-      <filterJointsParam>joint_names</filterJointsParam>
-    </plugin>
-  </gazebo-->
   <hokuyo name="hokuyo" parent="base_link">
     <origin xyz="${hokuyo_x} ${hokuyo_y} ${hokuyo_z}" rpy="${hokuyo_roll} ${hokuyo_pitch} ${hokuyo_yaw}"/>
   </hokuyo>
-  <!--kinect name="kinect" parent="base_link">
-    <origin xyz="${kinect_x} ${kinect_y} ${kinect_z}" rpy="${kinect_roll} ${kinect_pitch} ${kinect_yaw}"/>
-  </kinect-->
-  <!--anglebracketusb name="anglebracketusb" parent="base_link">
-    <origin xyz="${anglebracketusb_x} ${anglebracketusb_y} ${anglebracketusb_z}" rpy="${anglebracketusb_roll} ${anglebracketusb_pitch} ${anglebracketusb_yaw}"/>
-  </anglebracketusb-->
   <tilt_axis name="tilt" parent="base_link">
     <origin xyz="${tilt_x} ${tilt_y} ${tilt_z}" rpy="${tilt_roll} ${tilt_pitch} ${tilt_yaw}"/>
@@ -32,12 +20,3 @@
     <origin xyz="${kinect_x} ${kinect_y} ${kinect_z}" rpy="${kinect_roll} ${kinect_pitch} ${kinect_yaw}"/>
   </kinect>
-  <gazebo>
-    <plugin name="ros_control" filename="libmulti_hw_interface_gazebo_ros_control.so">
-      <robotNamespace>tilt_controller</robotNamespace>
-      <filterJointsParam>joint_names</filterJointsParam>
-    </plugin>
-  </gazebo>
-  <!--anglebracketusb name="anglebracketusb" parent="base_link">
-      <origin xyz="${anglebracketusb_x} ${anglebracketusb_y} ${anglebracketusb_z}" rpy="${anglebracketusb_roll} ${anglebracketusb_pitch} ${anglebracketusb_yaw}"/>
-  </anglebracketusb-->
 </robot>

File: robotino_description/urdf/tilt_axis.urdf.xacro (robot description, xacro)
@@ -25,10 +25,7 @@
     <transmission name="${name}_trans">
       <type>transmission_interface/SimpleTransmission</type>
-      <joint name="${name}_joint">
-        <!--hardwareInterface>EffortJointInterface</hardwareInterface>
-        <hardwareInterface>VelocityJointInterface</hardwareInterface-->
-        <hardwareInterface>PositionJointInterface</hardwareInterface>
-      </joint>
+      <joint name="${name}_joint"/>
       <actuator name="${name}_motor">
+        <hardwareInterface>EffortJointInterface</hardwareInterface>
         <mechanicalReduction>1</mechanicalReduction>
       </actuator>

Commit message: simulator working

File: robotino_description/urdf/gazebo.urdf.xacro (robot description, xacro)
@@ -1,9 +1,9 @@
 <?xml version="1.0"?>
 <robot xmlns:xacro="http://www.ros.org/wiki/xacro">
-  <gazebo>
+  <!--gazebo>
     <plugin name="gazebo_ros_control" filename="libgazebo_ros_control.so">
       <robotNamespace>/robotino</robotNamespace>
     </plugin>
-  </gazebo>
+  </gazebo-->
   <xacro:macro name="wheel_gazebo" params="name">
     <gazebo reference="${name}_link">

File: robotino_description/urdf/kinect.urdf.xacro (robot description, xacro)
@@ -29,10 +29,10 @@
       </collision>
     </link>
-    <joint name="${name}_frame_joint" type="fixed">
-      <origin xyz="0 0 0" rpy="${M_PI/2} -${M_PI/2} 0" />
+    <!--joint name="${name}_frame_joint" type="fixed">
+      <origin xyz="0 0 0" rpy="-${M_PI/2} 0 -${M_PI/2}" />
       <parent link="${name}_link"/>
       <child link="${name}_frame"/>
     </joint>
-    <link name="${name}_frame"/>
+    <link name="${name}_frame"/-->
     <!-- gazebo extensions -->
     <xacro:kinect_gazebo name="kinect" ros_topic="kinect" />
@@ -40,5 +40,5 @@
   <!-- GAZEBO OPENNI PLUGIN -->
   <xacro:macro name="kinect_gazebo" params="name ros_topic">
-    <gazebo reference="${name}_frame">
+    <gazebo reference="${name}_link">
       <sensor type="depth" name="${name}_frame_sensor">
         <always_on>true</always_on>
@@ -64,5 +64,5 @@
           <updateRate>20.0</updateRate>
           <cameraName>${ros_topic}</cameraName>
-          <frameName>${name}_link</frameName>
+          <frameName>${name}_optical_depth_frame</frameName>
           <imageTopicName>rgb/image_raw</imageTopicName>
           <depthImageTopicName>depth/image_raw</depthImageTopicName>

File: robotino_description/urdf/properties.urdf.xacro (robot description, xacro)
@@ -40,5 +40,5 @@
   <property name="kinect_z" value="0.0"/>
   <property name="kinect_roll" value="0.0"/>
-  <property name="kinect_pitch" value="0.0"/>
+  <property name="kinect_pitch" value="-${M_PI/2}"/>
   <property name="kinect_yaw" value="0.0"/>
   <!-- anglebracketusb mount positions | handeye calibration | relative to base_link -->

File: robotino_description/urdf/robotino.urdf.xacro (robot description, xacro)
@@ -33,5 +33,5 @@
   </kinect>
   <gazebo>
-    <plugin name="ros_control" filename="libmulti_hw_interface_gazebo_ros_control.so">
+    <plugin name="ros_control" filename="libgazebo_ros_control.so">
       <robotNamespace>tilt_controller</robotNamespace>
       <filterJointsParam>joint_names</filterJointsParam>

Commit message: redefined tf tree

File: robotino_description/urdf/gazebo.urdf.xacro (robot description, xacro)
@@ -53,5 +53,5 @@
 			<odometryFrame>odom</odometryFrame>
 			<odometryRate>20.0</odometryRate>
-			<robotBaseFrame>base_footprint</robotBaseFrame>
+			<robotBaseFrame>base_link</robotBaseFrame>
 		</plugin>
 	</gazebo>

File: robotino_description/urdf/robotino_body.urdf.xacro (robot description, xacro)
@@ -3,9 +3,9 @@
   <xacro:macro name="body" params="name">
    <link name="${name}_footprint"/>
-   <joint name="${name}_footprint_joint" type="fixed">
+<!--   <joint name="${name}_footprint_joint" type="fixed">
       <origin xyz="0 0 0" rpy="0 0 0" />
       <child link="${name}_link" />
       <parent link="${name}_footprint"/>
-   </joint>
+   </joint> -->
    <link name="${name}_link">
       <inertial>
