Commit message: removed footprint

File: robotino_description/urdf/robotino_body.urdf.xacro (robot description, xacro)
@@ -2,10 +2,10 @@
 <root xmlns:xacro="http://www.ros.org/wiki/xacro">
   <xacro:macro name="body" params="name">
-    <link name="${name}_footprint"/>
-    <joint name="${name}_footprint_joint" type="fixed">
-      <origin xyz="0 0 0" rpy="0 0 0" />
-      <child link="${name}_link" />
-      <parent link="${name}_footprint"/>
-    </joint>
+    <!-- <link name="${name}_footprint"/> -->
+    <!-- <joint name="${name}_footprint_joint" type="fixed"> -->
+    <!--   <origin xyz="0 0 0" rpy="0 0 0" /> -->
+    <!--   <child link="${name}_link" /> -->
+    <!--   <parent link="${name}_footprint"/> -->
+    <!-- </joint> -->
    <link name="${name}_link">
       <inertial>

Commit message: fixed inertial matrix for the base

File: robotino_description/urdf/robotino_body.urdf.xacro (robot description, xacro)
@@ -12,7 +12,7 @@
         <mass value="${BASE_MASS}" />
         <origin xyz="0 0 0" />
-        <inertia ixx="1.0" ixy="0.0" ixz="0.0"
-          iyy="1.0" iyz="0.0"
-          izz="1.0" />
+        <inertia ixx="75.0" ixy="0.0" ixz="0.0"
+          iyy="75.0" iyz="0.0"
+          izz="75.0" />
       </inertial>
       <visual>

Commit message: removed footprint frame

File: robotino_description/urdf/robotino_body.urdf.xacro (robot description, xacro)
@@ -2,6 +2,6 @@
 <root xmlns:xacro="http://www.ros.org/wiki/xacro">
   <xacro:macro name="body" params="name">
-   <link name="${name}_footprint"/>
-<!--   <joint name="${name}_footprint_joint" type="fixed">
+<!--<link name="${name}_footprint"/>
+   <joint name="${name}_footprint_joint" type="fixed">
       <origin xyz="0 0 0" rpy="0 0 0" />
       <child link="${name}_link" />
