Commit message: collision error

File: robotino_description/urdf/arm.urdf.xacro (robot description, xacro)
@@ -38,5 +38,5 @@
       </visual>
       <collision>
-        <origin xyz="0.0 0.175 0.0" rpy="1.57 0.0 0.0" />
+        <origin xyz="0.0 0.0 0.175" rpy="0 0.0 0.0" />
         <geometry>
           <cylinder radius="0.03" length="0.35"/>

Commit message: simplify model

File: robotino_description/urdf/arm.urdf.xacro (robot description, xacro)
@@ -105,5 +105,5 @@
       <parent link="arm_2_link" />
       <child link = "arm_3_link" />
-      <origin xyz="0.0 0.25 0.05" rpy="0.0 0.0 0.0" />
+      <origin xyz="0.0 0.25 -0.05" rpy="0.0 0.0 0.0" />
       <axis xyz="0 0 1" />
       <calibration rising="${arm_3_ref}"/>

File: robotino_description/urdf/robotino_body.urdf.xacro (robot description, xacro)
@@ -25,5 +25,5 @@
         <origin xyz="0.01 0 0" rpy="0 0 0"/>
         <geometry>
-          <mesh filename="package://robotino_description/meshes/RobotinoBody.dae"/>
+          <mesh filename="package://robotino_description/meshes/RobotinoBody.stl"/>
         </geometry>
       </collision>
