Commit message: new base_pan link

File: robotino_description/urdf/pan_tilt_axis.urdf.xacro (robot description, xacro)
@@ -2,7 +2,21 @@
 <root xmlns:xacro="http://www.ros.org/wiki/xacro">
   <xacro:macro name="pan_tilt_axis" params="parent *origin">
-    <joint name="pan_joint" type="revolute">
+    <joint name="base_pan_joint" type="fixed">
       <insert_block name="origin" />
       <parent link="${parent}"/>
+      <child link="base_pan_link" />
+    </joint>
+    <link name="base_pan_link">
+      <inertial>
+        <mass value="0.00001" />
+        <origin xyz="0 0 0" />
+        <inertia ixx="1.0" ixy="0.0" ixz="0.0"
+          iyy="1.0" iyz="0.0"
+          izz="1.0" />
+      </inertial>
+    </link>
+    <joint name="pan_joint" type="revolute">
+			<origin xyz="0 0 0" rpy="0 0 0"/>
+      <parent link="base_pan_link"/>
       <child link="pan_link" />
       <axis xyz="0 0 1" />

Commit message: new pan_tilt mesh model

File: robotino_description/urdf/pan_tilt_axis.urdf.xacro (robot description, xacro)
@@ -3,5 +3,5 @@
   <xacro:macro name="pan_tilt_axis" params="parent *origin">
     <joint name="base_pan_joint" type="fixed">
-      <insert_block name="origin" />
+			<origin xyz="0 0 0" rpy="0 0 0"/>
       <parent link="${parent}"/>
       <child link="base_pan_link" />
@@ -20,4 +20,5 @@
           <mesh filename="package://robotino_description/meshes/pan_tilt.stl"/>
         </geometry>
+        <material name="Black"/>
       </visual>
       <collision>
@@ -28,6 +29,11 @@
       </collision>
     </link>
+    <gazebo reference="base_pan_link">
+      <gravity>true</gravity>
+      <self_collide>false</self_collide>
+      <material>Gazebo/Black</material>
+    </gazebo>
     <joint name="pan_joint" type="revolute">
-			<origin xyz="0 0 0" rpy="0 0 0"/>
+      <insert_block name="origin" />
       <parent link="base_pan_link"/>
       <child link="pan_link" />

Commit message: a parent link has to have a collision and visual model

File: robotino_description/urdf/pan_tilt_axis.urdf.xacro (robot description, xacro)
@@ -3,5 +3,5 @@
   <xacro:macro name="pan_tilt_axis" params="parent *origin">
     <joint name="profile_joint" type="fixed">
-			<origin xyz="0 0 0" rpy="0 0 0"/>
+      <origin xyz="0 0 0" rpy="0 0 0"/>
       <parent link="${parent}"/>
       <child link="profile_link" />
@@ -40,5 +40,30 @@
     </joint>
     <link name="base_pan_link">
+      <inertial>
+        <mass value="0.00001" />
+        <origin xyz="0 0 0" />
+        <inertia ixx="1.0" ixy="0.0" ixz="0.0"
+          iyy="1.0" iyz="0.0"
+          izz="1.0" />
+      </inertial>
+      <visual>
+        <origin xyz="0 0 0" rpy="0 0 0" />
+        <geometry>
+          <box size="0.001 0.001 0.001" />
+        </geometry>
+        <material name="Black"/>
+      </visual>
+      <collision>
+        <origin xyz="0 0 0" rpy="0 0 0" />
+        <geometry>
+          <box size="0.001 0.001 0.001" />
+        </geometry>
+      </collision>
     </link>
+    <gazebo reference="base_pan_link">
+      <gravity>true</gravity>
+      <self_collide>false</self_collide>
+      <material>Gazebo/Black</material>
+    </gazebo>
     <joint name="pan_joint" type="revolute">
       <origin xyz="0 0 0" rpy="0 0 0"/>

File: robotino_description/urdf/pan_tilt_tuw_axis.urdf.xacro (robot description, xacro)
@@ -3,5 +3,5 @@
   <xacro:macro name="pan_tilt_axis" params="parent *origin">
     <joint name="profile_joint" type="fixed">
-			<origin xyz="0 0 0" rpy="0 0 0"/>
+      <origin xyz="0 0 0" rpy="0 0 0"/>
       <parent link="${parent}"/>
       <child link="profile_link" />
@@ -40,5 +40,30 @@
     </joint>
     <link name="base_pan_link">
+      <inertial>
+        <mass value="0.00001" />
+        <origin xyz="0 0 0" />
+        <inertia ixx="1.0" ixy="0.0" ixz="0.0"
+          iyy="1.0" iyz="0.0"
+          izz="1.0" />
+      </inertial>
+      <visual>
+        <origin xyz="0 0 0" rpy="0 0 0" />
+        <geometry>
+          <box size="0.001 0.001 0.001" />
+        </geometry>
+        <material name="Black"/>
+      </visual>
+      <collision>
+        <origin xyz="0 0 0" rpy="0 0 0" />
+        <geometry>
+          <box size="0.001 0.001 0.001" />
+        </geometry>
+      </collision>
     </link>
+    <gazebo reference="base_pan_link">
+      <gravity>true</gravity>
+      <self_collide>false</self_collide>
+      <material>Gazebo/Black</material>
+    </gazebo>
     <joint name="pan_joint" type="revolute">
       <origin xyz="0 0 0" rpy="0 0 0"/>
