Commit message: added footprint frame and tilt controllers

File: robotino_bringup/robots/ipa-robotino/urdf/robotino.urdf.xacro (robot description, xacro)
@@ -14,7 +14,4 @@
     <origin xyz="${hokuyo_x} ${hokuyo_y} ${hokuyo_z}" rpy="${hokuyo_roll} ${hokuyo_pitch} ${hokuyo_yaw}"/>
   </hokuyo>
-  <!--anglebracketusb name="anglebracketusb" parent="base_link">
-    <origin xyz="${anglebracketusb_x} ${anglebracketusb_y} ${anglebracketusb_z}" rpy="${anglebracketusb_roll} ${anglebracketusb_pitch} ${anglebracketusb_yaw}"/>
-  </anglebracketusb-->
   <tilt_axis name="tilt" parent="base_link">
     <origin xyz="${tilt_x} ${tilt_y} ${tilt_z}" rpy="${tilt_roll} ${tilt_pitch} ${tilt_yaw}"/>
@@ -23,9 +20,9 @@
     <origin xyz="${kinect_x} ${kinect_y} ${kinect_z}" rpy="${kinect_roll} ${kinect_pitch} ${kinect_yaw}"/>
   </kinect>
-  <!--gazebo>
+  <gazebo>
     <plugin name="ros_control" filename="libmulti_hw_interface_gazebo_ros_control.so">
       <robotNamespace>tilt_controller</robotNamespace>
       <filterJointsParam>joint_names</filterJointsParam>
     </plugin>
-  </gazebo-->
+  </gazebo>
 </robot>

File: robotino_description/urdf/robotino_body.urdf.xacro (robot description, xacro)
@@ -2,10 +2,10 @@
 <root xmlns:xacro="http://www.ros.org/wiki/xacro">
   <xacro:macro name="body" params="name">
-    <!-- <link name="${name}_footprint"/> -->
-	  <!-- <joint name="${name}_footprint_joint" type="fixed"> -->
-		<!--   <origin xyz="0 0 0" rpy="0 0 0" /> -->
-		<!--   <child link="${name}_link" /> -->
-		<!--   <parent link="${name}_footprint"/> -->
-	  <!-- </joint> -->
+   <link name="${name}_footprint"/>
+   <joint name="${name}_footprint_joint" type="fixed">
+      <origin xyz="0 0 0" rpy="0 0 0" />
+      <child link="${name}_link" />
+      <parent link="${name}_footprint"/>
+   </joint>
    <link name="${name}_link">
       <inertial>
