Commit message: update model

File: robotino_bringup/robots/ipa-robotino/urdf/properties.urdf.xacro (robot description, xacro)
@@ -22,7 +22,7 @@
   <property name="camera_yaw" value="-${M_PI/2}"/>
   <!-- hokuyo mount positions | relative to base_link -->
-  <property name="hokuyo_x" value="0.034"/>
+  <property name="hokuyo_x" value="0.064"/>
   <property name="hokuyo_y" value="0.0"/>
-  <property name="hokuyo_z" value="0.187"/>
+  <property name="hokuyo_z" value="0.22"/>
   <property name="hokuyo_roll" value="0.0"/>
   <property name="hokuyo_pitch" value="0.0"/>

File: robotino_bringup/robots/robotino/urdf/properties.urdf.xacro (robot description, xacro)
@@ -22,7 +22,7 @@
   <property name="camera_yaw" value="-${M_PI/2}"/>
   <!-- hokuyo mount positions | relative to base_link -->
-  <property name="hokuyo_x" value="0.034"/>
+  <property name="hokuyo_x" value="0.064"/>
   <property name="hokuyo_y" value="0.0"/>
-  <property name="hokuyo_z" value="0.187"/>
+  <property name="hokuyo_z" value="0.22"/>
   <property name="hokuyo_roll" value="0.0"/>
   <property name="hokuyo_pitch" value="0.0"/>
@@ -38,5 +38,5 @@
   <property name="arm_x" value="0.0"/>
   <property name="arm_y" value="0.0"/>
-  <property name="arm_z" value="0.0"/>
+  <property name="arm_z" value="0.35"/>
   <property name="arm_roll" value="0.0"/>
   <property name="arm_pitch" value="0.0"/>

File: robotino_bringup/robots/tuw-robotino/urdf/properties.urdf.xacro (robot description, xacro)
@@ -22,7 +22,7 @@
   <property name="camera_yaw" value="-${M_PI/2}"/>
   <!-- hokuyo mount positions | relative to base_link -->
-  <property name="hokuyo_x" value="0.034"/>
+  <property name="hokuyo_x" value="0.064"/>
   <property name="hokuyo_y" value="0.0"/>
-  <property name="hokuyo_z" value="0.187"/>
+  <property name="hokuyo_z" value="0.22"/>
   <property name="hokuyo_roll" value="0.0"/>
   <property name="hokuyo_pitch" value="0.0"/>

File: robotino_description/urdf/arm.urdf.xacro (robot description, xacro)
@@ -31,5 +31,5 @@
         <origin xyz="0.0 0.0 0.175" rpy="0 0.0 0.0" />
         <geometry>
-          <cylinder radius="0.03" length="0.35"/>
+          <cylinder radius="0.0" length="0.0"/>
         </geometry>
         <material name="LightGrey">
@@ -40,5 +40,5 @@
         <origin xyz="0.0 0.0 0.175" rpy="0 0.0 0.0" />
         <geometry>
-          <cylinder radius="0.03" length="0.35"/>
+          <cylinder radius="0.0" length="0.0"/>
         </geometry>
       </collision>
@@ -47,5 +47,5 @@
       <parent link="arm_base_link" />
       <child link = "arm_1_link" />
-      <origin xyz="0.15 0.0 0.35" rpy="-1.57 0.0 0.0" />
+      <origin xyz="0.0 0.0 0.0" rpy="0.0 0.0 0.0" />
       <axis xyz="0 0 1" />
       <calibration rising="${arm_1_ref}"/>
@@ -55,23 +55,26 @@
       <xacro:default_inertial/>
       <visual>
-        <origin xyz="0.125 0.0 0.0" rpy="0.0 1.57 0.0" />
-        <geometry>
-          <cylinder radius="0.025" length="0.25"/>
-        </geometry>
-        <material name="LightGrey">
-          <color rgba="0.7 0.7 0.7 1.0"/>
-        </material>
-      </visual>
-      <collision>
-        <origin xyz="0.125 0.0 0.0" rpy="0.0 1.57 0.0" />
-        <geometry>
-          <cylinder radius="0.025" length="0.25"/>
-        </geometry>
-      </collision>
-    </link>
+        <origin xyz="0.0 0.0 -0.04" rpy="0.0 0.0 0.0" />
+        <geometry>
+          <box size="0.08 0.08 0.08"/>
+        </geometry>
+        <material name="Black">
+          <color rgba="0 0 0 1.0"/>
+        </material>
+      </visual>
+      <collision>
+        <origin xyz="0.0 0.0 -0.04" rpy="0.0 0.0 0.0" />
+        <geometry>
+          <cylinder radius="0.025" length="0.08"/>
+        </geometry>
+      </collision>
+    </link>
+    <gazebo reference="arm_1_link">
+        <material>Gazebo/Black</material>
+    </gazebo>
     <joint name="arm_2_joint" type="revolute">
       <parent link="arm_1_link" />
       <child link = "arm_2_link" />
-      <origin xyz="0.25 0.0 0.0" rpy="0.0 0.0 0.0" />
+      <origin xyz="0.0 0.0 0.0" rpy="1.57 0.0 0.0" />
       <axis xyz="0 0 1" />
       <calibration rising="${arm_2_ref}"/>
@@ -81,21 +84,26 @@
       <xacro:default_inertial/>
       <visual>
-        <geometry>
-          <cylinder radius="0.03" length="0.05"/>
-        </geometry>
-        <material name="LightGrey">
-          <color rgba="0.7 0.7 0.7 1.0"/>
-        </material>
-      </visual>
-      <collision>
-        <geometry>
-          <box size="0.01 0.01 0.01"/>
-        </geometry>
-      </collision>
-    </link>
+        <origin xyz="0.0 0.125 0.0" rpy="1.57 0.0 0.0" />
+        <geometry>
+          <cylinder radius="0.025" length="0.25"/>
+        </geometry>
+        <material name="LightGrey">
+          <color rgba="0.7 0.7 0.7 1.0"/>
+        </material>
+      </visual>
+      <collision>
+        <origin xyz="0.0 0.125 0.0" rpy="1.57 0.0 0.0" />
+        <geometry>
+          <cylinder radius="0.025" length="0.25"/>
+        </geometry>
+      </collision>
+    </link>
+    <gazebo reference="arm_2_link">
+        <material>Gazebo/Grey</material>
+    </gazebo>
     <joint name="arm_3_joint" type="revolute">
       <parent link="arm_2_link" />
       <child link = "arm_3_link" />
-      <origin xyz="0.0 0.0 0.0" rpy="1.57 0.0 1.57" />
+      <origin xyz="0.0 0.25 0.05" rpy="0.0 0.0 0.0" />
       <axis xyz="0 0 1" />
       <calibration rising="${arm_3_ref}"/>
@@ -105,23 +113,26 @@
       <xacro:default_inertial/>
       <visual>
-        <origin xyz="0.0 0.0 0.125" rpy="0.0 0.0 0.0" />
-        <geometry>
-          <cylinder radius="0.025" length="0.25"/>
-        </geometry>
-        <material name="LightGrey">
-          <color rgba="0.7 0.7 0.7 1.0"/>
-        </material>
-      </visual>
-      <collision>
-        <origin xyz="0.0 0.0 0.125" rpy="0.0 0.0 0.0" />
-        <geometry>
-          <cylinder radius="0.025" length="0.25"/>
-        </geometry>
-      </collision>
-    </link>
+        <origin xyz="0.0 0.125 0.0" rpy="-1.57 0.0 0.0" />
+        <geometry>
+          <cylinder radius="0.025" length="0.25"/>
+        </geometry>
+        <material name="Black">
+          <color rgba="0 0 0 1.0"/>
+        </material>
+      </visual>
+      <collision>
+        <origin xyz="0.0 0.125 0.0" rpy="-1.57 0.0 0.0" />
+        <geometry>
+          <cylinder radius="0.025" length="0.25"/>
+        </geometry>
+      </collision>
+    </link>
+    <gazebo reference="arm_3_link">
+        <material>Gazebo/Black</material>
+    </gazebo>
     <joint name="arm_4_joint" type="revolute">
       <parent link="arm_3_link" />
       <child link = "arm_4_link" />
-      <origin xyz="0.0 0.0 0.25" rpy="-1.57 0.0 0.0" />
+      <origin xyz="0.0 0.175 0.0" rpy="-1.57 0.0 0.0" />
       <axis xyz="0 0 1" />
       <calibration rising="${arm_4_ref}"/>
@@ -131,21 +142,26 @@
       <xacro:default_inertial/>
       <visual>
-        <geometry>
-          <cylinder radius="0.03" length="0.05"/>
-        </geometry>
-        <material name="LightGrey">
-          <color rgba="0.7 0.7 0.7 1.0"/>
-        </material>
-      </visual>
-      <collision>
-        <geometry>
-          <box size="0.01 0.01 0.01"/>
-        </geometry>
-      </collision>
-    </link>
+        <origin xyz="0.0 0.0 -0.0375" rpy="0.0 0.0 0.0" />
+        <geometry>
+          <cylinder radius="0.04" length="0.05"/>
+        </geometry>
+        <material name="LightGrey">
+          <color rgba="0.7 0.7 0.7 1.0"/>
+        </material>
+      </visual>
+      <collision>
+        <origin xyz="0.0 0.0 -0.0375" rpy="0.0 0.0 0.0" />
+        <geometry>
+          <cylinder radius="0.04" length="0.05"/>
+        </geometry>
+      </collision>
+    </link>
+    <gazebo reference="arm_4_link">
+        <material>Gazebo/Grey</material>
+    </gazebo>
     <joint name="arm_5_joint" type="revolute">
       <parent link="arm_4_link" />
       <child link = "arm_5_link" />
-      <origin xyz="0.0 0.0 0.0" rpy="1.57 0.0 0.0" />
+      <origin xyz="0.0 0.05 0.075" rpy="1.57 0.0 0.0" />
       <axis xyz="0 0 1" />
       <calibration rising="${arm_5_ref}"/>
@@ -155,23 +171,26 @@
       <xacro:default_inertial/>
       <visual>
-        <origin xyz="0.0 0.0 0.0375" rpy="0.0 0.0 0.0" />
-        <geometry>
-          <cylinder radius="0.025" length="0.075"/>
-        </geometry>
-        <material name="LightGrey">
-          <color rgba="0.7 0.7 0.7 1.0"/>
-        </material>
-      </visual>
-      <collision>
-        <origin xyz="0.0 0.0 0.0375" rpy="0.0 0.0 0.0" />
-        <geometry>
-          <cylinder radius="0.025" length="0.075"/>
-        </geometry>
-      </collision>
-    </link>
+        <origin xyz="0.0 0.0175 0.0" rpy="-1.57 0.0 0.0" />
+        <geometry>
+          <cylinder radius="0.025" length="0.035"/>
+        </geometry>
+        <material name="Black">
+          <color rgba="0 0 0 1.0"/>
+        </material>
+      </visual>
+      <collision>
+        <origin xyz="0.0 0.0175 0.0" rpy="-1.57 0.0 0.0" />
+        <geometry>
+          <cylinder radius="0.025" length="0.035"/>
+        </geometry>
+      </collision>
+    </link>
+    <gazebo reference="arm_5_link">
+        <material>Gazebo/Black</material>
+    </gazebo>
     <joint name="arm_6_joint" type="revolute">
       <parent link="arm_5_link" />
       <child link = "arm_6_link" />
-      <origin xyz="0.0 0.0 0.075" rpy="0.0 0.0 0.0" />
+      <origin xyz="0.0 0.035 0.0" rpy="-1.57 0.0 0.0" />
       <axis xyz="0 0 1" />
       <calibration rising="${arm_6_ref}"/>
@@ -181,4 +200,5 @@
       <xacro:default_inertial/>
       <visual>
+        <origin xyz="0.0 0.0 0.0125" rpy="0.0 0.0 0.0" />
         <geometry>
           <cylinder radius="0.025" length="0.025"/>
@@ -189,9 +209,13 @@
       </visual>
       <collision>
-        <geometry>
-          <box size="0.01 0.01 0.01"/>
-        </geometry>
-      </collision>
-    </link>
+        <origin xyz="0.0 0.0 -0.0125" rpy="0.0 0.0 0.0" />
+        <geometry>
+          <cylinder radius="0.025" length="0.025"/>
+        </geometry>
+      </collision>
+    </link>
+    <gazebo reference="arm_6_link">
+        <material>Gazebo/Grey</material>
+    </gazebo>
     <xacro:arm_SimpleTransmission number="1"></xacro:arm_SimpleTransmission>
     <xacro:arm_SimpleTransmission number="2"></xacro:arm_SimpleTransmission>

File: robotino_description/urdf/robotino_body.urdf.xacro (robot description, xacro)
@@ -17,13 +17,13 @@
       </inertial>
       <visual>
-        <origin xyz="0.01 0 0" rpy="0 0 ${M_PI/2}"/>
+        <origin xyz="0.01 0 0" rpy="0 0 0"/>
         <geometry>
-          <mesh filename="package://robotino_description/meshes/RobotinoBody.dae" scale="${M_SCALE} ${M_SCALE} ${M_SCALE}"/>
+          <mesh filename="package://robotino_description/meshes/RobotinoBody.dae"/>
         </geometry>
       </visual>
       <collision>
-        <origin xyz="0.01 0 0" rpy="0 0 ${M_PI/2}"/>
+        <origin xyz="0.01 0 0" rpy="0 0 0"/>
         <geometry>
-          <mesh filename="package://robotino_description/meshes/RobotinoBody.dae" scale="${M_SCALE} ${M_SCALE} ${M_SCALE}"/>
+          <mesh filename="package://robotino_description/meshes/RobotinoBody.dae"/>
         </geometry>
       </collision>
@@ -31,5 +31,5 @@
     <base_gazebo name="base" />
     <wheel name="wheel0" parent="base_link">
-      <origin xyz="0.065 0.11 0.04" rpy="0 0 ${M_PI/3}"/>
+      <origin xyz="0.095 0.14 0.02" rpy="0 0 ${M_PI/3}"/>
       <axis xyz="-1 0 0"/>
     </wheel>
@@ -37,5 +37,5 @@
     <wheel_gazebo name="wheel0" />
     <wheel name="wheel1" parent="base_link">
-      <origin xyz="-0.13 0 0.04" rpy="0 0 0"/>
+      <origin xyz="-0.16 0 0.02" rpy="0 0 0"/>
       <axis xyz="1 0 0"/>
     </wheel>
@@ -43,5 +43,5 @@
     <wheel_gazebo name="wheel1" />
     <wheel name="wheel2" parent="base_link">
-      <origin xyz="0.065 -0.11 0.04" rpy="0 0 -${M_PI/3}"/>
+      <origin xyz="0.105 -0.15 0.02" rpy="0 0 -${M_PI/3}"/>
       <axis xyz="-1 0 0"/>
     </wheel>

Commit message: calibration

File: robotino_bringup/robots/ipa-robotino/urdf/properties.urdf.xacro (robot description, xacro)
@@ -11,7 +11,7 @@
   <property name="HOKUYO_RADIUS" value="0.02"/>
   <property name="HOKUYO_LENGTH" value="0.07"/>
-  <property name="KINECT_LENGTH" value="0.035"/>
-  <property name="KINECT_WIDTH" value="0.18"/>
-  <property name="KINECT_HEIGHT" value="0.05"/>
+  <property name="KINECT_LENGTH" value="0.18"/>
+  <property name="KINECT_WIDTH" value="0.035"/>
+  <property name="KINECT_HEIGHT" value="0.02"/>
   <!-- camera mount positions | handeye calibration | relative to base_link -->
   <property name="camera_x" value="0.0"/>
@@ -29,5 +29,5 @@
   <property name="hokuyo_yaw" value="0.0"/>
    <!-- tilt mount positions | handeye calibration | relative to base_link -->
-  <property name="tilt_x" value="-0.01"/>
+  <property name="tilt_x" value="0.02"/>
   <property name="tilt_y" value="0.0"/>
   <property name="tilt_z" value="0.45"/>

File: robotino_bringup/robots/robotino/urdf/properties.urdf.xacro (robot description, xacro)
@@ -11,7 +11,7 @@
   <property name="HOKUYO_RADIUS" value="0.02"/>
   <property name="HOKUYO_LENGTH" value="0.07"/>
-  <property name="KINECT_LENGTH" value="0.035"/>
-  <property name="KINECT_WIDTH" value="0.18"/>
-  <property name="KINECT_HEIGHT" value="0.05"/>
+  <property name="KINECT_LENGTH" value="0.18"/>
+  <property name="KINECT_WIDTH" value="0.035"/>
+  <property name="KINECT_HEIGHT" value="0.02"/>
   <!-- camera mount positions | handeye calibration | relative to base_link -->
   <property name="camera_x" value="0.0"/>

File: robotino_bringup/robots/tuw-robotino/urdf/properties.urdf.xacro (robot description, xacro)
@@ -11,7 +11,7 @@
   <property name="HOKUYO_RADIUS" value="0.02"/>
   <property name="HOKUYO_LENGTH" value="0.07"/>
-  <property name="KINECT_LENGTH" value="0.035"/>
-  <property name="KINECT_WIDTH" value="0.18"/>
-  <property name="KINECT_HEIGHT" value="0.05"/>
+  <property name="KINECT_LENGTH" value="0.18"/>
+  <property name="KINECT_WIDTH" value="0.035"/>
+  <property name="KINECT_HEIGHT" value="0.02"/>
   <!-- camera mount positions | handeye calibration | relative to base_link -->
   <property name="camera_x" value="0.0"/>

File: robotino_bringup/robots/uibk-robotino/urdf/properties.urdf.xacro (robot description, xacro)
@@ -11,7 +11,7 @@
   <property name="HOKUYO_RADIUS" value="0.02"/>
   <property name="HOKUYO_LENGTH" value="0.07"/>
-  <property name="KINECT_LENGTH" value="0.035"/>
-  <property name="KINECT_WIDTH" value="0.18"/>
-  <property name="KINECT_HEIGHT" value="0.05"/>
+  <property name="KINECT_LENGTH" value="0.18"/>
+  <property name="KINECT_WIDTH" value="0.035"/>
+  <property name="KINECT_HEIGHT" value="0.02"/>
   <!-- camera mount positions | handeye calibration | relative to base_link -->
   <property name="camera_x" value="0.0"/>

File: robotino_description/urdf/kinect.urdf.xacro (robot description, xacro)
@@ -18,5 +18,5 @@
         <origin xyz="0 0 0" rpy="0 0 0" />
         <geometry>
-          <box size="${KINECT_LENGTH} ${KINECT_WIDTH} ${KINECT_HEIGHT}"/>
+          <box size="${KINECT_WIDTH} ${KINECT_LENGTH} ${KINECT_HEIGHT}"/>
         </geometry>
         <material name="Grey"/>
@@ -25,5 +25,5 @@
         <origin xyz="0 0 0" rpy="0 0 0" />
         <geometry>
-          <box size="${KINECT_LENGTH} ${KINECT_WIDTH} ${KINECT_HEIGHT}"/>
+          <box size="${KINECT_WIDTH}  ${KINECT_LENGTH} ${KINECT_HEIGHT}"/>
         </geometry>
       </collision>
