Commit message: update and clean robot files

File: robotino_bringup/robots/ipa-robotino/urdf/properties.urdf.xacro (robot description, xacro)
@@ -14,11 +14,4 @@
   <property name="KINECT_WIDTH" value="0.035"/>
   <property name="KINECT_HEIGHT" value="0.02"/>
-  <!-- camera mount positions | handeye calibration | relative to base_link -->
-  <property name="camera_x" value="0.0"/>
-  <property name="camera_y" value="0.0"/>
-  <property name="camera_z" value="0.2"/>
-  <property name="camera_roll" value="0.0"/>
-  <property name="camera_pitch" value="0.0"/>
-  <property name="camera_yaw" value="-${M_PI/2}"/>
   <!-- hokuyo mount positions | relative to base_link -->
   <property name="hokuyo_x" value="0.064"/>
@@ -42,10 +35,3 @@
   <property name="kinect_pitch" value="-1.45"/>
   <property name="kinect_yaw" value="0.0"/>
-  <!-- anglebracketusb mount positions | handeye calibration | relative to base_link -->
-  <property name="anglebracketusb_x" value="0.008"/>
-  <property name="anglebracketusb_y" value="0.0"/>
-  <property name="anglebracketusb_z" value="0.137"/>
-  <property name="anglebracketusb_roll" value="0.0"/>
-  <property name="anglebracketusb_pitch" value="0.0"/>
-  <property name="anglebracketusb_yaw" value="0.0"/>
 </robot>

File: robotino_bringup/robots/ipa-robotino/urdf/robotino.urdf.xacro (robot description, xacro)
@@ -1,12 +1,12 @@
 <?xml version="1.0"?>
 <robot xmlns:xacro="http://www.ros.org/wiki/xacro"
-  name="robotino">
+  name="robot">
   <xacro:include filename="$(find robotino_bringup)/robots/ipa-robotino/urdf/properties.urdf.xacro" />
   <xacro:include filename="$(find robotino_description)/urdf/gazebo.urdf.xacro" />
-  <xacro:include filename="$(find robotino_description)/urdf/robotino_body.urdf.xacro" />
+  <xacro:include filename="$(find robotino_description)/urdf/base.urdf.xacro" />
   <xacro:include filename="$(find robotino_description)/urdf/hokuyo.urdf.xacro" />
   <xacro:include filename="$(find robotino_description)/urdf/kinect.urdf.xacro" />
   <xacro:include filename="$(find robotino_description)/urdf/tilt_axis.urdf.xacro" />
-  <xacro:body name="base"/>
+  <xacro:base name="base"/>
   <gazebo>
     <plugin name="ros_control" filename="libhwi_switch_gazebo_ros_control.so">

File: robotino_bringup/robots/kcl-hand/urdf/robotino.urdf.xacro (robot description, xacro)
@@ -5,8 +5,26 @@
   <xacro:include filename="$(find robotino_description)/urdf/gazebo.urdf.xacro" />
   <xacro:include filename="$(find kclhand_description)/urdf/kclhand.urdf.xacro" />
-  <link name="world"/>
+  <link name="base_link">
+    <inertial>
+      <mass value="3" />
+      <origin xyz="0 0 0" />
+      <inertia ixx="0.001" ixy="0.0" ixz="0.0" iyy="0.001" iyz="0.0" izz="0.001" />
+    </inertial>
+    <visual>
+      <origin xyz="0 0 0.3" rpy="0 0 0" />
+      <geometry>
+        <cylinder length="0.6" radius="0.1"/>
+      </geometry>
+    </visual>
+    <collision>
+      <origin xyz="0 0 0.3" rpy="0 0 0" />
+      <geometry>
+        <cylinder length="0.6" radius="0.1"/>
+      </geometry>
+    </collision>
+  </link>
   <!-- hand -->
-  <xacro:kclhand name="hand" parent="world">
-    <origin xyz="0 0 0.25" rpy="1.57 0 0" />
+  <xacro:kclhand name="hand" parent="base_link">
+    <origin xyz="0 0 0.55" rpy="1.57 0 0" />
   </xacro:kclhand>
   <gazebo>

File: robotino_bringup/robots/tuw-robotino/urdf/properties.urdf.xacro (robot description, xacro)
@@ -14,11 +14,4 @@
   <property name="KINECT_WIDTH" value="0.035"/>
   <property name="KINECT_HEIGHT" value="0.02"/>
-  <!-- camera mount positions | handeye calibration | relative to base_link -->
-  <property name="camera_x" value="0.0"/>
-  <property name="camera_y" value="0.0"/>
-  <property name="camera_z" value="0.2"/>
-  <property name="camera_roll" value="0.0"/>
-  <property name="camera_pitch" value="0.0"/>
-  <property name="camera_yaw" value="-${M_PI/2}"/>
   <!-- hokuyo mount positions | relative to base_link -->
   <property name="hokuyo_x" value="0.184"/>
@@ -28,10 +21,11 @@
   <property name="hokuyo_pitch" value="0.0"/>
   <property name="hokuyo_yaw" value="-0.015"/>
-  <property name="pan_tilt_x" value="0.191663"/>
-  <property name="pan_tilt_y" value="0.175084"/>
-  <property name="pan_tilt_z" value="0.616622"/>
-  <property name="pan_tilt_roll" value="0.01724"/>
-  <property name="pan_tilt_pitch" value="0.0135072"/>
-  <property name="pan_tilt_yaw" value="1.09491"/>
+  <!-- pan-tilt mount positions | relative to base_link -->
+  <property name="pan_tilt_x" value="0.193"/> <!--base_radius+0.013-->
+  <property name="pan_tilt_y" value="0.005"/>
+  <property name="pan_tilt_z" value="0.61"/>
+  <property name="pan_tilt_roll" value="0.0"/>
+  <property name="pan_tilt_pitch" value="0.0"/>
+  <property name="pan_tilt_yaw" value="0.0"/>
   <!-- kinect mount positions | handeye calibration | relative to pan_tilt_link -->
   <property name="kinect_x" value="-0.031924"/>
@@ -41,26 +35,3 @@
   <property name="kinect_pitch" value="0.00219856"/>
   <property name="kinect_yaw" value="0.00966127"/>
-  <!-- Federicos paramters-->
-  <!-- pan_tilt mount positions | handeye calibration | relative to base_pan_link -->
-  <!--<property name="pan_tilt_x" value="0.145"/>
-  <property name="pan_tilt_y" value="0.194"/>
-  <property name="pan_tilt_z" value="0.64"/>
-  <property name="pan_tilt_roll" value="0.0"/>
-  <property name="pan_tilt_pitch" value="0.0"/>
-  <property name="pan_tilt_yaw" value="1.0472"/> -->
-  <!-- kinect mount positions | handeye calibration | relative to pan_tilt_link -->
-  <!-- good for 0.75 -->
-  <!--<property name="kinect_x" value="0.03129"/>
-  <property name="kinect_y" value="0.038"/>
-  <property name="kinect_z" value="-0.0"/>
-  <property name="kinect_roll" value="-1.56905"/>
-  <property name="kinect_pitch" value="0.0434565"/>
-  <property name="kinect_yaw" value="0.00767917"/> -->
-  <!-- good for 0.75 -->
-  <!-- <property name="kinect_x" value="0.03129"/> -->
-  <!-- <property name="kinect_y" value="0.038"/> -->
-  <!-- <property name="kinect_z" value="-0.0"/> -->
-  <!-- <property name="kinect_roll" value="-1.56905"/> -->
-  <!-- <property name="kinect_pitch" value="0.0434565"/> -->
-  <!-- <property name="kinect_yaw" value="0.00667917"/> -->
 </robot>

File: robotino_bringup/robots/tuw-robotino/urdf/robotino.urdf.xacro (robot description, xacro)
@@ -1,18 +1,12 @@
 <?xml version="1.0"?>
 <robot xmlns:xacro="http://www.ros.org/wiki/xacro"
-  name="robotino">
+  name="robot">
   <xacro:include filename="$(find robotino_bringup)/robots/tuw-robotino/urdf/properties.urdf.xacro" />
   <xacro:include filename="$(find robotino_description)/urdf/gazebo.urdf.xacro" />
-  <xacro:include filename="$(find robotino_description)/urdf/robotino_body.urdf.xacro" />
+  <xacro:include filename="$(find robotino_description)/urdf/base.urdf.xacro" />
   <xacro:include filename="$(find robotino_description)/urdf/hokuyo.urdf.xacro" />
   <xacro:include filename="$(find robotino_description)/urdf/kinect.urdf.xacro" />
   <xacro:include filename="$(find robotino_description)/urdf/pan_tilt_tuw_axis.urdf.xacro" />
-  <xacro:body name="base"/>
-  <gazebo>
-    <plugin name="ros_control" filename="libhwi_switch_gazebo_ros_control.so">
-      <robotNamespace>base_controller</robotNamespace>
-      <filterJointsParam>joint_names</filterJointsParam>
-    </plugin>
-  </gazebo>
+  <xacro:base name="base"/>
   <gazebo>
     <plugin name="ros_control" filename="libhwi_switch_gazebo_ros_control.so">

File: robotino_bringup/robots/tuw-robotino2/urdf/properties.urdf.xacro (robot description, xacro)
@@ -14,11 +14,4 @@
   <property name="KINECT_WIDTH" value="0.035"/>
   <property name="KINECT_HEIGHT" value="0.02"/>
-  <!-- camera mount positions | handeye calibration | relative to base_link -->
-  <property name="camera_x" value="0.0"/>
-  <property name="camera_y" value="0.0"/>
-  <property name="camera_z" value="0.2"/>
-  <property name="camera_roll" value="0.0"/>
-  <property name="camera_pitch" value="0.0"/>
-  <property name="camera_yaw" value="-${M_PI/2}"/>
   <!-- hokuyo mount positions | relative to base_link -->
   <property name="hokuyo_x" value="0.184"/>

File: robotino_bringup/robots/uibk-robotino2/urdf/properties.urdf.xacro (robot description, xacro)
@@ -14,11 +14,4 @@
   <property name="KINECT_WIDTH" value="0.035"/>
   <property name="KINECT_HEIGHT" value="0.02"/>
-  <!-- camera mount positions | handeye calibration | relative to base_link -->
-  <property name="camera_x" value="0.0"/>
-  <property name="camera_y" value="0.0"/>
-  <property name="camera_z" value="0.2"/>
-  <property name="camera_roll" value="0.0"/>
-  <property name="camera_pitch" value="0.0"/>
-  <property name="camera_yaw" value="-${M_PI/2}"/>
   <!-- hokuyo mount positions | relative to base_link -->
   <property name="hokuyo_x" value="0.208610627"/>
