Commit message: first arm URDF version

File: robotino_bringup/robots/robotino/urdf/properties.urdf.xacro (robot description, xacro)
@@ -35,5 +35,19 @@
   <property name="tilt_pitch" value="${M_PI/2}"/>
   <property name="tilt_yaw" value="0"/>
-  <!-- kinect mount positions | handeye calibration | relative to tilt_link -->
+   <!-- arm mount positions | handeye calibration | relative to base_link -->
+  <property name="arm_x" value="0.0"/>
+  <property name="arm_y" value="0.0"/>
+  <property name="arm_z" value="0.35"/>
+  <property name="arm_roll" value="0.0"/>
+  <property name="arm_pitch" value="0"/>
+  <property name="arm_yaw" value="-${M_PI/2}"/>
+   <!-- arm calibration-->
+  <property name="arm_1_ref" value="0.0"/>
+  <property name="arm_2_ref" value="0.0"/>
+  <property name="arm_3_ref" value="0.0"/>
+  <property name="arm_4_ref" value="0.0"/>
+  <property name="arm_5_ref" value="0.0"/>
+  <property name="arm_6_ref" value="0.0"/>
+   <!-- kinect mount positions | handeye calibration | relative to tilt_link -->
   <property name="kinect_x" value="-0.03"/>
   <property name="kinect_y" value="0.0"/>
@@ -42,5 +56,5 @@
   <property name="kinect_pitch" value="-1.45"/>
   <property name="kinect_yaw" value="0.0"/>
-  <!-- anglebracketusb mount positions | handeye calibration | relative to base_link -->
+   <!-- anglebracketusb mount positions | handeye calibration | relative to base_link -->
   <property name="anglebracketusb_x" value="0.008"/>
   <property name="anglebracketusb_y" value="0.0"/>

File: robotino_bringup/robots/robotino/urdf/robotino.urdf.xacro (robot description, xacro)
@@ -10,17 +10,18 @@
   <xacro:include filename="$(find robotino_description)/urdf/kinect.urdf.xacro" />
   <xacro:include filename="$(find robotino_description)/urdf/tilt_axis.urdf.xacro" />
+  <xacro:include filename="$(find robotino_description)/urdf/arm.urdf.xacro" />
   <xacro:body name="base"/>
   <hokuyo name="hokuyo" parent="base_link">
     <origin xyz="${hokuyo_x} ${hokuyo_y} ${hokuyo_z}" rpy="${hokuyo_roll} ${hokuyo_pitch} ${hokuyo_yaw}"/>
   </hokuyo>
-  <tilt_axis name="tilt" parent="base_link">
+  <!--tilt_axis name="tilt" parent="base_link">
     <origin xyz="${tilt_x} ${tilt_y} ${tilt_z}" rpy="${tilt_roll} ${tilt_pitch} ${tilt_yaw}"/>
   </tilt_axis>
   <kinect name="kinect" parent="tilt_link">
     <origin xyz="${kinect_x} ${kinect_y} ${kinect_z}" rpy="${kinect_roll} ${kinect_pitch} ${kinect_yaw}"/>
-  </kinect>
-  <!--anglebracketusb name="anglebracketusb" parent="base_link">
-    <origin xyz="${anglebracketusb_x} ${anglebracketusb_y} ${anglebracketusb_z}" rpy="${anglebracketusb_roll} ${anglebracketusb_pitch} ${anglebracketusb_yaw}"/>
-  </anglebracketusb-->
+  </kinect-->
+  <arm parent="base_link">
+    <origin xyz="${arm_x} ${arm_y} ${arm_z}" rpy="${arm_roll} ${arm_pitch} ${arm_yaw}"/>
+  </arm>
   <gazebo>
     <plugin name="ros_control" filename="libmulti_hw_interface_gazebo_ros_control.so">

Commit message: review arm kinematic

File: robotino_bringup/robots/robotino/urdf/properties.urdf.xacro (robot description, xacro)
@@ -39,7 +39,7 @@
   <property name="arm_y" value="0.0"/>
   <property name="arm_z" value="0.35"/>
-  <property name="arm_roll" value="0.0"/>
-  <property name="arm_pitch" value="0"/>
-  <property name="arm_yaw" value="-${M_PI/2}"/>
+  <property name="arm_roll" value="-${M_PI/2}"/>
+  <property name="arm_pitch" value="0.0"/>
+  <property name="arm_yaw" value="0.0"/>
    <!-- arm calibration-->
   <property name="arm_1_ref" value="0.0"/>

File: robotino_description/urdf/arm.urdf.xacro (robot description, xacro)
@@ -31,5 +31,5 @@
       <parent link="arm_1_link" />
       <child link = "arm_2_link" />
-      <origin xyz="0.0 0.0 0.25" rpy="0.0 0.0 0.0" />
+      <origin xyz="0.25 0.0 0.0" rpy="0.0 0.0 0.0" />
       <axis xyz="0 0 1" />
       <calibration rising="${arm_2_ref}"/>
@@ -79,5 +79,5 @@
       <parent link="arm_3_link" />
       <child link = "arm_4_link" />
-      <origin xyz="0.0 0.0 0.25" rpy="0.0 0.0 -1.57" />
+      <origin xyz="0.0 0.0 0.25" rpy="-1.57 0.0 0.0" />
       <axis xyz="0 0 1" />
       <calibration rising="${arm_4_ref}"/>
@@ -103,5 +103,5 @@
       <parent link="arm_4_link" />
       <child link = "arm_5_link" />
-      <origin xyz="0.0 0.0 0.0" rpy="0.0 0.0 1.57" />
+      <origin xyz="0.0 0.0 0.0" rpy="1.57 0.0 0.0" />
       <axis xyz="0 0 1" />
       <calibration rising="${arm_5_ref}"/>

Commit message: add arm controllers

File: robotino_bringup/robots/robotino/urdf/properties.urdf.xacro (robot description, xacro)
@@ -38,6 +38,6 @@
   <property name="arm_x" value="0.0"/>
   <property name="arm_y" value="0.0"/>
-  <property name="arm_z" value="0.35"/>
-  <property name="arm_roll" value="-${M_PI/2}"/>
+  <property name="arm_z" value="0.0"/>
+  <property name="arm_roll" value="0.0"/>
   <property name="arm_pitch" value="0.0"/>
   <property name="arm_yaw" value="0.0"/>

File: robotino_bringup/robots/robotino/urdf/robotino.urdf.xacro (robot description, xacro)
@@ -26,5 +26,5 @@
   <gazebo>
     <plugin name="ros_control" filename="libhwi_switch_gazebo_ros_control.so">
-      <robotNamespace>tilt_controller</robotNamespace>
+      <robotNamespace>arm_controller</robotNamespace>
       <filterJointsParam>joint_names</filterJointsParam>
     </plugin>

File: robotino_description/urdf/arm.urdf.xacro (robot description, xacro)
@@ -8,4 +8,16 @@
     </inertial>
   </xacro:macro>
+  <xacro:macro name="arm_SimpleTransmission" params="number">
+    <transmission name="arm_${number}_trans">
+      <type>transmission_interface/SimpleTransmission</type>
+      <joint name="arm_${number}_joint">
+        <hardwareInterface>PositionJointInterface</hardwareInterface>
+        <hardwareInterface>VelocityJointInterface</hardwareInterface>
+      </joint>
+      <actuator name="arm_${number}_motor">
+        <mechanicalReduction>1</mechanicalReduction>
+      </actuator>
+    </transmission>
+  </xacro:macro>
   <xacro:macro name="arm" params="parent *origin">
     <joint name="arm_base_joint" type="fixed">
@@ -16,9 +28,24 @@
     <link name="arm_base_link" >
       <xacro:default_inertial/>
+      <visual>
+        <origin xyz="0.0 0.0 0.175" rpy="0 0.0 0.0" />
+        <geometry>
+          <cylinder radius="0.03" length="0.35"/>
+        </geometry>
+        <material name="LightGrey">
+          <color rgba="0.7 0.7 0.7 1.0"/>
+        </material>
+      </visual>
+      <collision>
+        <origin xyz="0.0 0.175 0.0" rpy="1.57 0.0 0.0" />
+        <geometry>
+          <cylinder radius="0.03" length="0.35"/>
+        </geometry>
+      </collision>
     </link>
     <joint name="arm_1_joint" type="revolute">
       <parent link="arm_base_link" />
       <child link = "arm_1_link" />
-      <origin xyz="0.0 0.0 0.0" rpy="0.0 0.0 0.0" />
+      <origin xyz="0.15 0.0 0.35" rpy="-1.57 0.0 0.0" />
       <axis xyz="0 0 1" />
       <calibration rising="${arm_1_ref}"/>
@@ -27,4 +54,19 @@
     <link name="arm_1_link">
       <xacro:default_inertial/>
+      <visual>
+        <origin xyz="0.125 0.0 0.0" rpy="0.0 1.57 0.0" />
+        <geometry>
+          <cylinder radius="0.025" length="0.25"/>
+        </geometry>
+        <material name="LightGrey">
+          <color rgba="0.7 0.7 0.7 1.0"/>
+        </material>
+      </visual>
+      <collision>
+        <origin xyz="0.125 0.0 0.0" rpy="0.0 1.57 0.0" />
+        <geometry>
+          <cylinder radius="0.025" length="0.25"/>
+        </geometry>
+      </collision>
     </link>
     <joint name="arm_2_joint" type="revolute">
@@ -40,5 +82,5 @@
       <visual>
         <geometry>
-          <box size="0.01 0.01 0.01"/>
+          <cylinder radius="0.03" length="0.05"/>
         </geometry>
         <material name="LightGrey">
@@ -63,14 +105,16 @@
       <xacro:default_inertial/>
       <visual>
-        <geometry>
-          <box size="0.01 0.01 0.01"/>
-        </geometry>
-        <material name="LightGrey">
-          <color rgba="0.7 0.7 0.7 1.0"/>
-        </material>
-      </visual>
-      <collision>
-        <geometry>
-          <box size="0.01 0.01 0.01"/>
+        <origin xyz="0.0 0.0 0.125" rpy="0.0 0.0 0.0" />
+        <geometry>
+          <cylinder radius="0.025" length="0.25"/>
+        </geometry>
+        <material name="LightGrey">
+          <color rgba="0.7 0.7 0.7 1.0"/>
+        </material>
+      </visual>
+      <collision>
+        <origin xyz="0.0 0.0 0.125" rpy="0.0 0.0 0.0" />
+        <geometry>
+          <cylinder radius="0.025" length="0.25"/>
         </geometry>
       </collision>
@@ -88,5 +132,5 @@
       <visual>
         <geometry>
-          <box size="0.01 0.01 0.01"/>
+          <cylinder radius="0.03" length="0.05"/>
         </geometry>
         <material name="LightGrey">
@@ -111,14 +155,16 @@
       <xacro:default_inertial/>
       <visual>
-        <geometry>
-          <box size="0.01 0.01 0.01"/>
-        </geometry>
-        <material name="LightGrey">
-          <color rgba="0.7 0.7 0.7 1.0"/>
-        </material>
-      </visual>
-      <collision>
-        <geometry>
-          <box size="0.01 0.01 0.01"/>
+        <origin xyz="0.0 0.0 0.0375" rpy="0.0 0.0 0.0" />
+        <geometry>
+          <cylinder radius="0.025" length="0.075"/>
+        </geometry>
+        <material name="LightGrey">
+          <color rgba="0.7 0.7 0.7 1.0"/>
+        </material>
+      </visual>
+      <collision>
+        <origin xyz="0.0 0.0 0.0375" rpy="0.0 0.0 0.0" />
+        <geometry>
+          <cylinder radius="0.025" length="0.075"/>
         </geometry>
       </collision>
@@ -136,16 +182,23 @@
       <visual>
         <geometry>
+          <cylinder radius="0.025" length="0.025"/>
+        </geometry>
+        <material name="LightGrey">
+          <color rgba="0.7 0.7 0.7 1.0"/>
+        </material>
+      </visual>
+      <collision>
+        <geometry>
           <box size="0.01 0.01 0.01"/>
         </geometry>
-        <material name="LightGrey">
-          <color rgba="0.7 0.7 0.7 1.0"/>
-        </material>
-      </visual>
-      <collision>
-        <geometry>
-          <box size="0.01 0.01 0.01"/>
-        </geometry>
-      </collision>
-    </link>
+      </collision>
+    </link>
+    <xacro:arm_SimpleTransmission number="1"></xacro:arm_SimpleTransmission>
+    <xacro:arm_SimpleTransmission number="2"></xacro:arm_SimpleTransmission>
+    <xacro:arm_SimpleTransmission number="3"></xacro:arm_SimpleTransmission>
+    <xacro:arm_SimpleTransmission number="4"></xacro:arm_SimpleTransmission>
+    <xacro:arm_SimpleTransmission number="5"></xacro:arm_SimpleTransmission>
+    <xacro:arm_SimpleTransmission number="6"></xacro:arm_SimpleTransmission>
+    <xacro:arm_SimpleTransmission number="7"></xacro:arm_SimpleTransmission>
   </xacro:macro>
 </robot>
