Commit message: package restructuration

File: robotino_bringup/robots/robotino/urdf/robotino.urdf.xacro (robot description, xacro)
@@ -2,5 +2,5 @@
 <robot xmlns:xacro="http://www.ros.org/wiki/xacro"
   name="robotino">
-  <xacro:include filename="$(find robotino_description)/urdf/properties.urdf.xacro" />
+  <xacro:include filename="$(find robotino_bringup)/robots/robotino/urdf/properties.urdf.xacro" />
   <xacro:include filename="$(find robotino_description)/urdf/gazebo.urdf.xacro" />
   <xacro:include filename="$(find robotino_description)/urdf/robotino_body.urdf.xacro" />
@@ -11,19 +11,7 @@
   <xacro:include filename="$(find robotino_description)/urdf/tilt_axis.urdf.xacro" />
   <xacro:body name="base"/>
-  <!--gazebo>
-    <plugin name="ros_control" filename="libmulti_hw_interface_gazebo_ros_control.so">
-      <robotNamespace>base_controller</robotNamespace>
-      <filterJointsParam>joint_names</filterJointsParam>
-    </plugin>
-  </gazebo-->
   <hokuyo name="hokuyo" parent="base_link">
     <origin xyz="${hokuyo_x} ${hokuyo_y} ${hokuyo_z}" rpy="${hokuyo_roll} ${hokuyo_pitch} ${hokuyo_yaw}"/>
   </hokuyo>
-  <!--kinect name="kinect" parent="base_link">
-    <origin xyz="${kinect_x} ${kinect_y} ${kinect_z}" rpy="${kinect_roll} ${kinect_pitch} ${kinect_yaw}"/>
-  </kinect-->
-  <!--anglebracketusb name="anglebracketusb" parent="base_link">
-    <origin xyz="${anglebracketusb_x} ${anglebracketusb_y} ${anglebracketusb_z}" rpy="${anglebracketusb_roll} ${anglebracketusb_pitch} ${anglebracketusb_yaw}"/>
-  </anglebracketusb-->
   <tilt_axis name="tilt" parent="base_link">
     <origin xyz="${tilt_x} ${tilt_y} ${tilt_z}" rpy="${tilt_roll} ${tilt_pitch} ${tilt_yaw}"/>
@@ -32,12 +20,12 @@
     <origin xyz="${kinect_x} ${kinect_y} ${kinect_z}" rpy="${kinect_roll} ${kinect_pitch} ${kinect_yaw}"/>
   </kinect>
+  <!--anglebracketusb name="anglebracketusb" parent="base_link">
+    <origin xyz="${anglebracketusb_x} ${anglebracketusb_y} ${anglebracketusb_z}" rpy="${anglebracketusb_roll} ${anglebracketusb_pitch} ${anglebracketusb_yaw}"/>
+  </anglebracketusb-->
   <gazebo>
-    <plugin name="ros_control" filename="libgazebo_ros_control.so">
+    <plugin name="ros_control" filename="libmulti_hw_interface_gazebo_ros_control.so">
       <robotNamespace>tilt_controller</robotNamespace>
       <filterJointsParam>joint_names</filterJointsParam>
     </plugin>
   </gazebo>
-  <!--anglebracketusb name="anglebracketusb" parent="base_link">
-      <origin xyz="${anglebracketusb_x} ${anglebracketusb_y} ${anglebracketusb_z}" rpy="${anglebracketusb_roll} ${anglebracketusb_pitch} ${anglebracketusb_yaw}"/>
-  </anglebracketusb-->
 </robot>

Commit message: robotino_arm packages integration

File: robotino_bringup/robots/robotino/urdf/robotino.urdf.xacro (robot description, xacro)
@@ -1,5 +1,5 @@
 <?xml version="1.0"?>
 <robot xmlns:xacro="http://www.ros.org/wiki/xacro"
-  name="robotino">
+  name="robot">
   <xacro:include filename="$(find robotino_bringup)/robots/robotino/urdf/properties.urdf.xacro" />
   <xacro:include filename="$(find robotino_description)/urdf/gazebo.urdf.xacro" />
@@ -10,5 +10,5 @@
   <xacro:include filename="$(find robotino_description)/urdf/kinect.urdf.xacro" />
   <xacro:include filename="$(find robotino_description)/urdf/tilt_axis.urdf.xacro" />
-  <xacro:include filename="$(find robotino_description)/urdf/arm.urdf.xacro" />
+  <xacro:include filename="$(find robotino_arm_description)/xacro/arm_model.urdf.xacro" />
   <xacro:body name="base"/>
   <hokuyo name="hokuyo" parent="base_link">
@@ -21,7 +21,18 @@
     <origin xyz="${kinect_x} ${kinect_y} ${kinect_z}" rpy="${kinect_roll} ${kinect_pitch} ${kinect_yaw}"/>
   </kinect-->
-  <arm parent="base_link">
+  <joint name="fixed_base_link_base" type="fixed">
+      <parent link="base_link"/>
+      <child link="base"/>
+      <origin xyz="0.0 0.0 0.185" rpy="0 0 -1.0471975511965976" />
+  </joint>
+  <link name="odomp"/>
+  <joint name="rotatory" type="fixed">
+    <parent link="odomp"/>
+    <child link="base_link"/>
+  </joint>
+  <xacro:arm />
+  <!--arm parent="base_link">
     <origin xyz="${arm_x} ${arm_y} ${arm_z}" rpy="${arm_roll} ${arm_pitch} ${arm_yaw}"/>
-  </arm>
+  </arm-->
   <gazebo>
     <plugin name="ros_control" filename="libhwi_switch_gazebo_ros_control.so">

Commit message: added hand to the robotino

File: robotino_bringup/robots/robotino/urdf/robotino.urdf.xacro (robot description, xacro)
@@ -11,14 +11,9 @@
   <xacro:include filename="$(find robotino_description)/urdf/tilt_axis.urdf.xacro" />
   <xacro:include filename="$(find robotino_arm_description)/xacro/arm_model.urdf.xacro" />
+  <xacro:include filename="$(find kclhand_description)/urdf/kclhand.urdf.xacro" />
   <xacro:body name="base"/>
   <hokuyo name="hokuyo" parent="base_link">
     <origin xyz="${hokuyo_x} ${hokuyo_y} ${hokuyo_z}" rpy="${hokuyo_roll} ${hokuyo_pitch} ${hokuyo_yaw}"/>
   </hokuyo>
-  <!--tilt_axis name="tilt" parent="base_link">
-    <origin xyz="${tilt_x} ${tilt_y} ${tilt_z}" rpy="${tilt_roll} ${tilt_pitch} ${tilt_yaw}"/>
-  </tilt_axis>
-  <kinect name="kinect" parent="tilt_link">
-    <origin xyz="${kinect_x} ${kinect_y} ${kinect_z}" rpy="${kinect_roll} ${kinect_pitch} ${kinect_yaw}"/>
-  </kinect-->
   <joint name="fixed_base_link_base" type="fixed">
       <parent link="base_link"/>
@@ -32,7 +27,4 @@
   </joint>
   <xacro:arm />
-  <!--arm parent="base_link">
-    <origin xyz="${arm_x} ${arm_y} ${arm_z}" rpy="${arm_roll} ${arm_pitch} ${arm_yaw}"/>
-  </arm-->
   <gazebo>
     <plugin name="ros_control" filename="libhwi_switch_gazebo_ros_control.so">
@@ -41,3 +33,13 @@
     </plugin>
   </gazebo>
+  <!-- hand -->
+  <xacro:kclhand name="hand" parent="link5">
+    <origin xyz="0 0 0.151" rpy="1.57 0 0" />
+  </xacro:kclhand>
+  <gazebo>
+    <plugin name="ros_control" filename="libhwi_switch_gazebo_ros_control.so">
+      <robotNamespace>hand_controller</robotNamespace>
+      <filterJointsParam>joint_names</filterJointsParam>
+    </plugin>
+  </gazebo>
 </robot>

Commit message: fixed hand position

File: robotino_bringup/robots/robotino/urdf/robotino.urdf.xacro (robot description, xacro)
@@ -35,5 +35,5 @@
   <!-- hand -->
   <xacro:kclhand name="hand" parent="link5">
-    <origin xyz="0 0 0.151" rpy="1.57 0 0" />
+    <origin xyz="0 0.02105 0.151" rpy="1.5707963 0 -1.04719755" />
   </xacro:kclhand>
   <gazebo>

Commit message: added wrist

File: robotino_bringup/robots/robotino/urdf/robotino.urdf.xacro (robot description, xacro)
@@ -35,5 +35,5 @@
   <!-- hand -->
   <xacro:kclhand name="hand" parent="link5">
-    <origin xyz="0 0.02105 0.151" rpy="1.5707963 0 -1.04719755" />
+    <origin xyz="0 0 0" rpy="1.5707963 0 0" />
   </xacro:kclhand>
   <gazebo>

Commit message: added frame odomp for the simulation

File: robotino_bringup/robots/robotino/urdf/robotino.urdf.xacro (robot description, xacro)
@@ -21,9 +21,9 @@
       <origin xyz="0.0 0.0 0.185" rpy="0 0 -1.0471975511965976" />
   </joint>
-  <link name="odomp"/>
+  <!--link name="odomp"/>
   <joint name="rotatory" type="fixed">
     <parent link="odomp"/>
     <child link="base_link"/>
-  </joint>
+  </joint-->
   <xacro:arm />
   <gazebo>
