Commit message: simulation integration

File: robotino_bringup/robots/uibk-robotino/urdf/robotino.urdf.xacro (robot description, xacro)
@@ -5,7 +5,5 @@
   <xacro:include filename="$(find robotino_description)/urdf/gazebo.urdf.xacro" />
   <xacro:include filename="$(find robotino_description)/urdf/robotino_body.urdf.xacro" />
-  <xacro:include filename="$(find robotino_description)/urdf/hokuyo.urdf.xacro" />
-  <xacro:include filename="$(find robotino_description)/urdf/camera.urdf.xacro" />
-  <xacro:include filename="$(find robotino_description)/urdf/angle_bracket.urdf.xacro" />
+  <xacro:include filename="$(find robotino_description)/urdf/hokuyo.urdf.xacro" />>
   <xacro:include filename="$(find robotino_description)/urdf/kinect.urdf.xacro" />
   <xacro:include filename="$(find robotino_description)/urdf/pan_tilt_axis.urdf.xacro" />
@@ -17,15 +15,12 @@
     <origin xyz="${pan_tilt_x} ${pan_tilt_y} ${pan_tilt_z}" rpy="${pan_tilt_roll} ${pan_tilt_pitch} ${pan_tilt_yaw}"/>
   </pan_tilt_axis>
+  <gazebo>
+    <plugin name="ros_control" filename="libhwi_switch_gazebo_ros_control.so">
+      <robotNamespace>pan_tilt_controller</robotNamespace>
+      <filterJointsParam>joint_names</filterJointsParam>
+    </plugin>
+  </gazebo>
   <kinect name="kinect" parent="tilt_link">
     <origin xyz="${kinect_x} ${kinect_y} ${kinect_z}" rpy="${kinect_roll} ${kinect_pitch} ${kinect_yaw}"/>
   </kinect>
-  <!--anglebracketusb name="anglebracketusb" parent="base_link">
-    <origin xyz="${anglebracketusb_x} ${anglebracketusb_y} ${anglebracketusb_z}" rpy="${anglebracketusb_roll} ${anglebracketusb_pitch} ${anglebracketusb_yaw}"/>
-  </anglebracketusb-->
-  <gazebo>
-    <plugin name="ros_control" filename="libhwi_switch_gazebo_ros_control.so">
-      <robotNamespace>tilt_controller</robotNamespace>
-      <filterJointsParam>joint_names</filterJointsParam>
-    </plugin>
-  </gazebo>
 </robot>
