Commit message: created a new pan-tilt link

File: robotino_bringup/robots/uibk-robotino/urdf/properties.urdf.xacro (robot description, xacro)
@@ -28,17 +28,17 @@
   <property name="hokuyo_pitch" value="0.0"/>
   <property name="hokuyo_yaw" value="0.0"/>
-   <!-- tilt mount positions | handeye calibration | relative to base_link -->
-  <property name="tilt_x" value="-0.01"/>
-  <property name="tilt_y" value="0.0"/>
-  <property name="tilt_z" value="0.45"/>
-  <property name="tilt_roll" value="-0.05"/>
-  <property name="tilt_pitch" value="${M_PI/2}"/>
-  <property name="tilt_yaw" value="0"/>
-  <!-- kinect mount positions | handeye calibration | relative to tilt_link -->
-  <property name="kinect_x" value="-0.03"/>
-  <property name="kinect_y" value="0.0"/>
+   <!-- pan_tilt mount positions | handeye calibration | relative to base_link -->
+  <property name="pan_tilt_x" value="0.25"/>
+  <property name="pan_tilt_y" value="0.0"/>
+  <property name="pan_tilt_z" value="0.5"/>
+  <property name="pan_tilt_roll" value="0"/>
+  <property name="pan_tilt_pitch" value="0"/>
+  <property name="pan_tilt_yaw" value="0"/>
+  <!-- kinect mount positions | handeye calibration | relative to pan_tilt_link -->
+  <property name="kinect_x" value="0.0"/>
+  <property name="kinect_y" value="0.03"/>
   <property name="kinect_z" value="0.0"/>
-  <property name="kinect_roll" value="-0.02"/>
-  <property name="kinect_pitch" value="-1.45"/>
+  <property name="kinect_roll" value="-1.57"/>
+  <property name="kinect_pitch" value="0"/>
   <property name="kinect_yaw" value="0.0"/>
   <!-- anglebracketusb mount positions | handeye calibration | relative to base_link -->

File: robotino_bringup/robots/uibk-robotino/urdf/robotino.urdf.xacro (robot description, xacro)
@@ -2,5 +2,5 @@
 <robot xmlns:xacro="http://www.ros.org/wiki/xacro"
   name="robotino">
-  <xacro:include filename="$(find robotino_bringup)/robots/robotino/urdf/properties.urdf.xacro" />
+  <xacro:include filename="$(find robotino_bringup)/robots/uibk-robotino/urdf/properties.urdf.xacro" />
   <xacro:include filename="$(find robotino_description)/urdf/gazebo.urdf.xacro" />
   <xacro:include filename="$(find robotino_description)/urdf/robotino_body.urdf.xacro" />
@@ -9,12 +9,12 @@
   <xacro:include filename="$(find robotino_description)/urdf/angle_bracket.urdf.xacro" />
   <xacro:include filename="$(find robotino_description)/urdf/kinect.urdf.xacro" />
-  <xacro:include filename="$(find robotino_description)/urdf/tilt_axis.urdf.xacro" />
+  <xacro:include filename="$(find robotino_description)/urdf/pan_tilt_axis.urdf.xacro" />
   <xacro:body name="base"/>
   <hokuyo name="hokuyo" parent="base_link">
     <origin xyz="${hokuyo_x} ${hokuyo_y} ${hokuyo_z}" rpy="${hokuyo_roll} ${hokuyo_pitch} ${hokuyo_yaw}"/>
   </hokuyo>
-  <tilt_axis name="tilt" parent="base_link">
-    <origin xyz="${tilt_x} ${tilt_y} ${tilt_z}" rpy="${tilt_roll} ${tilt_pitch} ${tilt_yaw}"/>
-  </tilt_axis>
+  <pan_tilt_axis parent="base_link">
+    <origin xyz="${pan_tilt_x} ${pan_tilt_y} ${pan_tilt_z}" rpy="${pan_tilt_roll} ${pan_tilt_pitch} ${pan_tilt_yaw}"/>
+  </pan_tilt_axis>
   <kinect name="kinect" parent="tilt_link">
     <origin xyz="${kinect_x} ${kinect_y} ${kinect_z}" rpy="${kinect_roll} ${kinect_pitch} ${kinect_yaw}"/>

Commit message: robot test

File: robotino_bringup/robots/uibk-robotino/urdf/properties.urdf.xacro (robot description, xacro)
@@ -24,5 +24,5 @@
   <property name="hokuyo_x" value="0.131740483"/>
   <property name="hokuyo_y" value="0.00937244242"/>
-  <property name="hokuyo_z" value="0.5"/> <!-- not used, apprx -->
+  <property name="hokuyo_z" value="0.05"/> <!-- not used, apprx -->
   <property name="hokuyo_roll" value="0.0"/>
   <property name="hokuyo_pitch" value="0.0"/>

File: robotino_description/urdf/pan_tilt_axis.urdf.xacro (robot description, xacro)
@@ -23,5 +23,5 @@
       <parent link="pan_link"/>
       <child link="tilt_link" />
-      <axis xyz="0 0 1" />
+      <axis xyz="0 0 -1" />
       <calibration rising="0.1"/>
       <limit effort="100" lower="-1.57" upper="1.57" velocity="1.4"/>
