Commit message: updated model

File: robotino_bringup/robots/robotinoSH/urdf/robotino_simple.urdf.xacro (robot description, xacro)
@@ -13,7 +13,7 @@
   <xacro:include filename="$(find robotino_description)/urdf/soft_hand_simple.urdf.xacro" />
   <xacro:body name="base"/>
-  <hokuyo name="hokuyo" parent="base_link">
+  <!--hokuyo name="hokuyo" parent="base_link">
     <origin xyz="${hokuyo_x} ${hokuyo_y} ${hokuyo_z}" rpy="${hokuyo_roll} ${hokuyo_pitch} ${hokuyo_yaw}"/>
-  </hokuyo>
+  </hokuyo-->
   <joint name="fixed_base_link_base" type="fixed">
       <parent link="base_link"/>
@@ -22,7 +22,8 @@
   </joint>
   <link name="odomp"/>
-  <joint name="rotatory" type="fixed">
+  <joint name="rotatory" type="continuous">
     <parent link="odomp"/>
     <child link="base_link"/>
+    <axis xyz="0 0 1" />
   </joint>
   <xacro:arm />

File: robotino_description/urdf/robotino_simple_body.urdf.xacro (robot description, xacro)
@@ -17,13 +17,15 @@
       </inertial>
       <visual>
-        <origin xyz="0 0 0.12" rpy="0 0 0"/>
+        <origin xyz="0 0 0" rpy="0 0 0"/>
         <geometry>
-          <cylinder length="0.24" radius="0.23"/>
+          <mesh filename="package://robotino_description/meshes/RobotinoBody.dae"/>
+          <!--cylinder length="0.24" radius="0.23"/-->
         </geometry>
       </visual>
       <collision>
-        <origin xyz="0 0 0.12" rpy="0 0 0"/>
+        <origin xyz="0 0 0" rpy="0 0 0"/>
         <geometry>
-          <cylinder length="0.24" radius="0.23"/>
+          <mesh filename="package://robotino_description/meshes/RobotinoBody.dae"/>
+          <!--cylinder length="0.24" radius="0.23"/-->
         </geometry>
       </collision>
