Commit message: moveit 6dof working!

File: robotino_bringup/robots/robotino_6dof/urdf/robotino.urdf.xacro (robot description, xacro)
@@ -4,4 +4,5 @@
   <xacro:include filename="$(find robotino_bringup)/robots/robotino/urdf/properties.urdf.xacro" />
   <xacro:include filename="$(find robotino_description)/urdf/robotino_body.urdf.xacro" />
+  <xacro:include filename="$(find robotino_description)/urdf/rotatory.urdf.xacro" />
   <xacro:include filename="$(find robotino_description)/urdf/hokuyo.urdf.xacro" />
   <xacro:include filename="$(find robotino_description)/urdf/kinect.urdf.xacro" />
@@ -17,9 +18,11 @@
     <origin xyz="${hokuyo_x} ${hokuyo_y} ${hokuyo_z}" rpy="${hokuyo_roll} ${hokuyo_pitch} ${hokuyo_yaw}"/>
   </hokuyo>
-  <joint name="fixed_base_link_base" type="fixed">
-      <parent link="base_link"/>
-      <child link="base"/>
-      <origin xyz="0.0 0.0 0.185" rpy="0 0 -1.0471975511965976" />
-  </joint>
+  <xacro:rotatory />
+  <gazebo>
+    <plugin name="ros_control" filename="libhwi_switch_gazebo_ros_control.so">
+      <robotNamespace>rotatory_controller</robotNamespace>
+      <filterJointsParam>joint_names</filterJointsParam>
+    </plugin>
+  </gazebo>
   <xacro:arm />
   <gazebo>

File: robotino_description/urdf/robotino_body.urdf.xacro (robot description, xacro)
@@ -1,4 +1,5 @@
 <?xml version="1.0"?>
 <root xmlns:xacro="http://www.ros.org/wiki/xacro">
+  <xacro:include filename="$(find robotino_description)/urdf/gazebo.urdf.xacro" />
   <xacro:macro name="body" params="name">
 <!--<link name="${name}_footprint"/>
@@ -48,7 +49,4 @@
     <wheel_transmission name="wheel2" />
     <wheel_gazebo name="wheel2" />
-    <command_bridge name="command_bridge" parent="base_link">
-      <origin xyz="-0.05 0 0.13" rpy="0 0 ${M_PI/2}"/>
-    </command_bridge>
   </xacro:macro>
   <!-- WHEEL -->
@@ -95,26 +93,3 @@
     </transmission>
   </xacro:macro>
-  <!-- COMMAND BRIDGE -->
-  <xacro:macro name="command_bridge" params="parent name *origin">
-    <joint name="${name}_joint" type="fixed">
-      <insert_block name="origin" />
-      <parent link="${parent}"/>
-      <child link="${name}_link" />
-    </joint>
-    <link name="${name}_link">
-      <inertial>
-        <mass value="0.00001" />
-        <origin xyz="0 0 0" />
-        <inertia ixx="1.0" ixy="0.0" ixz="0.0"
-          iyy="1.0" iyz="0.0"
-          izz="1.0" />
-      </inertial>
-      <collision>
-        <origin xyz="0 0 0" rpy="0 0 0" />
-        <geometry>
-          <box size="0.25 0.11 0.16"/>
-        </geometry>
-      </collision>
-    </link>
-  </xacro:macro>
 </root>

File: robotino_description/urdf/robotino_simple_body.urdf.xacro (robot description, xacro)
@@ -49,8 +49,5 @@
     </wheel>
     <wheel_transmission name="wheel2" />
-    <wheel_gazebo name="wheel2" />
-    <command_bridge name="command_bridge" parent="base_link">
-      <origin xyz="-0.05 0 0.13" rpy="0 0 ${M_PI/2}"/>
-    </command_bridge-->
+    <wheel_gazebo name="wheel2" /-->
   </xacro:macro>
   <!-- WHEEL -->
@@ -97,26 +94,3 @@
     </transmission>
   </xacro:macro>
-  <!-- COMMAND BRIDGE -->
-  <xacro:macro name="command_bridge" params="parent name *origin">
-    <joint name="${name}_joint" type="fixed">
-      <insert_block name="origin" />
-      <parent link="${parent}"/>
-      <child link="${name}_link" />
-    </joint>
-    <link name="${name}_link">
-      <inertial>
-        <mass value="0.00001" />
-        <origin xyz="0 0 0" />
-        <inertia ixx="1.0" ixy="0.0" ixz="0.0"
-          iyy="1.0" iyz="0.0"
-          izz="1.0" />
-      </inertial>
-      <collision>
-        <origin xyz="0 0 0" rpy="0 0 0" />
-        <geometry>
-          <box size="0.25 0.11 0.16"/>
-        </geometry>
-      </collision>
-    </link>
-  </xacro:macro>
 </root>
