Commit message: added pan unit in robot configuration files

File: robotino_bringup/robots/tuw-robotino/urdf/properties.urdf.xacro (robot description, xacro)
@@ -13,5 +13,5 @@
   <property name="KINECT_LENGTH" value="0.18"/>
   <property name="KINECT_WIDTH" value="0.035"/>
-  <property name="KINECT_HEIGHT" value="0.05"/>
+  <property name="KINECT_HEIGHT" value="0.02"/>
   <!-- camera mount positions | handeye calibration | relative to base_link -->
   <property name="camera_x" value="0.0"/>
@@ -28,17 +28,17 @@
   <property name="hokuyo_pitch" value="0.0"/>
   <property name="hokuyo_yaw" value="0.0"/>
-   <!-- tilt mount positions | handeye calibration | relative to base_link -->
-  <property name="tilt_x" value="0.02"/>
-  <property name="tilt_y" value="0.0"/>
-  <property name="tilt_z" value="0.675"/>
-  <property name="tilt_roll" value="-0.05"/>
-  <property name="tilt_pitch" value="${M_PI/2}"/>
-  <property name="tilt_yaw" value="0"/>
-  <!-- kinect mount positions | handeye calibration | relative to tilt_link -->
-  <property name="kinect_x" value="-0.03"/>
-  <property name="kinect_y" value="0.0"/>
-  <property name="kinect_z" value="0.053"/>
-  <property name="kinect_roll" value="-0.02"/>
-  <property name="kinect_pitch" value="-1.45"/>
+   <!-- pan_tilt mount positions | handeye calibration | relative to base_link -->
+  <property name="pan_tilt_x" value="0.03"/>
+  <property name="pan_tilt_y" value="0.03"/>
+  <property name="pan_tilt_z" value="0.64"/>
+  <property name="pan_tilt_roll" value="0"/>
+  <property name="pan_tilt_pitch" value="0"/> <!--${M_PI/2}"/> -->
+  <property name="pan_tilt_yaw" value="0"/>
+  <!-- kinect mount positions | handeye calibration | relative to pan_tilt_link -->
+  <property name="kinect_x" value="0.0"/>
+  <property name="kinect_y" value="0.065"/>
+  <property name="kinect_z" value="0.0"/>
+  <property name="kinect_roll" value="-${M_PI/2}"/>
+  <property name="kinect_pitch" value="0"/>
   <property name="kinect_yaw" value="0.0"/>
   <!-- anglebracketusb mount positions | handeye calibration | relative to base_link -->

File: robotino_bringup/robots/tuw-robotino/urdf/robotino.urdf.xacro (robot description, xacro)
@@ -9,5 +9,5 @@
   <xacro:include filename="$(find robotino_description)/urdf/angle_bracket.urdf.xacro" />
   <xacro:include filename="$(find robotino_description)/urdf/kinect.urdf.xacro" />
-  <xacro:include filename="$(find robotino_description)/urdf/tilt_axis.urdf.xacro" />
+  <xacro:include filename="$(find robotino_description)/urdf/pan_tilt_axis.urdf.xacro" />
   <xacro:body name="base"/>
   <hokuyo name="hokuyo" parent="base_link">
@@ -20,7 +20,7 @@
     <origin xyz="${anglebracketusb_x} ${anglebracketusb_y} ${anglebracketusb_z}" rpy="${anglebracketusb_roll} ${anglebracketusb_pitch} ${anglebracketusb_yaw}"/>
   </anglebracketusb-->
-  <tilt_axis name="tilt" parent="base_link">
-    <origin xyz="${tilt_x} ${tilt_y} ${tilt_z}" rpy="${tilt_roll} ${tilt_pitch} ${tilt_yaw}"/>
-  </tilt_axis>
+  <pan_tilt_axis parent="base_link">
+    <origin xyz="${pan_tilt_x} ${pan_tilt_y} ${pan_tilt_z}" rpy="${pan_tilt_roll} ${pan_tilt_pitch} ${pan_tilt_yaw}"/>
+  </pan_tilt_axis>
   <kinect name="kinect" parent="tilt_link">
     <origin xyz="${kinect_x} ${kinect_y} ${kinect_z}" rpy="${kinect_roll} ${kinect_pitch} ${kinect_yaw}"/>
@@ -28,5 +28,5 @@
   <gazebo>
     <plugin name="ros_control" filename="libhwi_switch_gazebo_ros_control.so">
-      <robotNamespace>tilt_controller</robotNamespace>
+      <robotNamespace>pan_tilt_controller</robotNamespace>
       <filterJointsParam>joint_names</filterJointsParam>
     </plugin>

Commit message: calibration try

File: robotino_bringup/robots/tuw-robotino/urdf/properties.urdf.xacro (robot description, xacro)
@@ -22,23 +22,47 @@
   <property name="camera_yaw" value="-${M_PI/2}"/>
   <!-- hokuyo mount positions | relative to base_link -->
-  <property name="hokuyo_x" value="0.0757694625"/>
-  <property name="hokuyo_y" value="0.0105994255"/>
-  <property name="hokuyo_z" value="0.25"/>
+  <property name="hokuyo_x" value="0.184"/>
+  <property name="hokuyo_y" value="0.004"/>
+  <property name="hokuyo_z" value="0.16"/>
   <property name="hokuyo_roll" value="0.0"/>
   <property name="hokuyo_pitch" value="0.0"/>
-  <property name="hokuyo_yaw" value="0.0031523481"/>
-   <!-- pan_tilt mount positions | handeye calibration | relative to base_link -->
-  <property name="pan_tilt_x" value="0.03"/>
-  <property name="pan_tilt_y" value="0.03"/>
+  <property name="hokuyo_yaw" value="-0.015"/>
+  <!-- pan_tilt mount positions | handeye calibration | relative to base_pan_link -->
+  <property name="pan_tilt_x" value="0.145"/>
+  <property name="pan_tilt_y" value="0.194"/>
   <property name="pan_tilt_z" value="0.64"/>
-  <property name="pan_tilt_roll" value="0"/>
-  <property name="pan_tilt_pitch" value="0"/> <!--${M_PI/2}"/> -->
-  <property name="pan_tilt_yaw" value="0"/>
-  <!-- kinect mount positions | handeye calibration | relative to pan_tilt_link -->
-  <property name="kinect_x" value="0.0"/>
-  <property name="kinect_y" value="0.065"/>
-  <property name="kinect_z" value="0.0"/>
-  <property name="kinect_roll" value="-${M_PI/2}"/>
-  <property name="kinect_pitch" value="0"/>
+  <property name="pan_tilt_roll" value="0.0"/>
+  <property name="pan_tilt_pitch" value="0.0"/>
+  <property name="pan_tilt_yaw" value="1.0472"/>
+  <!-- <property name="pan_tilt_x" value="0.163"/> -->
+  <!-- <property name="pan_tilt_y" value="0.125"/> -->
+  <!-- <property name="pan_tilt_z" value="0.573"/> -->
+  <!-- <property name="pan_tilt_roll" value="0.0"/> -->
+  <!-- <property name="pan_tilt_pitch" value="0.0"/> -->
+  <!-- <property name="pan_tilt_yaw" value="1.0472"/> -->
+  <!-- <property name="pan_tilt_x" value="0.157"/> -->
+  <!-- <property name="pan_tilt_y" value="0.17"/> -->
+  <!-- <property name="pan_tilt_z" value="0.64"/> -->
+  <!-- <property name="pan_tilt_roll" value="0.030897"/> -->
+  <!-- <property name="pan_tilt_pitch" value="0.0174498"/>  -->
+  <!-- <property name="pan_tilt_yaw" value="1.11926"/> -->
+  <!-- kinect mount positions | handeye calibration | relative to tilt_link -->
+  <!-- <property name="kinect_x" value="0.03129"/> -->
+  <!-- <property name="kinect_y" value="0.0579456"/> -->
+  <!-- <property name="kinect_z" value="0.000183902"/> -->
+  <!-- <property name="kinect_roll" value="-1.56905"/> -->
+  <!-- <property name="kinect_pitch" value="0.00434565"/> -->
+  <!-- <property name="kinect_yaw" value="0.00667917"/> -->
+  <!-- <property name="kinect_x" value="0.05"/> -->
+  <!-- <property name="kinect_y" value="0.14"/> -->
+  <!-- <property name="kinect_z" value="-0.05"/> -->
+  <!-- <property name="kinect_roll" value="-1.5707963268"/> -->
+  <!-- <property name="kinect_pitch" value="0.0628318530718"/> -->
+  <!-- <property name="kinect_yaw" value="-0.025"/> -->
+  <property name="kinect_x" value="0.1"/>
+  <property name="kinect_y" value="0.0"/>
+  <property name="kinect_z" value="-0.0"/>
+  <property name="kinect_roll" value="-1.5707963268"/>
+  <property name="kinect_pitch" value="0.075"/>
   <property name="kinect_yaw" value="0.0"/>
   <!-- anglebracketusb mount positions | handeye calibration | relative to base_link -->

File: robotino_bringup/robots/tuw-robotino2/urdf/properties.urdf.xacro (robot description, xacro)
@@ -22,10 +22,16 @@
   <property name="camera_yaw" value="-${M_PI/2}"/>
   <!-- hokuyo mount positions | relative to base_link -->
-  <property name="hokuyo_x" value="0.064"/>
-  <property name="hokuyo_y" value="0.0"/>
-  <property name="hokuyo_z" value="0.22"/>
+  <!-- <property name="hokuyo_x" value="0.064"/> -->
+  <!-- <property name="hokuyo_y" value="0.0"/> -->
+  <!-- <property name="hokuyo_z" value="0.22"/> -->
+  <!-- <property name="hokuyo_roll" value="0.0"/> -->
+  <!-- <property name="hokuyo_pitch" value="0.0"/> -->
+  <!-- <property name="hokuyo_yaw" value="0.0"/> -->
+  <property name="hokuyo_x" value="0.184"/>
+  <property name="hokuyo_y" value="0.004"/>
+  <property name="hokuyo_z" value="0.16"/>
   <property name="hokuyo_roll" value="0.0"/>
   <property name="hokuyo_pitch" value="0.0"/>
-  <property name="hokuyo_yaw" value="0.0"/>
+  <property name="hokuyo_yaw" value="-0.015"/>
    <!-- pan_tilt mount positions | handeye calibration | relative to base_link -->
   <property name="pan_tilt_x" value="0.203"/>

File: robotino_description/urdf/pan_tilt_axis.urdf.xacro (robot description, xacro)
@@ -2,10 +2,10 @@
 <root xmlns:xacro="http://www.ros.org/wiki/xacro">
   <xacro:macro name="pan_tilt_axis" params="parent *origin">
-    <joint name="base_pan_joint" type="fixed">
+    <joint name="profile_joint" type="fixed">
 			<origin xyz="0 0 0" rpy="0 0 0"/>
       <parent link="${parent}"/>
-      <child link="base_pan_link" />
+      <child link="profile_link" />
     </joint>
-    <link name="base_pan_link">
+    <link name="profile_link">
       <inertial>
         <mass value="0.00001" />
@@ -29,11 +29,18 @@
       </collision>
     </link>
-    <gazebo reference="base_pan_link">
+    <gazebo reference="profile_link">
       <gravity>true</gravity>
       <self_collide>false</self_collide>
       <material>Gazebo/Black</material>
     </gazebo>
+    <joint name="base_pan_joint" type="fixed">
+      <insert_block name="origin" />
+      <parent link="profile_link"/>
+      <child link="base_pan_link" />
+    </joint>
+    <link name="base_pan_link">
+    </link>
     <joint name="pan_joint" type="revolute">
-      <insert_block name="origin" />
+      <origin xyz="0 0 0" rpy="0 0 0"/>
       <parent link="base_pan_link"/>
       <child link="pan_link" />

Commit message: new pan tilt prrofile for tuw

File: robotino_bringup/robots/tuw-robotino/urdf/properties.urdf.xacro (robot description, xacro)
@@ -22,30 +22,23 @@
   <property name="camera_yaw" value="-${M_PI/2}"/>
   <!-- hokuyo mount positions | relative to base_link -->
-  <property name="hokuyo_x" value="0.064"/>
-  <property name="hokuyo_y" value="0.0"/>
-  <property name="hokuyo_z" value="0.22"/>
+  <property name="hokuyo_x" value="0.184"/>
+  <property name="hokuyo_y" value="0.004"/>
+  <property name="hokuyo_z" value="0.16"/>
   <property name="hokuyo_roll" value="0.0"/>
   <property name="hokuyo_pitch" value="0.0"/>
-  <property name="hokuyo_yaw" value="0.0"/>
-   <!-- pan_tilt mount positions | handeye calibration | relative to base_link -->
-  <property name="pan_tilt_x" value="0.03"/>
-  <property name="pan_tilt_y" value="0.03"/>
+  <property name="hokuyo_yaw" value="-0.015"/>
+  <!-- pan_tilt mount positions | handeye calibration | relative to base_pan_link -->
+  <property name="pan_tilt_x" value="0.145"/>
+  <property name="pan_tilt_y" value="0.194"/>
   <property name="pan_tilt_z" value="0.64"/>
-  <property name="pan_tilt_roll" value="0"/>
-  <property name="pan_tilt_pitch" value="0"/> <!--${M_PI/2}"/> -->
-  <property name="pan_tilt_yaw" value="0"/>
+  <property name="pan_tilt_roll" value="0.0"/>
+  <property name="pan_tilt_pitch" value="0.0"/>
+  <property name="pan_tilt_yaw" value="1.0472"/>
   <!-- kinect mount positions | handeye calibration | relative to pan_tilt_link -->
-  <property name="kinect_x" value="0.0"/>
-  <property name="kinect_y" value="0.065"/>
-  <property name="kinect_z" value="0.0"/>
-  <property name="kinect_roll" value="-${M_PI/2}"/>
-  <property name="kinect_pitch" value="0"/>
+  <property name="kinect_x" value="0.1"/>
+  <property name="kinect_y" value="0.0"/>
+  <property name="kinect_z" value="-0.0"/>
+  <property name="kinect_roll" value="-1.5707963268"/>
+  <property name="kinect_pitch" value="0.075"/>
   <property name="kinect_yaw" value="0.0"/>
-  <!-- anglebracketusb mount positions | handeye calibration | relative to base_link -->
-  <property name="anglebracketusb_x" value="0.008"/>
-  <property name="anglebracketusb_y" value="0.0"/>
-  <property name="anglebracketusb_z" value="0.137"/>
-  <property name="anglebracketusb_roll" value="0.0"/>
-  <property name="anglebracketusb_pitch" value="0.0"/>
-  <property name="anglebracketusb_yaw" value="0.0"/>
 </robot>

File: robotino_bringup/robots/tuw-robotino/urdf/robotino.urdf.xacro (robot description, xacro)
@@ -7,6 +7,12 @@
   <xacro:include filename="$(find robotino_description)/urdf/hokuyo.urdf.xacro" />
   <xacro:include filename="$(find robotino_description)/urdf/kinect.urdf.xacro" />
-  <xacro:include filename="$(find robotino_description)/urdf/pan_tilt_axis.urdf.xacro" />
+  <xacro:include filename="$(find robotino_description)/urdf/pan_tilt_tuw_axis.urdf.xacro" />
   <xacro:body name="base"/>
+  <gazebo>
+    <plugin name="ros_control" filename="libhwi_switch_gazebo_ros_control.so">
+      <robotNamespace>base_controller</robotNamespace>
+      <filterJointsParam>joint_names</filterJointsParam>
+    </plugin>
+  </gazebo>
   <gazebo>
     <plugin name="ros_control" filename="libhwi_switch_gazebo_ros_control.so">

File: robotino_bringup/robots/tuw-robotino2/urdf/properties.urdf.xacro (robot description, xacro)
@@ -22,23 +22,23 @@
   <property name="camera_yaw" value="-${M_PI/2}"/>
   <!-- hokuyo mount positions | relative to base_link -->
-  <property name="hokuyo_x" value="0.064"/>
-  <property name="hokuyo_y" value="0.0"/>
-  <property name="hokuyo_z" value="0.22"/>
+  <property name="hokuyo_x" value="0.184"/>
+  <property name="hokuyo_y" value="0.004"/>
+  <property name="hokuyo_z" value="0.16"/>
   <property name="hokuyo_roll" value="0.0"/>
   <property name="hokuyo_pitch" value="0.0"/>
-  <property name="hokuyo_yaw" value="0.0"/>
-   <!-- pan_tilt mount positions | handeye calibration | relative to base_link -->
-  <property name="pan_tilt_x" value="0.203"/>
-  <property name="pan_tilt_y" value="0.003"/>
-  <property name="pan_tilt_z" value="0.55"/>
-  <property name="pan_tilt_roll" value="0"/>
-  <property name="pan_tilt_pitch" value="0"/> <!--${M_PI/2}"/> -->
-  <property name="pan_tilt_yaw" value="0.0"/>
+  <property name="hokuyo_yaw" value="-0.015"/>
+  <!-- pan_tilt mount positions | handeye calibration | relative to base_pan_link -->
+  <property name="pan_tilt_x" value="0.145"/>
+  <property name="pan_tilt_y" value="0.194"/>
+  <property name="pan_tilt_z" value="0.64"/>
+  <property name="pan_tilt_roll" value="0.0"/>
+  <property name="pan_tilt_pitch" value="0.0"/>
+  <property name="pan_tilt_yaw" value="1.0472"/>
   <!-- kinect mount positions | handeye calibration | relative to pan_tilt_link -->
-  <property name="kinect_x" value="0.0"/>
-  <property name="kinect_y" value="0.065"/>
-  <property name="kinect_z" value="0.0"/>
-  <property name="kinect_roll" value="-${M_PI/2}"/>
-  <property name="kinect_pitch" value="0"/>
+  <property name="kinect_x" value="0.1"/>
+  <property name="kinect_y" value="0.0"/>
+  <property name="kinect_z" value="-0.0"/>
+  <property name="kinect_roll" value="-1.5707963268"/>
+  <property name="kinect_pitch" value="0.075"/>
   <property name="kinect_yaw" value="0.0"/>
    <!-- arm mount positions | handeye calibration | relative to base_link -->

File: robotino_bringup/robots/tuw-robotino2/urdf/robotino.urdf.xacro (robot description, xacro)
@@ -8,5 +8,5 @@
   <xacro:include filename="$(find robotino_description)/urdf/hokuyo.urdf.xacro" />
   <xacro:include filename="$(find robotino_description)/urdf/kinect.urdf.xacro" />
-  <xacro:include filename="$(find robotino_description)/urdf/pan_tilt_axis.urdf.xacro" />
+  <xacro:include filename="$(find robotino_description)/urdf/pan_tilt_tuw_axis.urdf.xacro" />
   <xacro:include filename="$(find robotino_arm_description)/xacro/arm_model.urdf.xacro" />
   <xacro:include filename="$(find kclhand_description)/urdf/kclhand.urdf.xacro" />

File: robotino_description/urdf/pan_tilt_tuw_axis.urdf.xacro (robot description, xacro)
@@ -18,5 +18,5 @@
         <origin xyz="0 0 0" rpy="0 0 0" />
         <geometry>
-          <mesh filename="package://robotino_description/meshes/pan_tilt.stl"/>
+          <mesh filename="package://robotino_description/meshes/pan_tilt_tuw.stl"/>
         </geometry>
         <material name="Black"/>
@@ -25,5 +25,5 @@
         <origin xyz="0 0 0" rpy="0 0 0" />
         <geometry>
-          <mesh filename="package://robotino_description/meshes/pan_tilt.stl"/>
+          <mesh filename="package://robotino_description/meshes/pan_tilt_tuw.stl"/>
         </geometry>
       </collision>
