Commit message: new parameteres for odometry node

File: robotino_bringup/robots/alufr-robotino/urdf/properties.urdf.xacro (robot description, xacro)
@@ -29,5 +29,5 @@
   <property name="hokuyo_yaw" value="0.0"/>
    <!-- tilt mount positions | handeye calibration | relative to base_link -->
-  <property name="tilt_x" value="-0.01"/>
+  <property name="tilt_x" value="0.02"/>
   <property name="tilt_y" value="0.0"/>
   <property name="tilt_z" value="0.45"/>
@@ -35,19 +35,5 @@
   <property name="tilt_pitch" value="${M_PI/2}"/>
   <property name="tilt_yaw" value="0"/>
-   <!-- arm mount positions | handeye calibration | relative to base_link -->
-  <property name="arm_x" value="0.0"/>
-  <property name="arm_y" value="0.0"/>
-  <property name="arm_z" value="0.35"/>
-  <property name="arm_roll" value="0.0"/>
-  <property name="arm_pitch" value="0.0"/>
-  <property name="arm_yaw" value="0.0"/>
-   <!-- arm calibration-->
-  <property name="arm_1_ref" value="0.0"/>
-  <property name="arm_2_ref" value="0.0"/>
-  <property name="arm_3_ref" value="0.0"/>
-  <property name="arm_4_ref" value="0.0"/>
-  <property name="arm_5_ref" value="0.0"/>
-  <property name="arm_6_ref" value="0.0"/>
-   <!-- kinect mount positions | handeye calibration | relative to tilt_link -->
+  <!-- kinect mount positions | handeye calibration | relative to tilt_link -->
   <property name="kinect_x" value="-0.03"/>
   <property name="kinect_y" value="0.0"/>
@@ -56,5 +42,5 @@
   <property name="kinect_pitch" value="-1.45"/>
   <property name="kinect_yaw" value="0.0"/>
-   <!-- anglebracketusb mount positions | handeye calibration | relative to base_link -->
+  <!-- anglebracketusb mount positions | handeye calibration | relative to base_link -->
   <property name="anglebracketusb_x" value="0.008"/>
   <property name="anglebracketusb_y" value="0.0"/>

File: robotino_bringup/robots/alufr-robotino/urdf/robotino.urdf.xacro (robot description, xacro)
@@ -1,6 +1,6 @@
 <?xml version="1.0"?>
 <robot xmlns:xacro="http://www.ros.org/wiki/xacro"
-  name="robot">
-  <xacro:include filename="$(find robotino_bringup)/robots/robotino/urdf/properties.urdf.xacro" />
+  name="robotino">
+  <xacro:include filename="$(find robotino_bringup)/robots/alufr-robotino/urdf/properties.urdf.xacro" />
   <xacro:include filename="$(find robotino_description)/urdf/gazebo.urdf.xacro" />
   <xacro:include filename="$(find robotino_description)/urdf/robotino_body.urdf.xacro" />
@@ -10,32 +10,17 @@
   <xacro:include filename="$(find robotino_description)/urdf/kinect.urdf.xacro" />
   <xacro:include filename="$(find robotino_description)/urdf/tilt_axis.urdf.xacro" />
-  <xacro:include filename="$(find robotino_arm_description)/xacro/arm_model.urdf.xacro" />
   <xacro:body name="base"/>
   <hokuyo name="hokuyo" parent="base_link">
     <origin xyz="${hokuyo_x} ${hokuyo_y} ${hokuyo_z}" rpy="${hokuyo_roll} ${hokuyo_pitch} ${hokuyo_yaw}"/>
   </hokuyo>
-  <!--tilt_axis name="tilt" parent="base_link">
+  <tilt_axis name="tilt" parent="base_link">
     <origin xyz="${tilt_x} ${tilt_y} ${tilt_z}" rpy="${tilt_roll} ${tilt_pitch} ${tilt_yaw}"/>
   </tilt_axis>
   <kinect name="kinect" parent="tilt_link">
     <origin xyz="${kinect_x} ${kinect_y} ${kinect_z}" rpy="${kinect_roll} ${kinect_pitch} ${kinect_yaw}"/>
-  </kinect-->
-  <joint name="fixed_base_link_base" type="fixed">
-      <parent link="base_link"/>
-      <child link="base"/>
-      <origin xyz="0.0 0.0 0.185" rpy="0 0 -1.0471975511965976" />
-  </joint>
-  <link name="odomp"/>
-  <joint name="rotatory" type="fixed">
-    <parent link="odomp"/>
-    <child link="base_link"/>
-  </joint>
-  <xacro:arm />
-  <!--arm parent="base_link">
-    <origin xyz="${arm_x} ${arm_y} ${arm_z}" rpy="${arm_roll} ${arm_pitch} ${arm_yaw}"/>
-  </arm-->
+  </kinect>
   <gazebo>
     <plugin name="ros_control" filename="libhwi_switch_gazebo_ros_control.so">
-      <robotNamespace>arm_controller</robotNamespace>
+      <robotNamespace>tilt_controller</robotNamespace>
       <filterJointsParam>joint_names</filterJointsParam>
     </plugin>

Commit message: review alufr files

File: robotino_bringup/robots/alufr-robotino/urdf/properties.urdf.xacro (robot description, xacro)
@@ -14,11 +14,4 @@
   <property name="KINECT_WIDTH" value="0.035"/>
   <property name="KINECT_HEIGHT" value="0.02"/>
-  <!-- camera mount positions | handeye calibration | relative to base_link -->
-  <property name="camera_x" value="0.0"/>
-  <property name="camera_y" value="0.0"/>
-  <property name="camera_z" value="0.2"/>
-  <property name="camera_roll" value="0.0"/>
-  <property name="camera_pitch" value="0.0"/>
-  <property name="camera_yaw" value="-${M_PI/2}"/>
   <!-- hokuyo mount positions | relative to base_link -->
   <property name="hokuyo_x" value="0.064"/>
@@ -28,5 +21,5 @@
   <property name="hokuyo_pitch" value="0.0"/>
   <property name="hokuyo_yaw" value="0.0"/>
-   <!-- tilt mount positions | handeye calibration | relative to base_link -->
+  <!-- tilt mount positions | handeye calibration | relative to base_link -->
   <property name="tilt_x" value="0.02"/>
   <property name="tilt_y" value="0.0"/>
@@ -42,10 +35,17 @@
   <property name="kinect_pitch" value="-1.45"/>
   <property name="kinect_yaw" value="0.0"/>
-  <!-- anglebracketusb mount positions | handeye calibration | relative to base_link -->
-  <property name="anglebracketusb_x" value="0.008"/>
-  <property name="anglebracketusb_y" value="0.0"/>
-  <property name="anglebracketusb_z" value="0.137"/>
-  <property name="anglebracketusb_roll" value="0.0"/>
-  <property name="anglebracketusb_pitch" value="0.0"/>
-  <property name="anglebracketusb_yaw" value="0.0"/>
+   <!-- arm mount positions | handeye calibration | relative to base_link -->
+  <property name="arm_x" value="0.0"/>
+  <property name="arm_y" value="-0.01591"/>
+  <property name="arm_z" value="0.32"/>
+  <property name="arm_roll" value="0.0"/>
+  <property name="arm_pitch" value="0.0"/>
+  <property name="arm_yaw" value="-1"/>
+   <!-- arm calibration-->
+  <property name="arm_1_ref" value="0.0"/>
+  <property name="arm_2_ref" value="0.0"/>
+  <property name="arm_3_ref" value="0.0"/>
+  <property name="arm_4_ref" value="0.0"/>
+  <property name="arm_5_ref" value="0.0"/>
+  <property name="arm_6_ref" value="0.0"/>
 </robot>

File: robotino_bringup/robots/alufr-robotino/urdf/robotino.urdf.xacro (robot description, xacro)
@@ -1,12 +1,13 @@
 <?xml version="1.0"?>
 <robot xmlns:xacro="http://www.ros.org/wiki/xacro"
-  name="robotino">
+  name="robot">
   <xacro:include filename="$(find robotino_bringup)/robots/alufr-robotino/urdf/properties.urdf.xacro" />
   <xacro:include filename="$(find robotino_description)/urdf/gazebo.urdf.xacro" />
-  <xacro:include filename="$(find robotino_description)/urdf/robotino_body.urdf.xacro" />
+  <xacro:include filename="$(find robotino_description)/urdf/base.urdf.xacro" />
   <xacro:include filename="$(find robotino_description)/urdf/hokuyo.urdf.xacro" />
   <xacro:include filename="$(find robotino_description)/urdf/kinect.urdf.xacro" />
   <xacro:include filename="$(find robotino_description)/urdf/tilt_axis.urdf.xacro" />
-  <xacro:body name="base"/>
+  <xacro:include filename="$(find robotino_description)/urdf/arm.urdf.xacro" />
+  <xacro:base name="base"/>
   <gazebo>
     <plugin name="ros_control" filename="libhwi_switch_gazebo_ros_control.so">
@@ -18,5 +19,14 @@
     <origin xyz="${hokuyo_x} ${hokuyo_y} ${hokuyo_z}" rpy="${hokuyo_roll} ${hokuyo_pitch} ${hokuyo_yaw}"/>
   </hokuyo>
-  <tilt_axis name="tilt" parent="base_link">
+  <xacro:arm name="arm_" parent="base_link">
+    <origin xyz="${arm_x} ${arm_y} ${arm_z}" rpy="${arm_roll} ${arm_pitch} ${arm_yaw}"/>
+  </xacro:arm>
+  <gazebo>
+    <plugin name="ros_control" filename="libhwi_switch_gazebo_ros_control.so">
+      <robotNamespace>arm_controller</robotNamespace>
+      <filterJointsParam>joint_names</filterJointsParam>
+    </plugin>
+  </gazebo>
+  <!--tilt_axis name="tilt" parent="base_link">
     <origin xyz="${tilt_x} ${tilt_y} ${tilt_z}" rpy="${tilt_roll} ${tilt_pitch} ${tilt_yaw}"/>
   </tilt_axis>
@@ -29,4 +39,4 @@
       <filterJointsParam>joint_names</filterJointsParam>
     </plugin>
-  </gazebo>
+  </gazebo-->
 </robot>
