Commit message: updated models

File: robotino_bringup/robots/alufr-robotino/urdf/robotino.urdf.xacro (robot description, xacro)
@@ -6,6 +6,4 @@
   <xacro:include filename="$(find robotino_description)/urdf/robotino_body.urdf.xacro" />
   <xacro:include filename="$(find robotino_description)/urdf/hokuyo.urdf.xacro" />
-  <xacro:include filename="$(find robotino_description)/urdf/camera.urdf.xacro" />
-  <xacro:include filename="$(find robotino_description)/urdf/angle_bracket.urdf.xacro" />
   <xacro:include filename="$(find robotino_description)/urdf/kinect.urdf.xacro" />
   <xacro:include filename="$(find robotino_description)/urdf/tilt_axis.urdf.xacro" />

File: robotino_bringup/robots/ipa-robotino/urdf/robotino.urdf.xacro (robot description, xacro)
@@ -6,6 +6,4 @@
   <xacro:include filename="$(find robotino_description)/urdf/robotino_body.urdf.xacro" />
   <xacro:include filename="$(find robotino_description)/urdf/hokuyo.urdf.xacro" />
-  <xacro:include filename="$(find robotino_description)/urdf/camera.urdf.xacro" />
-  <xacro:include filename="$(find robotino_description)/urdf/angle_bracket.urdf.xacro" />
   <xacro:include filename="$(find robotino_description)/urdf/kinect.urdf.xacro" />
   <xacro:include filename="$(find robotino_description)/urdf/tilt_axis.urdf.xacro" />

File: robotino_bringup/robots/robotino_6dof/urdf/robotino.urdf.xacro (robot description, xacro)
@@ -2,5 +2,5 @@
 <robot xmlns:xacro="http://www.ros.org/wiki/xacro"
   name="robot">
-  <xacro:include filename="$(find robotino_bringup)/robots/robotino/urdf/properties.urdf.xacro" />
+  <xacro:include filename="$(find robotino_bringup)/robots/robotino_6dof/urdf/properties.urdf.xacro" />
   <xacro:include filename="$(find robotino_description)/urdf/robotino_body.urdf.xacro" />
   <xacro:include filename="$(find robotino_description)/urdf/rotatory.urdf.xacro" />

File: robotino_bringup/robots/tuw-robotino/urdf/robotino.urdf.xacro (robot description, xacro)
@@ -6,6 +6,4 @@
   <xacro:include filename="$(find robotino_description)/urdf/robotino_body.urdf.xacro" />
   <xacro:include filename="$(find robotino_description)/urdf/hokuyo.urdf.xacro" />
-  <xacro:include filename="$(find robotino_description)/urdf/camera.urdf.xacro" />
-  <xacro:include filename="$(find robotino_description)/urdf/angle_bracket.urdf.xacro" />
   <xacro:include filename="$(find robotino_description)/urdf/kinect.urdf.xacro" />
   <xacro:include filename="$(find robotino_description)/urdf/pan_tilt_axis.urdf.xacro" />
@@ -14,10 +12,4 @@
     <origin xyz="${hokuyo_x} ${hokuyo_y} ${hokuyo_z}" rpy="${hokuyo_roll} ${hokuyo_pitch} ${hokuyo_yaw}"/>
   </hokuyo>
-  <!--kinect name="kinect" parent="base_link">
-    <origin xyz="${kinect_x} ${kinect_y} ${kinect_z}" rpy="${kinect_roll} ${kinect_pitch} ${kinect_yaw}"/>
-  </kinect-->
-  <!--anglebracketusb name="anglebracketusb" parent="base_link">
-    <origin xyz="${anglebracketusb_x} ${anglebracketusb_y} ${anglebracketusb_z}" rpy="${anglebracketusb_roll} ${anglebracketusb_pitch} ${anglebracketusb_yaw}"/>
-  </anglebracketusb-->
   <pan_tilt_axis parent="base_link">
     <origin xyz="${pan_tilt_x} ${pan_tilt_y} ${pan_tilt_z}" rpy="${pan_tilt_roll} ${pan_tilt_pitch} ${pan_tilt_yaw}"/>
@@ -32,6 +24,3 @@
     </plugin>
   </gazebo>
-  <!--anglebracketusb name="anglebracketusb" parent="base_link">
-      <origin xyz="${anglebracketusb_x} ${anglebracketusb_y} ${anglebracketusb_z}" rpy="${anglebracketusb_roll} ${anglebracketusb_pitch} ${anglebracketusb_yaw}"/>
-  </anglebracketusb-->
 </robot>

File: robotino_bringup/robots/tuw-robotino2/urdf/properties.urdf.xacro (robot description, xacro)
@@ -29,7 +29,7 @@
   <property name="hokuyo_yaw" value="0.0"/>
    <!-- pan_tilt mount positions | handeye calibration | relative to base_link -->
-  <property name="pan_tilt_x" value="0.03"/>
-  <property name="pan_tilt_y" value="0.03"/>
-  <property name="pan_tilt_z" value="0.64"/>
+  <property name="pan_tilt_x" value="0.25"/>
+  <property name="pan_tilt_y" value="0.0"/>
+  <property name="pan_tilt_z" value="0.55"/>
   <property name="pan_tilt_roll" value="0"/>
   <property name="pan_tilt_pitch" value="0"/> <!--${M_PI/2}"/> -->
@@ -42,10 +42,17 @@
   <property name="kinect_pitch" value="0"/>
   <property name="kinect_yaw" value="0.0"/>
-  <!-- anglebracketusb mount positions | handeye calibration | relative to base_link -->
-  <property name="anglebracketusb_x" value="0.008"/>
-  <property name="anglebracketusb_y" value="0.0"/>
-  <property name="anglebracketusb_z" value="0.137"/>
-  <property name="anglebracketusb_roll" value="0.0"/>
-  <property name="anglebracketusb_pitch" value="0.0"/>
-  <property name="anglebracketusb_yaw" value="0.0"/>
+   <!-- arm mount positions | handeye calibration | relative to base_link -->
+  <property name="arm_x" value="0.0"/>
+  <property name="arm_y" value="0.0"/>
+  <property name="arm_z" value="0.35"/>
+  <property name="arm_roll" value="0.0"/>
+  <property name="arm_pitch" value="0.0"/>
+  <property name="arm_yaw" value="0.0"/>
+   <!-- arm calibration-->
+  <property name="arm_1_ref" value="0.0"/>
+  <property name="arm_2_ref" value="0.0"/>
+  <property name="arm_3_ref" value="0.0"/>
+  <property name="arm_4_ref" value="0.0"/>
+  <property name="arm_5_ref" value="0.0"/>
+  <property name="arm_6_ref" value="0.0"/>
 </robot>

File: robotino_bringup/robots/tuw-robotino2/urdf/robotino.urdf.xacro (robot description, xacro)
@@ -1,15 +1,41 @@
 <?xml version="1.0"?>
 <robot xmlns:xacro="http://www.ros.org/wiki/xacro"
-  name="robotino">
-  <xacro:include filename="$(find robotino_bringup)/robots/uibk-robotino/urdf/properties.urdf.xacro" />
+  name="robot">
+  <xacro:include filename="$(find robotino_bringup)/robots/tuw-robotino2/urdf/properties.urdf.xacro" />
   <xacro:include filename="$(find robotino_description)/urdf/gazebo.urdf.xacro" />
   <xacro:include filename="$(find robotino_description)/urdf/robotino_body.urdf.xacro" />
+  <xacro:include filename="$(find robotino_description)/urdf/rotatory.urdf.xacro" />
   <xacro:include filename="$(find robotino_description)/urdf/hokuyo.urdf.xacro" />
   <xacro:include filename="$(find robotino_description)/urdf/kinect.urdf.xacro" />
   <xacro:include filename="$(find robotino_description)/urdf/pan_tilt_axis.urdf.xacro" />
+  <xacro:include filename="$(find robotino_arm_description)/xacro/arm_model.urdf.xacro" />
+  <xacro:include filename="$(find kclhand_description)/urdf/kclhand.urdf.xacro" />
   <xacro:body name="base"/>
   <hokuyo name="hokuyo" parent="base_link">
     <origin xyz="${hokuyo_x} ${hokuyo_y} ${hokuyo_z}" rpy="${hokuyo_roll} ${hokuyo_pitch} ${hokuyo_yaw}"/>
   </hokuyo>
+  <xacro:rotatory />
+  <gazebo>
+    <plugin name="ros_control" filename="libhwi_switch_gazebo_ros_control.so">
+      <robotNamespace>rotatory_controller</robotNamespace>
+      <filterJointsParam>joint_names</filterJointsParam>
+    </plugin>
+  </gazebo>
+  <xacro:arm />
+  <gazebo>
+    <plugin name="ros_control" filename="libhwi_switch_gazebo_ros_control.so">
+      <robotNamespace>arm_controller</robotNamespace>
+      <filterJointsParam>joint_names</filterJointsParam>
+    </plugin>
+  </gazebo>
+  <xacro:kclhand name="hand" parent="link5">
+    <origin xyz="0 0 0" rpy="1.5707963 0 0" />
+  </xacro:kclhand>
+  <gazebo>
+    <plugin name="ros_control" filename="libhwi_switch_gazebo_ros_control.so">
+      <robotNamespace>hand_controller</robotNamespace>
+      <filterJointsParam>joint_names</filterJointsParam>
+    </plugin>
+  </gazebo>
   <pan_tilt_axis parent="base_link">
     <origin xyz="${pan_tilt_x} ${pan_tilt_y} ${pan_tilt_z}" rpy="${pan_tilt_roll} ${pan_tilt_pitch} ${pan_tilt_yaw}"/>

File: robotino_bringup/robots/uibk-robotino/urdf/properties.urdf.xacro (robot description, xacro)
@@ -29,9 +29,9 @@
   <property name="hokuyo_yaw" value="-0.0536545473"/>
    <!-- pan_tilt mount positions | handeye calibration | relative to base_link -->
-  <property name="pan_tilt_x" value="0.25"/>
-  <property name="pan_tilt_y" value="0.0"/>
-  <property name="pan_tilt_z" value="0.5"/>
+  <property name="pan_tilt_x" value="0.03"/>
+  <property name="pan_tilt_y" value="0.03"/>
+  <property name="pan_tilt_z" value="0.64"/>
   <property name="pan_tilt_roll" value="0"/>
-  <property name="pan_tilt_pitch" value="0"/>
+  <property name="pan_tilt_pitch" value="0"/> <!--${M_PI/2}"/> -->
   <property name="pan_tilt_yaw" value="0"/>
   <!-- kinect mount positions | handeye calibration | relative to pan_tilt_link -->
@@ -42,10 +42,3 @@
   <property name="kinect_pitch" value="0"/>
   <property name="kinect_yaw" value="0.0"/>
-  <!-- anglebracketusb mount positions | handeye calibration | relative to base_link -->
-  <property name="anglebracketusb_x" value="0.008"/>
-  <property name="anglebracketusb_y" value="0.0"/>
-  <property name="anglebracketusb_z" value="0.137"/>
-  <property name="anglebracketusb_roll" value="0.0"/>
-  <property name="anglebracketusb_pitch" value="0.0"/>
-  <property name="anglebracketusb_yaw" value="0.0"/>
 </robot>

File: robotino_bringup/robots/uibk-robotino2/urdf/properties.urdf.xacro (robot description, xacro)
@@ -28,19 +28,33 @@
   <property name="hokuyo_pitch" value="0.0"/>
   <property name="hokuyo_yaw" value="0.0"/>
-   <!-- pan_tilt mount positions | handeye calibration | relative to base_link -->
-  <property name="pan_tilt_x" value="0.03"/>
-  <property name="pan_tilt_y" value="0.03"/>
-  <property name="pan_tilt_z" value="0.64"/>
-  <property name="pan_tilt_roll" value="0"/>
-  <property name="pan_tilt_pitch" value="0"/> <!--${M_PI/2}"/> -->
-  <property name="pan_tilt_yaw" value="0"/>
-  <!-- kinect mount positions | handeye calibration | relative to pan_tilt_link -->
-  <property name="kinect_x" value="0.0"/>
-  <property name="kinect_y" value="0.065"/>
+   <!-- tilt mount positions | handeye calibration | relative to base_link -->
+  <property name="tilt_x" value="-0.01"/>
+  <property name="tilt_y" value="0.0"/>
+  <property name="tilt_z" value="0.45"/>
+  <property name="tilt_roll" value="-0.05"/>
+  <property name="tilt_pitch" value="${M_PI/2}"/>
+  <property name="tilt_yaw" value="0"/>
+   <!-- arm mount positions | handeye calibration | relative to base_link -->
+  <property name="arm_x" value="0.0"/>
+  <property name="arm_y" value="0.0"/>
+  <property name="arm_z" value="0.35"/>
+  <property name="arm_roll" value="0.0"/>
+  <property name="arm_pitch" value="0.0"/>
+  <property name="arm_yaw" value="0.0"/>
+   <!-- arm calibration-->
+  <property name="arm_1_ref" value="0.0"/>
+  <property name="arm_2_ref" value="0.0"/>
+  <property name="arm_3_ref" value="0.0"/>
+  <property name="arm_4_ref" value="0.0"/>
+  <property name="arm_5_ref" value="0.0"/>
+  <property name="arm_6_ref" value="0.0"/>
+   <!-- kinect mount positions | handeye calibration | relative to tilt_link -->
+  <property name="kinect_x" value="-0.03"/>
+  <property name="kinect_y" value="0.0"/>
   <property name="kinect_z" value="0.0"/>
-  <property name="kinect_roll" value="-${M_PI/2}"/>
-  <property name="kinect_pitch" value="0"/>
+  <property name="kinect_roll" value="-0.02"/>
+  <property name="kinect_pitch" value="-1.45"/>
   <property name="kinect_yaw" value="0.0"/>
-  <!-- anglebracketusb mount positions | handeye calibration | relative to base_link -->
+   <!-- anglebracketusb mount positions | handeye calibration | relative to base_link -->
   <property name="anglebracketusb_x" value="0.008"/>
   <property name="anglebracketusb_y" value="0.0"/>

Commit message: extra links not needed

File: robotino_bringup/robots/alufr-robotino/urdf/robotino.urdf.xacro (robot description, xacro)
@@ -8,5 +8,5 @@
   <xacro:include filename="$(find robotino_description)/urdf/tilt_axis.urdf.xacro" />
   <xacro:include filename="$(find robotino_description)/urdf/arm.urdf.xacro" />
-  <xacro:base name="base" has_8dof="true"/>
+  <xacro:base name="base" has_8dof="false"/>
   <gazebo>
     <plugin name="ros_control" filename="libhwi_switch_gazebo_ros_control.so">
@@ -15,8 +15,8 @@
     </plugin>
   </gazebo>
-  <hokuyo name="hokuyo" parent="base_linkz">
+  <hokuyo name="hokuyo" parent="base_link">
     <origin xyz="${hokuyo_x} ${hokuyo_y} ${hokuyo_z}" rpy="${hokuyo_roll} ${hokuyo_pitch} ${hokuyo_yaw}"/>
   </hokuyo>
-  <xacro:arm name="arm_" parent="base_linkz">
+  <xacro:arm name="arm_" parent="base_link">
     <origin xyz="${arm_x} ${arm_y} ${arm_z}" rpy="${arm_roll} ${arm_pitch} ${arm_yaw}"/>
   </xacro:arm>

File: robotino_bringup/robots/tuw-robotino2/urdf/robotino.urdf.xacro (robot description, xacro)
@@ -9,5 +9,5 @@
   <xacro:include filename="$(find robotino_description)/urdf/arm.urdf.xacro" />
   <xacro:include filename="$(find robotino_description)/urdf/kclhand_withCableCanal.urdf.xacro" />
-  <xacro:base name="base" has_8dof="true"/>
+  <xacro:base name="base" has_8dof="false"/>
   <gazebo>
     <plugin name="ros_control" filename="libhwi_switch_gazebo_ros_control.so">
@@ -16,8 +16,8 @@
     </plugin>
   </gazebo>
-  <hokuyo name="hokuyo" parent="base_linkz">
+  <hokuyo name="hokuyo" parent="base_link">
     <origin xyz="${hokuyo_x} ${hokuyo_y} ${hokuyo_z}" rpy="${hokuyo_roll} ${hokuyo_pitch} ${hokuyo_yaw}"/>
   </hokuyo>
-  <xacro:arm name="arm_" parent="base_linkz">
+  <xacro:arm name="arm_" parent="base_link">
     <origin xyz="${arm_x} ${arm_y} ${arm_z}" rpy="${arm_roll} ${arm_pitch} ${arm_yaw}"/>
   </xacro:arm>
@@ -37,5 +37,5 @@
     </plugin>
   </gazebo>
-  <pan_tilt_axis parent="base_linkz">
+  <pan_tilt_axis parent="base_link">
     <origin xyz="${pan_tilt_x} ${pan_tilt_y} ${pan_tilt_z}" rpy="${pan_tilt_roll} ${pan_tilt_pitch} ${pan_tilt_yaw}"/>
   </pan_tilt_axis>

File: robotino_bringup/robots/uibk-robotino2-sh/urdf/robotino.urdf.xacro (robot description, xacro)
@@ -9,5 +9,5 @@
   <xacro:include filename="$(find robotino_description)/urdf/arm.urdf.xacro" />
   <xacro:include filename="$(find soft_hand_description)/model/softhand_withCableCanal.urdf.xacro" />
-  <xacro:base name="base" has_8dof="true"/>
+  <xacro:base name="base" has_8dof="false"/>
   <gazebo>
     <plugin name="ros_control" filename="libhwi_switch_gazebo_ros_control.so">
@@ -16,8 +16,8 @@
     </plugin>
   </gazebo>
-  <hokuyo name="hokuyo" parent="base_linkz">
+  <hokuyo name="hokuyo" parent="base_link">
     <origin xyz="${hokuyo_x} ${hokuyo_y} ${hokuyo_z}" rpy="${hokuyo_roll} ${hokuyo_pitch} ${hokuyo_yaw}"/>
   </hokuyo>
-  <xacro:arm name="arm_" parent="base_linkz">
+  <xacro:arm name="arm_" parent="base_link">
     <origin xyz="${arm_x} ${arm_y} ${arm_z}" rpy="${arm_roll} ${arm_pitch} ${arm_yaw}"/>
   </xacro:arm>
@@ -37,5 +37,5 @@
     </plugin>
   </gazebo>
-  <pan_tilt_axis parent="base_linkz">
+  <pan_tilt_axis parent="base_link">
     <origin xyz="${pan_tilt_x} ${pan_tilt_y} ${pan_tilt_z}" rpy="${pan_tilt_roll} ${pan_tilt_pitch} ${pan_tilt_yaw}"/>
   </pan_tilt_axis>

File: robotino_bringup/robots/uibk-robotino2-sh/urdf/robotino_base_plan.urdf.xacro (robot description, xacro)
@@ -8,6 +8,6 @@
   <xacro:include filename="$(find robotino_description)/urdf/pan_tilt_axis.urdf.xacro" />
   <xacro:include filename="$(find robotino_description)/urdf/arm.urdf.xacro" />
-  <xacro:include filename="$(find robotino_description)/urdf/kclhand_withCableCanal.urdf.xacro" />
-  <xacro:base name="base" has_8dof="false"/>
+  <xacro:include filename="$(find soft_hand_description)/model/softhand_withCableCanal.urdf.xacro" />
+  <xacro:base name="base" has_8dof="true"/>
   <gazebo>
     <plugin name="ros_control" filename="libhwi_switch_gazebo_ros_control.so">
@@ -16,8 +16,8 @@
     </plugin>
   </gazebo>
-  <hokuyo name="hokuyo" parent="base_link">
+  <hokuyo name="hokuyo" parent="base_linkz">
     <origin xyz="${hokuyo_x} ${hokuyo_y} ${hokuyo_z}" rpy="${hokuyo_roll} ${hokuyo_pitch} ${hokuyo_yaw}"/>
   </hokuyo>
-  <xacro:arm name="arm_" parent="base_link">
+  <xacro:arm name="arm_" parent="base_linkz">
     <origin xyz="${arm_x} ${arm_y} ${arm_z}" rpy="${arm_roll} ${arm_pitch} ${arm_yaw}"/>
   </xacro:arm>
@@ -28,7 +28,7 @@
     </plugin>
   </gazebo>
-  <xacro:kclhand name="hand" parent="arm_link5">
+  <xacro:soft_hand name="hand" parent="arm_link5" withAdaptiveTransmission="false" useMimicTag="false" left="false">
     <origin xyz="0 0 0" rpy="1.5707963 0 0" />
-  </xacro:kclhand>
+  </xacro:soft_hand>
   <gazebo>
     <plugin name="ros_control" filename="libhwi_switch_gazebo_ros_control.so">
@@ -37,5 +37,5 @@
     </plugin>
   </gazebo>
-  <pan_tilt_axis parent="base_link">
+  <pan_tilt_axis parent="base_linkz">
     <origin xyz="${pan_tilt_x} ${pan_tilt_y} ${pan_tilt_z}" rpy="${pan_tilt_roll} ${pan_tilt_pitch} ${pan_tilt_yaw}"/>
   </pan_tilt_axis>

File: robotino_bringup/robots/uibk-robotino2/urdf/robotino.urdf (robot description, URDF)
Before this commit: robot robot, 35 links, 34 joints
Links:
- removed link origin
- link base_linkx: mass 10 -> 0.01; geometry collision box size=0.001 0.001 0.001; visual box size=0.001 0.001 0.001
- link base_linky: mass 10 -> 0.01; geometry collision box size=0.001 0.001 0.001; visual box size=0.001 0.001 0.001
- link base_linkz: mass 10 -> 0.01; geometry collision box size=0.001 0.001 0.001; visual box size=0.001 0.001 0.001
Joints:
- removed joint origin_joint
- joint base_jointx: limit lower=-10 upper=10 effort=190 velocity=30 -> lower=-10 upper=10 effort=0 velocity=0
- joint base_jointy: limit lower=-10 upper=10 effort=190 velocity=30 -> lower=-10 upper=10 effort=0 velocity=0
- joint base_jointz: limit lower=-3.14 upper=3.14 effort=190 velocity=30 -> lower=-3.14 upper=3.14 effort=0 velocity=0
- joint hokuyo_joint: parent base_link -> base_linkz
- joint profile_joint: parent base_link -> base_linkz

File: robotino_bringup/robots/uibk-robotino2/urdf/robotino_base_plan.urdf.xacro (robot description, xacro)
@@ -9,5 +9,5 @@
   <xacro:include filename="$(find robotino_description)/urdf/arm.urdf.xacro" />
   <xacro:include filename="$(find robotino_description)/urdf/kclhand_withCableCanal.urdf.xacro" />
-  <xacro:base name="base" has_8dof="false"/>
+  <xacro:base name="base" has_8dof="true"/>
   <gazebo>
     <plugin name="ros_control" filename="libhwi_switch_gazebo_ros_control.so">
@@ -16,8 +16,8 @@
     </plugin>
   </gazebo>
-  <hokuyo name="hokuyo" parent="base_link">
+  <hokuyo name="hokuyo" parent="base_linkz">
     <origin xyz="${hokuyo_x} ${hokuyo_y} ${hokuyo_z}" rpy="${hokuyo_roll} ${hokuyo_pitch} ${hokuyo_yaw}"/>
   </hokuyo>
-  <xacro:arm name="arm_" parent="base_link">
+  <xacro:arm name="arm_" parent="base_linkz">
     <origin xyz="${arm_x} ${arm_y} ${arm_z}" rpy="${arm_roll} ${arm_pitch} ${arm_yaw}"/>
   </xacro:arm>
@@ -37,5 +37,5 @@
     </plugin>
   </gazebo>
-  <pan_tilt_axis parent="base_link">
+  <pan_tilt_axis parent="base_linkz">
     <origin xyz="${pan_tilt_x} ${pan_tilt_y} ${pan_tilt_z}" rpy="${pan_tilt_roll} ${pan_tilt_pitch} ${pan_tilt_yaw}"/>
   </pan_tilt_axis>
