Commit message: update base model

File: robotino_bringup/robots/alufr-robotino/urdf/robotino.urdf.xacro (robot description, xacro)
@@ -15,8 +15,8 @@
     </plugin>
   </gazebo>
-  <hokuyo name="hokuyo" parent="base_link">
+  <hokuyo name="hokuyo" parent="base_linkz">
     <origin xyz="${hokuyo_x} ${hokuyo_y} ${hokuyo_z}" rpy="${hokuyo_roll} ${hokuyo_pitch} ${hokuyo_yaw}"/>
   </hokuyo>
-  <xacro:arm name="arm_" parent="base_link">
+  <xacro:arm name="arm_" parent="base_linkz">
     <origin xyz="${arm_x} ${arm_y} ${arm_z}" rpy="${arm_roll} ${arm_pitch} ${arm_yaw}"/>
   </xacro:arm>
@@ -27,15 +27,3 @@
     </plugin>
   </gazebo>
-  <!--tilt_axis name="tilt" parent="base_link">
-    <origin xyz="${tilt_x} ${tilt_y} ${tilt_z}" rpy="${tilt_roll} ${tilt_pitch} ${tilt_yaw}"/>
-  </tilt_axis>
-  <kinect name="kinect" parent="tilt_link">
-    <origin xyz="${kinect_x} ${kinect_y} ${kinect_z}" rpy="${kinect_roll} ${kinect_pitch} ${kinect_yaw}"/>
-  </kinect>
-  <gazebo>
-    <plugin name="ros_control" filename="libhwi_switch_gazebo_ros_control.so">
-      <robotNamespace>tilt_controller</robotNamespace>
-      <filterJointsParam>joint_names</filterJointsParam>
-    </plugin>
-  </gazebo-->
 </robot>

File: robotino_bringup/robots/ipa-robotino/urdf/robotino.urdf.xacro (robot description, xacro)
@@ -14,11 +14,11 @@
     </plugin>
   </gazebo>
-  <hokuyo name="hokuyo" parent="base_link">
+  <hokuyo name="hokuyo" parent="base_linkz">
     <origin xyz="${hokuyo_x} ${hokuyo_y} ${hokuyo_z}" rpy="${hokuyo_roll} ${hokuyo_pitch} ${hokuyo_yaw}"/>
   </hokuyo>
-  <tilt_axis name="tilt" parent="base_link">
+  <tilt_axis name="tilt" parent="base_linkz">
     <origin xyz="${tilt_x} ${tilt_y} ${tilt_z}" rpy="${tilt_roll} ${tilt_pitch} ${tilt_yaw}"/>
   </tilt_axis>
-  <kinect name="kinect" parent="tilt_link">
+  <kinect name="kinect" parent="tilt_linkz">
     <origin xyz="${kinect_x} ${kinect_y} ${kinect_z}" rpy="${kinect_roll} ${kinect_pitch} ${kinect_yaw}"/>
   </kinect>

File: robotino_bringup/robots/tuw-robotino2/urdf/robotino.urdf.xacro (robot description, xacro)
@@ -17,11 +17,11 @@
     </plugin>
   </gazebo>
-  <xacro:shell name="base_shell" parent="base_link">
+  <xacro:shell name="base_shell" parent="base_linkz">
     <origin xyz="0 0 0" rpy="0 0 0"/>
   </xacro:shell>
-  <hokuyo name="hokuyo" parent="base_link">
+  <hokuyo name="hokuyo" parent="base_linkz">
     <origin xyz="${hokuyo_x} ${hokuyo_y} ${hokuyo_z}" rpy="${hokuyo_roll} ${hokuyo_pitch} ${hokuyo_yaw}"/>
   </hokuyo>
-  <xacro:arm name="arm_" parent="base_link">
+  <xacro:arm name="arm_" parent="base_linkz">
     <origin xyz="${arm_x} ${arm_y} ${arm_z}" rpy="${arm_roll} ${arm_pitch} ${arm_yaw}"/>
   </xacro:arm>
@@ -41,5 +41,5 @@
     </plugin>
   </gazebo>
-  <pan_tilt_axis parent="base_link">
+  <pan_tilt_axis parent="base_linkz">
     <origin xyz="${pan_tilt_x} ${pan_tilt_y} ${pan_tilt_z}" rpy="${pan_tilt_roll} ${pan_tilt_pitch} ${pan_tilt_yaw}"/>
   </pan_tilt_axis>

File: robotino_bringup/robots/uibk-robotino/urdf/robotino.urdf.xacro (robot description, xacro)
@@ -14,8 +14,8 @@
     </plugin>
   </gazebo>
-  <hokuyo name="hokuyo" parent="base_link">
+  <hokuyo name="hokuyo" parent="base_linkz">
     <origin xyz="${hokuyo_x} ${hokuyo_y} ${hokuyo_z}" rpy="${hokuyo_roll} ${hokuyo_pitch} ${hokuyo_yaw}"/>
   </hokuyo>
-  <pan_tilt_axis parent="base_link">
+  <pan_tilt_axis parent="base_linkz">
     <origin xyz="${pan_tilt_x} ${pan_tilt_y} ${pan_tilt_z}" rpy="${pan_tilt_roll} ${pan_tilt_pitch} ${pan_tilt_yaw}"/>
   </pan_tilt_axis>

File: robotino_bringup/robots/uibk-robotino2-sh/urdf/robotino.urdf.xacro (robot description, xacro)
@@ -16,8 +16,8 @@
     </plugin>
   </gazebo>
-  <hokuyo name="hokuyo" parent="base_link">
+  <hokuyo name="hokuyo" parent="base_linkz">
     <origin xyz="${hokuyo_x} ${hokuyo_y} ${hokuyo_z}" rpy="${hokuyo_roll} ${hokuyo_pitch} ${hokuyo_yaw}"/>
   </hokuyo>
-  <xacro:arm name="arm_" parent="base_link">
+  <xacro:arm name="arm_" parent="base_linkz">
     <origin xyz="${arm_x} ${arm_y} ${arm_z}" rpy="${arm_roll} ${arm_pitch} ${arm_yaw}"/>
   </xacro:arm>
@@ -37,5 +37,5 @@
     </plugin>
   </gazebo>
-  <pan_tilt_axis parent="base_link">
+  <pan_tilt_axis parent="base_linkz">
     <origin xyz="${pan_tilt_x} ${pan_tilt_y} ${pan_tilt_z}" rpy="${pan_tilt_roll} ${pan_tilt_pitch} ${pan_tilt_yaw}"/>
   </pan_tilt_axis>

File: robotino_bringup/robots/uibk-robotino2/urdf/robotino.urdf.xacro (robot description, xacro)
@@ -16,8 +16,8 @@
     </plugin>
   </gazebo>
-  <hokuyo name="hokuyo" parent="base_link">
+  <hokuyo name="hokuyo" parent="base_linkz">
     <origin xyz="${hokuyo_x} ${hokuyo_y} ${hokuyo_z}" rpy="${hokuyo_roll} ${hokuyo_pitch} ${hokuyo_yaw}"/>
   </hokuyo>
-  <xacro:arm name="arm_" parent="base_link">
+  <xacro:arm name="arm_" parent="base_linkz">
     <origin xyz="${arm_x} ${arm_y} ${arm_z}" rpy="${arm_roll} ${arm_pitch} ${arm_yaw}"/>
   </xacro:arm>
@@ -37,5 +37,5 @@
     </plugin>
   </gazebo>
-  <pan_tilt_axis parent="base_link">
+  <pan_tilt_axis parent="base_linkz">
     <origin xyz="${pan_tilt_x} ${pan_tilt_y} ${pan_tilt_z}" rpy="${pan_tilt_roll} ${pan_tilt_pitch} ${pan_tilt_yaw}"/>
   </pan_tilt_axis>

Commit message: remove simulation model

File: robotino_bringup/robots/alufr-robotino/urdf/robotino.urdf.xacro (robot description, xacro)
@@ -27,3 +27,12 @@
     </plugin>
   </gazebo>
+  <xacro:tilt_axis name="tilt" parent="base_linkz">
+    <origin xyz="${tilt_x} ${tilt_y} ${tilt_z}" rpy="${tilt_roll} ${tilt_pitch} ${tilt_yaw}"/>
+  </xacro:tilt_axis>
+  <gazebo>
+    <plugin name="ros_control" filename="libhwi_switch_gazebo_ros_control.so">
+      <robotNamespace>tilt_controller</robotNamespace>
+      <filterJointsParam>joint_names</filterJointsParam>
+    </plugin>
+  </gazebo>
 </robot>
