Commit message: moved the collision

File: robotino_bringup/robots/uibk-robotino2/urdf/robotino.urdf.xacro (robot description, xacro)
@@ -29,5 +29,5 @@
   </hokuyo>
   <case name="case" parent="base_link">
-    <origin xyz="0 0 0" rpy="0 0 0"/>
+    <origin xyz="0 0 0" rpy="0 0 -0.5"/>
   </case>
   <xacro:rotatory />

Commit message: addapted base to 8 dof modus

File: robotino_bringup/robots/uibk-robotino2/urdf/robotino.urdf.xacro (robot description, xacro)
@@ -3,5 +3,4 @@
   name="robot">
   <xacro:include filename="$(find robotino_bringup)/robots/uibk-robotino2/urdf/properties.urdf.xacro" />
-  <xacro:include filename="$(find robotino_description)/urdf/gazebo.urdf.xacro" />
   <xacro:include filename="$(find robotino_description)/urdf/base.urdf.xacro" />
   <xacro:include filename="$(find robotino_description)/urdf/hokuyo.urdf.xacro" />
@@ -10,14 +9,5 @@
   <xacro:include filename="$(find robotino_description)/urdf/arm.urdf.xacro" />
   <xacro:include filename="$(find robotino_description)/urdf/kclhand_withCableCanal.urdf.xacro" />
-  <xacro:base name="base"/>
-  <link name="origin">
-      <inertial>
-        <mass value="10" />
-        <origin xyz="0 0 0" />
-        <inertia ixx="75.0" ixy="0.0" ixz="0.0"
-          iyy="75.0" iyz="0.0"
-          izz="75.0" />
-      </inertial>
-    </link>
+  <xacro:base name="base" has_8dof="true"/>
   <gazebo>
     <plugin name="ros_control" filename="libhwi_switch_gazebo_ros_control.so">
