Commit message: removed kcl hand

File: robotino_bringup/robots/uibk-robotino2/urdf/robotino.urdf (robot description, URDF)
Before this commit: robot robot, 34 links, 33 joints
Links:
- removed link hand_base_link
- removed link hand_cableCanal_link
- removed link hand_left_coupler
- removed link hand_left_crank
- removed link hand_left_finger_lower_link
- removed link hand_left_finger_upper_link
- removed link hand_middle_finger_lower_link
- removed link hand_middle_finger_upper_link
- removed link hand_right_coupler
- removed link hand_right_crank
- removed link hand_right_finger_lower_link
- removed link hand_right_finger_upper_link
- removed link hand_wrist_link
Joints:
- removed joint hand_base_joint
- removed joint hand_cableCanal_joint
- removed joint hand_left_coupler_crank_joint
- removed joint hand_left_crank_base_joint
- removed joint hand_left_finger_lower_joint
- removed joint hand_left_finger_upper_joint
- removed joint hand_middle_finger_lower_joint
- removed joint hand_middle_finger_upper_joint
- removed joint hand_right_coupler_crank_joint
- removed joint hand_right_crank_base_joint
- removed joint hand_right_finger_lower_joint
- removed joint hand_right_finger_upper_joint
- removed joint hand_wrist_joint
- joint base_pan_joint: origin xyz=0.320469 0.00236992 0.658982 rpy=-0.0832053 -0.0319834 0.0585037 -> xyz=0.257201 0.0587815 0.637117 rpy=0.012045 -0.0565489 0.0113182
- joint kinect_joint: origin xyz=0.0341998 0.117973 -0.0696038 rpy=1.65 -3.05142 3.13415 -> xyz=0.0772857 0.117459 -0.0273189 rpy=1.57297 -3.11833 3.10173

File: robotino_bringup/robots/uibk-robotino2/urdf/robotino.urdf.xacro (robot description, xacro)
@@ -9,5 +9,5 @@
   <xacro:include filename="$(find robotino_description)/urdf/pan_tilt_axis.urdf.xacro" />
   <xacro:include filename="$(find robotino_description)/urdf/arm.urdf.xacro" />
-  <xacro:include filename="$(find robotino_description)/urdf/kclhand_withCableCanal.urdf.xacro" />
+  <!--<xacro:include filename="$(find robotino_description)/urdf/kclhand_withCableCanal.urdf.xacro" />-->
   <xacro:base name="base"/>
   <gazebo>
@@ -29,7 +29,9 @@
     </plugin>
   </gazebo>
+<!--
   <xacro:kclhand name="hand" parent="arm_link5">
     <origin xyz="0 0 0" rpy="1.5707963 0 0" />
   </xacro:kclhand>
+-->
   <gazebo>
     <plugin name="ros_control" filename="libhwi_switch_gazebo_ros_control.so">

Commit message: rolled my stuff back to the original urdf.xacro

File: robotino_bringup/robots/uibk-robotino2/urdf/robotino.urdf (robot description, URDF)
Before this commit: robot robot, 34 links, 33 joints
Links:
- removed link base_body_link
- removed link base_linkx
- removed link base_linky
- removed link base_linkz
- link base_link: geometry collision mesh filename=package://robotino_description/meshes/RobotinoBody.stl; visual mesh filename=package://robotino_description/meshes/RobotinoBody.dae
Joints:
- removed joint base_body_joint
- removed joint base_jointx
- removed joint base_jointy
- removed joint base_jointz
- joint arm_base_joint: parent base_linkz -> base_link
- joint base_pan_joint: origin xyz=0.320469 0.00236992 0.658982 rpy=-0.0832053 -0.0319834 0.0585037 -> xyz=0.257201 0.0587815 0.637117 rpy=0.012045 -0.0565489 0.0113182
- joint hokuyo_joint: origin xyz=0.208610627 0.0 0.15 rpy=0.0 0.0 0.0 -> xyz=0.208610627 0.0 0.095 rpy=0.0 0.0 0.0; parent base_linkz -> base_link
- joint kinect_joint: origin xyz=0.0341998 0.117973 -0.0696038 rpy=1.65 -3.05142 3.13415 -> xyz=0.0772857 0.117459 -0.0273189 rpy=1.57297 -3.11833 3.10173
- joint profile_joint: parent base_linkz -> base_link
- joint wheel0_joint: parent base_linkz -> base_link
- joint wheel1_joint: parent base_linkz -> base_link
- joint wheel2_joint: parent base_linkz -> base_link

Commit message: fixed several issues in robot model (8-dof planning not possible because base joints were not in the same chain; profile like was not attached to the moving base, ...)

File: robotino_bringup/robots/uibk-robotino2/urdf/robotino.urdf (robot description, URDF)
Before this commit: robot robot, 30 links, 29 joints
Links:
- added link base_body_link, mass 10; collision mesh filename=package://robotino_description/meshes/RobotinoBody.stl; visual mesh filename=package://robotino_description/meshes/RobotinoBody.dae
- added link base_linkx, mass 10
- added link base_linky, mass 10
- added link base_linkz, mass 10
- link base_link: geometry 
Joints:
- added joint base_body_joint: type fixed, parent base_linkz, child base_body_link, origin xyz=0 0 0 rpy=0 0 0
- added joint base_jointx: type prismatic, parent base_link, child base_linkx, origin xyz=0 0 0 rpy=0 0 0, axis 1 0 0, limit lower=-10 upper=10 effort=190 velocity=30
- added joint base_jointy: type prismatic, parent base_linkx, child base_linky, origin xyz=0 0 0 rpy=0 0 0, axis 0 1 0, limit lower=-10 upper=10 effort=190 velocity=30
- added joint base_jointz: type revolute, parent base_linky, child base_linkz, origin xyz=0 0 0 rpy=0 0 0, axis 0 0 1, limit lower=-3.14 upper=3.14 effort=190 velocity=30
- joint arm_base_joint: parent base_link -> base_linkz
- joint hokuyo_joint: parent base_link -> base_linkz
- joint profile_joint: parent base_link -> base_linkz
- joint wheel0_joint: parent base_link -> base_linkz
- joint wheel1_joint: parent base_link -> base_linkz
- joint wheel2_joint: parent base_link -> base_linkz

File: robotino_bringup/robots/uibk-robotino2/urdf/robotino.urdf.xacro (robot description, xacro)
@@ -17,8 +17,8 @@
     </plugin>
   </gazebo>
-  <hokuyo name="hokuyo" parent="base_link">
+  <hokuyo name="hokuyo" parent="base_linkz">
     <origin xyz="${hokuyo_x} ${hokuyo_y} ${hokuyo_z}" rpy="${hokuyo_roll} ${hokuyo_pitch} ${hokuyo_yaw}"/>
   </hokuyo>
-  <xacro:arm name="arm_" parent="base_link">
+  <xacro:arm name="arm_" parent="base_linkz">
     <origin xyz="${arm_x} ${arm_y} ${arm_z}" rpy="${arm_roll} ${arm_pitch} ${arm_yaw}"/>
   </xacro:arm>
@@ -38,5 +38,5 @@
     </plugin>
   </gazebo>
-  <pan_tilt_axis parent="base_link">
+  <pan_tilt_axis parent="base_linkz">
     <origin xyz="${pan_tilt_x} ${pan_tilt_y} ${pan_tilt_z}" rpy="${pan_tilt_roll} ${pan_tilt_pitch} ${pan_tilt_yaw}"/>
   </pan_tilt_axis>

Commit message: made navigation and planning to work in parallel

File: robotino_bringup/robots/uibk-robotino2/urdf/robotino.urdf (robot description, URDF)
Before this commit: robot robot, 34 links, 33 joints
Links:
- added link origin, mass 10
Joints:
- added joint origin_joint: type prismatic, parent origin, child base_link, origin xyz=0 0 0 rpy=0 0 0, axis 1 0 0, limit lower=-10 upper=10 effort=190 velocity=30
- joint base_jointx: parent base_link -> origin
- joint hokuyo_joint: parent base_linkz -> base_link
- joint profile_joint: parent base_linkz -> base_link

File: robotino_bringup/robots/uibk-robotino2/urdf/robotino.urdf.xacro (robot description, xacro)
@@ -11,4 +11,13 @@
   <xacro:include filename="$(find robotino_description)/urdf/kclhand_withCableCanal.urdf.xacro" />
   <xacro:base name="base"/>
+  <link name="origin">
+      <inertial>
+        <mass value="10" />
+        <origin xyz="0 0 0" />
+        <inertia ixx="75.0" ixy="0.0" ixz="0.0"
+          iyy="75.0" iyz="0.0"
+          izz="75.0" />
+      </inertial>
+    </link>
   <gazebo>
     <plugin name="ros_control" filename="libhwi_switch_gazebo_ros_control.so">
@@ -17,5 +26,5 @@
     </plugin>
   </gazebo>
-  <hokuyo name="hokuyo" parent="base_linkz">
+  <hokuyo name="hokuyo" parent="base_link">
     <origin xyz="${hokuyo_x} ${hokuyo_y} ${hokuyo_z}" rpy="${hokuyo_roll} ${hokuyo_pitch} ${hokuyo_yaw}"/>
   </hokuyo>
@@ -38,5 +47,5 @@
     </plugin>
   </gazebo>
-  <pan_tilt_axis parent="base_linkz">
+  <pan_tilt_axis parent="base_link">
     <origin xyz="${pan_tilt_x} ${pan_tilt_y} ${pan_tilt_z}" rpy="${pan_tilt_roll} ${pan_tilt_pitch} ${pan_tilt_yaw}"/>
   </pan_tilt_axis>

Commit message: siple model

File: robotino_bringup/robots/uibk-robotino2/urdf/robotino.urdf (robot description, URDF)
Before this commit: robot robot, 34 links, 34 joints
Links:
- link base_body_link: geometry collision cylinder length=0.24 radius=0.23; visual mesh filename=package://robotino_description/meshes/RobotinoBody.dae
- link base_linkx: geometry 
- link base_linky: geometry 
- link base_linkz: geometry 
