Commit message: added uibk2 simulation model

File: robotino_bringup/robots/uibk-robotino2/urdf/properties.urdf.xacro (robot description, xacro)
@@ -28,11 +28,18 @@
   <property name="hokuyo_pitch" value="0.0"/>
   <property name="hokuyo_yaw" value="0.0"/>
-   <!-- tilt mount positions | handeye calibration | relative to base_link -->
-  <property name="tilt_x" value="-0.01"/>
-  <property name="tilt_y" value="0.0"/>
-  <property name="tilt_z" value="0.45"/>
-  <property name="tilt_roll" value="-0.05"/>
-  <property name="tilt_pitch" value="${M_PI/2}"/>
-  <property name="tilt_yaw" value="0"/>
+   <!-- pan_tilt mount positions | handeye calibration | relative to base_link -->
+  <property name="pan_tilt_x" value="0.25"/>
+  <property name="pan_tilt_y" value="0.0"/>
+  <property name="pan_tilt_z" value="0.55"/>
+  <property name="pan_tilt_roll" value="0"/>
+  <property name="pan_tilt_pitch" value="0"/> <!--${M_PI/2}"/> -->
+  <property name="pan_tilt_yaw" value="0"/>
+  <!-- kinect mount positions | handeye calibration | relative to pan_tilt_link -->
+  <property name="kinect_x" value="0.0"/>
+  <property name="kinect_y" value="0.065"/>
+  <property name="kinect_z" value="0.0"/>
+  <property name="kinect_roll" value="-${M_PI/2}"/>
+  <property name="kinect_pitch" value="0"/>
+  <property name="kinect_yaw" value="0.0"/>
    <!-- arm mount positions | handeye calibration | relative to base_link -->
   <property name="arm_x" value="0.0"/>
@@ -49,17 +56,3 @@
   <property name="arm_5_ref" value="0.0"/>
   <property name="arm_6_ref" value="0.0"/>
-   <!-- kinect mount positions | handeye calibration | relative to tilt_link -->
-  <property name="kinect_x" value="-0.03"/>
-  <property name="kinect_y" value="0.0"/>
-  <property name="kinect_z" value="0.0"/>
-  <property name="kinect_roll" value="-0.02"/>
-  <property name="kinect_pitch" value="-1.45"/>
-  <property name="kinect_yaw" value="0.0"/>
-   <!-- anglebracketusb mount positions | handeye calibration | relative to base_link -->
-  <property name="anglebracketusb_x" value="0.008"/>
-  <property name="anglebracketusb_y" value="0.0"/>
-  <property name="anglebracketusb_z" value="0.137"/>
-  <property name="anglebracketusb_roll" value="0.0"/>
-  <property name="anglebracketusb_pitch" value="0.0"/>
-  <property name="anglebracketusb_yaw" value="0.0"/>
 </robot>

File: robotino_bringup/robots/uibk-robotino2/urdf/robotino.urdf.xacro (robot description, xacro)
@@ -2,28 +2,24 @@
 <robot xmlns:xacro="http://www.ros.org/wiki/xacro"
   name="robot">
-  <xacro:include filename="$(find robotino_bringup)/robots/robotino/urdf/properties.urdf.xacro" />
+  <xacro:include filename="$(find robotino_bringup)/robots/uibk-robotino2/urdf/properties.urdf.xacro" />
   <xacro:include filename="$(find robotino_description)/urdf/gazebo.urdf.xacro" />
   <xacro:include filename="$(find robotino_description)/urdf/robotino_body.urdf.xacro" />
+  <xacro:include filename="$(find robotino_description)/urdf/rotatory.urdf.xacro" />
   <xacro:include filename="$(find robotino_description)/urdf/hokuyo.urdf.xacro" />
-  <xacro:include filename="$(find robotino_description)/urdf/camera.urdf.xacro" />
-  <xacro:include filename="$(find robotino_description)/urdf/angle_bracket.urdf.xacro" />
   <xacro:include filename="$(find robotino_description)/urdf/kinect.urdf.xacro" />
-  <xacro:include filename="$(find robotino_description)/urdf/tilt_axis.urdf.xacro" />
+  <xacro:include filename="$(find robotino_description)/urdf/pan_tilt_axis.urdf.xacro" />
   <xacro:include filename="$(find robotino_arm_description)/xacro/arm_model.urdf.xacro" />
-  <xacro:include filename="$(find robotino_description)/urdf/soft_hand.urdf.xacro" />
+  <xacro:include filename="$(find kclhand_description)/urdf/kclhand.urdf.xacro" />
   <xacro:body name="base"/>
   <hokuyo name="hokuyo" parent="base_link">
     <origin xyz="${hokuyo_x} ${hokuyo_y} ${hokuyo_z}" rpy="${hokuyo_roll} ${hokuyo_pitch} ${hokuyo_yaw}"/>
   </hokuyo>
-  <joint name="fixed_base_link_base" type="fixed">
-      <parent link="base_link"/>
-      <child link="base"/>
-      <origin xyz="0.0 0.0 0.185" rpy="0 0 -1.0471975511965976" />
-  </joint>
-  <link name="odomp"/>
-  <joint name="rotatory" type="fixed">
-    <parent link="odomp"/>
-    <child link="base_link"/>
-  </joint>
+  <xacro:rotatory />
+  <gazebo>
+    <plugin name="ros_control" filename="libhwi_switch_gazebo_ros_control.so">
+      <robotNamespace>rotatory_controller</robotNamespace>
+      <filterJointsParam>joint_names</filterJointsParam>
+    </plugin>
+  </gazebo>
   <xacro:arm />
   <gazebo>
@@ -33,12 +29,24 @@
     </plugin>
   </gazebo>
-	<xacro:soft_hand parent="link5" name="soft_hand" withAdaptiveTransmission="true" useMimicTag="true" left="true">
-		<origin xyz="0.0 0.0 0.0" rpy="0 0 0"/>
-	</xacro:soft_hand>
-  <!--gazebo>
+  <xacro:kclhand name="hand" parent="link5">
+    <origin xyz="0 0 0" rpy="1.5707963 0 0" />
+  </xacro:kclhand>
+  <gazebo>
     <plugin name="ros_control" filename="libhwi_switch_gazebo_ros_control.so">
       <robotNamespace>hand_controller</robotNamespace>
       <filterJointsParam>joint_names</filterJointsParam>
     </plugin>
-  </gazebo-->
+  </gazebo>
+  <pan_tilt_axis parent="base_link">
+    <origin xyz="${pan_tilt_x} ${pan_tilt_y} ${pan_tilt_z}" rpy="${pan_tilt_roll} ${pan_tilt_pitch} ${pan_tilt_yaw}"/>
+  </pan_tilt_axis>
+  <kinect name="kinect" parent="tilt_link">
+    <origin xyz="${kinect_x} ${kinect_y} ${kinect_z}" rpy="${kinect_roll} ${kinect_pitch} ${kinect_yaw}"/>
+  </kinect>
+  <gazebo>
+    <plugin name="ros_control" filename="libhwi_switch_gazebo_ros_control.so">
+      <robotNamespace>pan_tilt_controller</robotNamespace>
+      <filterJointsParam>joint_names</filterJointsParam>
+    </plugin>
+  </gazebo>
 </robot>

Commit message: added the shell model and controllers to UIBK robotino

File: robotino_bringup/robots/uibk-robotino2/urdf/properties.urdf.xacro (robot description, xacro)
@@ -21,18 +21,25 @@
   <property name="hokuyo_pitch" value="0.0"/>
   <property name="hokuyo_yaw" value="0.0"/>
-  <!-- pan_tilt mount positions | handeye calibration | relative to base_link -->
-  <property name="pan_tilt_x" value="0.257172"/>
-  <property name="pan_tilt_y" value="-0.0242152"/>
-  <property name="pan_tilt_z" value="0.690907"/>
-  <property name="pan_tilt_roll" value="0.0795383"/>
-  <property name="pan_tilt_pitch" value="-0.0104906"/>
-  <property name="pan_tilt_yaw" value="0.080464"/>
-  <!-- kinect mount positions | handeye calibration | relative to pan_tilt_link -->
-  <property name="kinect_x" value="-0.018782"/>
-  <property name="kinect_y" value="0.0683005"/>
-  <property name="kinect_z" value="-0.066483"/>
-  <property name="kinect_roll" value="-1.57387"/>
-  <property name="kinect_pitch" value="-0.0194537"/>
-  <property name="kinect_yaw" value="0.0357054"/>
+  <!-- shell mount positions | relative to base_link -->
+  <property name="shell_x" value="0.0"/>
+  <property name="shell_y" value="0.0"/>
+  <property name="shell_z" value="0.0"/>
+  <property name="shell_roll" value="0.0"/>
+  <property name="shell_pitch" value="0.0"/>
+  <property name="shell_yaw" value="0.0"/>
+  <!-- base_neck_link mount positions | camera base calibration | relative to base_link -->
+  <property name="base_neck_x" value="0.0"/>
+  <property name="base_neck_y" value="0.0"/>
+  <property name="base_neck_z" value="0.676"/>
+  <property name="base_neck_roll" value="0.0"/>
+  <property name="base_neck_pitch" value="0.0"/>
+  <property name="base_neck_yaw" value="0.0"/>
+  <!-- kinect mount positions | camera base calibration | relative to neck_tilt_link -->
+  <property name="kinect_x" value="0.0"/>
+  <property name="kinect_y" value="0.0"/>
+  <property name="kinect_z" value="0.0"/>
+  <property name="kinect_roll" value="-1.57"/>
+  <property name="kinect_pitch" value="0.0"/>
+  <property name="kinect_yaw" value="0.0"/>
   <!-- arm mount positions | handeye calibration | relative to base_link -->
   <property name="arm_x" value="0.0"/>

File: robotino_bringup/robots/uibk-robotino2/urdf/robotino-sh.urdf.xacro (robot description, xacro)
@@ -4,7 +4,7 @@
   <xacro:include filename="$(find robotino_bringup)/robots/uibk-robotino2/urdf/properties.urdf.xacro" />
   <xacro:include filename="$(find robotino_description)/urdf/base.urdf.xacro" />
+  <xacro:include filename="$(find robotino_description)/urdf/shell.urdf.xacro" />
   <xacro:include filename="$(find robotino_description)/urdf/hokuyo.urdf.xacro" />
   <xacro:include filename="$(find robotino_description)/urdf/kinect.urdf.xacro" />
-  <xacro:include filename="$(find robotino_description)/urdf/pan_tilt_axis.urdf.xacro" />
   <xacro:include filename="$(find robotino_description)/urdf/arm.urdf.xacro" />
   <xacro:include filename="$(find softhand_description)/model/softhand_withCableCanal.urdf.xacro" />
@@ -13,4 +13,13 @@
     <plugin name="ros_control" filename="libhwi_switch_gazebo_ros_control.so">
       <robotNamespace>base_controller</robotNamespace>
+      <filterJointsParam>joint_names</filterJointsParam>
+    </plugin>
+  </gazebo>
+  <xacro:shell name="shell" parent="base_linkz" base_neck_x="${base_neck_x}" base_neck_y="${base_neck_y}" base_neck_z="${base_neck_z}" base_neck_roll="${base_neck_roll}" base_neck_pitch="${base_neck_pitch}" base_neck_yaw="${base_neck_yaw}">
+    <origin xyz="${shell_x} ${shell_y} ${shell_z}" rpy="${shell_roll} ${shell_pitch} ${shell_yaw}"/>
+  </xacro:shell>
+  <gazebo>
+    <plugin name="ros_control" filename="libhwi_switch_gazebo_ros_control.so">
+      <robotNamespace>shell_controller</robotNamespace>
       <filterJointsParam>joint_names</filterJointsParam>
     </plugin>
@@ -37,15 +46,6 @@
     </plugin>
   </gazebo>
-  <pan_tilt_axis parent="base_linkz">
-    <origin xyz="${pan_tilt_x} ${pan_tilt_y} ${pan_tilt_z}" rpy="${pan_tilt_roll} ${pan_tilt_pitch} ${pan_tilt_yaw}"/>
-  </pan_tilt_axis>
-  <kinect name="kinect" parent="tilt_link">
+  <kinect name="kinect" parent="neck_tilt_link">
     <origin xyz="${kinect_x} ${kinect_y} ${kinect_z}" rpy="${kinect_roll} ${kinect_pitch} ${kinect_yaw}"/>
   </kinect>
-  <gazebo>
-    <plugin name="ros_control" filename="libhwi_switch_gazebo_ros_control.so">
-      <robotNamespace>pan_tilt_controller</robotNamespace>
-      <filterJointsParam>joint_names</filterJointsParam>
-    </plugin>
-  </gazebo>
 </robot>

File: robotino_bringup/robots/uibk-robotino2/urdf/robotino.urdf.xacro (robot description, xacro)
@@ -4,7 +4,7 @@
   <xacro:include filename="$(find robotino_bringup)/robots/uibk-robotino2/urdf/properties.urdf.xacro" />
   <xacro:include filename="$(find robotino_description)/urdf/base.urdf.xacro" />
+  <xacro:include filename="$(find robotino_description)/urdf/shell.urdf.xacro" />
   <xacro:include filename="$(find robotino_description)/urdf/hokuyo.urdf.xacro" />
   <xacro:include filename="$(find robotino_description)/urdf/kinect.urdf.xacro" />
-  <xacro:include filename="$(find robotino_description)/urdf/pan_tilt_axis.urdf.xacro" />
   <xacro:include filename="$(find robotino_description)/urdf/arm.urdf.xacro" />
   <xacro:include filename="$(find robotino_description)/urdf/kclhand_withCableCanal.urdf.xacro" />
@@ -13,4 +13,13 @@
     <plugin name="ros_control" filename="libhwi_switch_gazebo_ros_control.so">
       <robotNamespace>base_controller</robotNamespace>
+      <filterJointsParam>joint_names</filterJointsParam>
+    </plugin>
+  </gazebo>
+  <xacro:shell name="shell" parent="base_linkz" base_neck_x="${base_neck_x}" base_neck_y="${base_neck_y}" base_neck_z="${base_neck_z}" base_neck_roll="${base_neck_roll}" base_neck_pitch="${base_neck_pitch}" base_neck_yaw="${base_neck_yaw}">
+    <origin xyz="${shell_x} ${shell_y} ${shell_z}" rpy="${shell_roll} ${shell_pitch} ${shell_yaw}"/>
+  </xacro:shell>
+  <gazebo>
+    <plugin name="ros_control" filename="libhwi_switch_gazebo_ros_control.so">
+      <robotNamespace>shell_controller</robotNamespace>
       <filterJointsParam>joint_names</filterJointsParam>
     </plugin>
@@ -37,15 +46,6 @@
     </plugin>
   </gazebo>
-  <pan_tilt_axis parent="base_linkz">
-    <origin xyz="${pan_tilt_x} ${pan_tilt_y} ${pan_tilt_z}" rpy="${pan_tilt_roll} ${pan_tilt_pitch} ${pan_tilt_yaw}"/>
-  </pan_tilt_axis>
-  <kinect name="kinect" parent="tilt_link">
+  <kinect name="kinect" parent="neck_tilt_link">
     <origin xyz="${kinect_x} ${kinect_y} ${kinect_z}" rpy="${kinect_roll} ${kinect_pitch} ${kinect_yaw}"/>
   </kinect>
-  <gazebo>
-    <plugin name="ros_control" filename="libhwi_switch_gazebo_ros_control.so">
-      <robotNamespace>pan_tilt_controller</robotNamespace>
-      <filterJointsParam>joint_names</filterJointsParam>
-    </plugin>
-  </gazebo>
 </robot>
