Commit message: set 8 dof

File: robotino_bringup/robots/uibk-robotino2-sh/urdf/robotino_base_plan.urdf.xacro (robot description, xacro)
@@ -10,13 +10,4 @@
   <xacro:include filename="$(find soft_hand_description)/model/softhand_withCableCanal.urdf.xacro" />
   <xacro:base name="base" has_8dof="true"/>
-  <link name="origin">
-    <inertial>
-      <mass value="10" />
-      <origin xyz="0 0 0" />
-      <inertia ixx="75.0" ixy="0.0" ixz="0.0"
-        iyy="75.0" iyz="0.0"
-        izz="75.0" />
-    </inertial>
-  </link>
   <gazebo>
     <plugin name="ros_control" filename="libhwi_switch_gazebo_ros_control.so">

File: robotino_bringup/robots/uibk-robotino2/urdf/robotino.urdf (robot description, URDF)
Before this commit: robot robot, 34 links, 34 joints
Links:
- added link origin, mass 10
Joints:
- joint base_pan_joint: origin xyz=0.257201 0.0587815 0.637117 rpy=0.012045 -0.0565489 0.0113182 -> xyz=0.316119 0.00148515 0.693471 rpy=-3.14019 3.06888 3.121
- joint kinect_joint: origin xyz=0.0772857 0.117459 -0.0273189 rpy=1.57297 -3.11833 3.10173 -> xyz=-0.0198375 0.0584679 -0.065069 rpy=-1.57688 0.0102826 0.0812996
