Commit message: removed shell

File: robotino_bringup/robots/uibk-robotino2-sh/urdf/robotino.urdf.xacro (robot description, xacro)
@@ -17,7 +17,4 @@
     </plugin>
   </gazebo>
-  <xacro:shell name="base_shell" parent="base_link">
-    <origin xyz="0 0 0" rpy="0 0 0"/>
-  </xacro:shell>
   <hokuyo name="hokuyo" parent="base_link">
     <origin xyz="${hokuyo_x} ${hokuyo_y} ${hokuyo_z}" rpy="${hokuyo_roll} ${hokuyo_pitch} ${hokuyo_yaw}"/>
