Commit message: fixed model

File: robotino_bringup/robots/uibk-robotino2-sh/urdf/robotino.urdf (robot description, URDF)
Before this commit: robot robot, 60 links, 59 joints
Links:
- link hand_base_link: geometry collision mesh filename=package://soft_hand_description/meshes/robotino_softhand_ad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; visual mesh filename=package://soft_hand_description/meshes/robotino_softhand_ad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
- link hand_wrist_link: geometry collision mesh filename=package://soft_hand_description/meshes/wrist.stl; visual mesh filename=package://soft_hand_description/meshes/wrist.stl
Joints:
- joint hand_base_link_hand_clamp_joint: origin xyz=0 0 0.01 rpy=0 0 0 -> xyz=-0.02 -0.145 0.07 rpy=0 -0.7854 0

File: robotino_bringup/robots/uibk-robotino2-sh/urdf/robotino.urdf.xacro (robot description, xacro)
@@ -30,5 +30,5 @@
   </gazebo>
   <xacro:soft_hand name="hand" parent="arm_link5" withAdaptiveTransmission="false" useMimicTag="false" left="false">
-    <origin xyz="0 0 0" rpy="1.5707963 0 0" />
+    <origin xyz="0 0 0" rpy="0 0 0" />
   </xacro:soft_hand>
   <gazebo>

Commit message: THE (hopefully) working model

File: robotino_bringup/robots/uibk-robotino2-sh/urdf/robotino.urdf (robot description, URDF)
Before this commit: robot robot, 60 links, 59 joints
Links:
- added link origin, mass 10
Joints:
- added joint origin_joint: type prismatic, parent origin, child base_link, origin xyz=0 0 0 rpy=0 0 0, axis 1 0 0, limit lower=-10 upper=10 effort=190 velocity=30
- joint base_jointx: parent base_link -> origin
- joint hand_wrist_joint: origin xyz=0 0 0 rpy=1.5707963 0 0 -> xyz=0 0 0 rpy=0 0 0

File: robotino_bringup/robots/uibk-robotino2-sh/urdf/robotino_base_plan.urdf.xacro (robot description, xacro)
@@ -4,5 +4,5 @@
   <xacro:include filename="$(find robotino_bringup)/robots/uibk-robotino2/urdf/properties.urdf.xacro" />
   <xacro:include filename="$(find robotino_description)/urdf/gazebo.urdf.xacro" />
-  <xacro:include filename="$(find robotino_description)/urdf/base_plan.urdf.xacro" />
+  <xacro:include filename="$(find robotino_description)/urdf/base_plan_sh.urdf.xacro" />
   <xacro:include filename="$(find robotino_description)/urdf/hokuyo.urdf.xacro" />
   <xacro:include filename="$(find robotino_description)/urdf/kinect.urdf.xacro" />
@@ -11,4 +11,13 @@
   <xacro:include filename="$(find soft_hand_description)/model/softhand_withCableCanal.urdf.xacro" />
   <xacro:base name="base"/>
+  <link name="origin">
+    <inertial>
+      <mass value="10" />
+      <origin xyz="0 0 0" />
+      <inertia ixx="75.0" ixy="0.0" ixz="0.0"
+        iyy="75.0" iyz="0.0"
+        izz="75.0" />
+    </inertial>
+  </link>
   <gazebo>
     <plugin name="ros_control" filename="libhwi_switch_gazebo_ros_control.so">
@@ -30,5 +39,5 @@
   </gazebo>
   <xacro:soft_hand name="hand" parent="arm_link5" withAdaptiveTransmission="false" useMimicTag="false" left="false">
-    <origin xyz="0 0 0" rpy="1.5707963 0 0" />
+    <origin xyz="0 0 0" rpy="0 0 0" />
   </xacro:soft_hand>
   <gazebo>

Commit message: test model

File: robotino_bringup/robots/uibk-robotino2-sh/urdf/robotino.urdf (robot description, URDF)
Before this commit: robot robot, 60 links, 59 joints
Links:
- added link origin, mass 10
- link base_body_link: geometry collision mesh filename=package://robotino_description/meshes/RobotinoBody.stl; visual mesh filename=package://robotino_description/meshes/RobotinoBody.dae
- link base_linkx: mass 10 -> 0.01; geometry collision box size=0.001 0.001 0.001; visual box size=0.001 0.001 0.001
- link base_linky: mass 10 -> 0.01; geometry collision box size=0.001 0.001 0.001; visual box size=0.001 0.001 0.001
- link base_linkz: mass 10 -> 0.01; geometry collision box size=0.001 0.001 0.001; visual box size=0.001 0.001 0.001
Joints:
- added joint origin_joint: type prismatic, parent origin, child base_link, origin xyz=0 0 0 rpy=0 0 0, axis 1 0 0, limit lower=-10 upper=10 effort=190 velocity=30
- joint base_jointx: limit lower=-10 upper=10 effort=190 velocity=30 -> lower=-10 upper=10 effort=0 velocity=0; parent base_link -> origin
- joint base_jointy: limit lower=-10 upper=10 effort=190 velocity=30 -> lower=-10 upper=10 effort=0 velocity=0
- joint base_jointz: limit lower=-3.14 upper=3.14 effort=190 velocity=30 -> lower=-3.14 upper=3.14 effort=0 velocity=0
- joint hand_wrist_joint: origin xyz=0 0 0 rpy=1.5707963 0 0 -> xyz=0 0 0 rpy=0 0 0

File: robotino_bringup/robots/uibk-robotino2-sh/urdf/robotino.urdf.xacro (robot description, xacro)
@@ -9,5 +9,5 @@
   <xacro:include filename="$(find robotino_description)/urdf/arm.urdf.xacro" />
   <xacro:include filename="$(find soft_hand_description)/model/softhand_withCableCanal.urdf.xacro" />
-  <xacro:base name="base" has_8dof="true"/>
+  <xacro:base name="base" has_8dof="false"/>
   <gazebo>
     <plugin name="ros_control" filename="libhwi_switch_gazebo_ros_control.so">

File: robotino_bringup/robots/uibk-robotino2-sh/urdf/robotino_base_plan.urdf.xacro (robot description, xacro)
@@ -10,4 +10,13 @@
   <xacro:include filename="$(find soft_hand_description)/model/softhand_withCableCanal.urdf.xacro" />
   <xacro:base name="base" has_8dof="true"/>
+  <link name="origin">
+    <inertial>
+      <mass value="10" />
+      <origin xyz="0 0 0" />
+      <inertia ixx="75.0" ixy="0.0" ixz="0.0"
+        iyy="75.0" iyz="0.0"
+        izz="75.0" />
+    </inertial>
+  </link>
   <gazebo>
     <plugin name="ros_control" filename="libhwi_switch_gazebo_ros_control.so">
@@ -29,5 +38,5 @@
   </gazebo>
   <xacro:soft_hand name="hand" parent="arm_link5" withAdaptiveTransmission="false" useMimicTag="false" left="false">
-    <origin xyz="0 0 0" rpy="1.5707963 0 0" />
+    <origin xyz="0 0 0" rpy="0 0 0" />
   </xacro:soft_hand>
   <gazebo>

File: robotino_bringup/robots/uibk-robotino2/urdf/robotino.urdf (robot description, URDF)
Before this commit: robot robot, 34 links, 33 joints
Joints:
- added joint origin_joint: type prismatic, parent origin, child base_link, origin xyz=0 0 0 rpy=0 0 0, axis 1 0 0, limit lower=-10 upper=10 effort=190 velocity=30

Commit message: removed collision and visual parts of vi rtual joints

File: robotino_bringup/robots/uibk-robotino2-sh/urdf/robotino.urdf (robot description, URDF)
Before this commit: robot robot, 61 links, 60 joints
Links:
- link base_linkx: geometry 
- link base_linky: geometry 
- link base_linkz: geometry 

Commit message: simple base

File: robotino_bringup/robots/uibk-robotino2-sh/urdf/robotino.urdf (robot description, URDF)
Before this commit: robot robot, 61 links, 60 joints
Links:
- link base_body_link: geometry collision cylinder length=0.24 radius=0.23; visual mesh filename=package://robotino_description/meshes/RobotinoBody.dae

Commit message: final fixes from Simon Haller to get it running

File: robotino_bringup/robots/uibk-robotino2-sh/urdf/robotino.urdf (robot description, URDF)
Before this commit: robot robot, 61 links, 60 joints
Joints:
- joint hand_index_abd_joint: axis 0 0 1 -> (none); limit lower=-0.523598775598 upper=0.523598775598 effort=100 velocity=100 -> (none); type revolute -> fixed
- joint hand_index_inner_joint: axis 0 -1 0 -> (none); limit lower=0.0 upper=0.785398163397 effort=100 velocity=100 -> (none); type revolute -> fixed
- joint hand_index_inner_joint_mimic: axis 0 -1 0 -> (none); limit lower=0.0 upper=0.785398163397 effort=100 velocity=100 -> (none); type revolute -> fixed
- joint hand_index_middle_joint: axis 0 -1 0 -> (none); limit lower=0.0 upper=0.785398163397 effort=100 velocity=100 -> (none); type revolute -> fixed
- joint hand_index_middle_joint_mimic: axis 0 -1 0 -> (none); limit lower=0.0 upper=0.785398163397 effort=100 velocity=100 -> (none); type revolute -> fixed
- joint hand_index_outer_joint: axis 0 -1 0 -> (none); limit lower=0.0 upper=0.785398163397 effort=100 velocity=100 -> (none); type revolute -> fixed
- joint hand_index_outer_joint_mimic: axis 0 -1 0 -> (none); limit lower=0.0 upper=0.785398163397 effort=100 velocity=100 -> (none); type revolute -> fixed
- joint hand_little_abd_joint: axis 0 0 1 -> (none); limit lower=-0.523598775598 upper=0.523598775598 effort=100 velocity=100 -> (none); type revolute -> fixed
- joint hand_little_inner_joint: axis 0 -1 0 -> (none); limit lower=0.0 upper=0.785398163397 effort=100 velocity=100 -> (none); type revolute -> fixed
- joint hand_little_inner_joint_mimic: axis 0 -1 0 -> (none); limit lower=0.0 upper=0.785398163397 effort=100 velocity=100 -> (none); type revolute -> fixed
- joint hand_little_middle_joint: axis 0 -1 0 -> (none); limit lower=0.0 upper=0.785398163397 effort=100 velocity=100 -> (none); type revolute -> fixed
- joint hand_little_middle_joint_mimic: axis 0 -1 0 -> (none); limit lower=0.0 upper=0.785398163397 effort=100 velocity=100 -> (none); type revolute -> fixed
- joint hand_little_outer_joint: axis 0 -1 0 -> (none); limit lower=0.0 upper=0.785398163397 effort=100 velocity=100 -> (none); type revolute -> fixed
- joint hand_little_outer_joint_mimic: axis 0 -1 0 -> (none); limit lower=0.0 upper=0.785398163397 effort=100 velocity=100 -> (none); type revolute -> fixed
- joint hand_middle_abd_joint: axis 0 0 1 -> (none); limit lower=-0.523598775598 upper=0.523598775598 effort=100 velocity=100 -> (none); type revolute -> fixed
- joint hand_middle_inner_joint: axis 0 -1 0 -> (none); limit lower=0.0 upper=0.785398163397 effort=100 velocity=100 -> (none); type revolute -> fixed
- joint hand_middle_inner_joint_mimic: axis 0 -1 0 -> (none); limit lower=0.0 upper=0.785398163397 effort=100 velocity=100 -> (none); type revolute -> fixed
- joint hand_middle_middle_joint: axis 0 -1 0 -> (none); limit lower=0.0 upper=0.785398163397 effort=100 velocity=100 -> (none); type revolute -> fixed
- joint hand_middle_middle_joint_mimic: axis 0 -1 0 -> (none); limit lower=0.0 upper=0.785398163397 effort=100 velocity=100 -> (none); type revolute -> fixed
- joint hand_middle_outer_joint: axis 0 -1 0 -> (none); limit lower=0.0 upper=0.785398163397 effort=100 velocity=100 -> (none); type revolute -> fixed
- joint hand_middle_outer_joint_mimic: axis 0 -1 0 -> (none); limit lower=0.0 upper=0.785398163397 effort=100 velocity=100 -> (none); type revolute -> fixed
- joint hand_ring_abd_joint: axis 0 0 1 -> (none); limit lower=-0.523598775598 upper=0.523598775598 effort=100 velocity=100 -> (none); type revolute -> fixed
- joint hand_ring_inner_joint: axis 0 -1 0 -> (none); limit lower=0.0 upper=0.785398163397 effort=100 velocity=100 -> (none); type revolute -> fixed
- joint hand_ring_inner_joint_mimic: axis 0 -1 0 -> (none); limit lower=0.0 upper=0.785398163397 effort=100 velocity=100 -> (none); type revolute -> fixed
- joint hand_ring_middle_joint: axis 0 -1 0 -> (none); limit lower=0.0 upper=0.785398163397 effort=100 velocity=100 -> (none); type revolute -> fixed
- joint hand_ring_middle_joint_mimic: axis 0 -1 0 -> (none); limit lower=0.0 upper=0.785398163397 effort=100 velocity=100 -> (none); type revolute -> fixed
- joint hand_ring_outer_joint: axis 0 -1 0 -> (none); limit lower=0.0 upper=0.785398163397 effort=100 velocity=100 -> (none); type revolute -> fixed
- joint hand_ring_outer_joint_mimic: axis 0 -1 0 -> (none); limit lower=0.0 upper=0.785398163397 effort=100 velocity=100 -> (none); type revolute -> fixed
- joint hand_synergy_joint: axis 0 0 1 -> (none); limit lower=0.0 upper=1.0 effort=100 velocity=100000 -> (none); type revolute -> fixed
- joint hand_thumb_abd_joint: axis 0 0 -1 -> (none); limit lower=0.0 upper=1.57079632679 effort=100 velocity=100 -> (none); type revolute -> fixed
- joint hand_thumb_inner_joint: axis 0 -1 0 -> (none); limit lower=0.0 upper=0.785398163397 effort=100 velocity=100 -> (none); type revolute -> fixed
- joint hand_thumb_inner_joint_mimic: limit lower=0.0 upper=0.785398163397 effort=100 velocity=100 -> (none); type revolute -> fixed
- joint hand_thumb_outer_joint: axis 0 -1 0 -> (none); limit lower=0.0 upper=0.785398163397 effort=100 velocity=100 -> (none); type revolute -> fixed
- joint hand_thumb_outer_joint_mimic: axis 0 -1 0 -> (none); limit lower=0.0 upper=0.785398163397 effort=100 velocity=100 -> (none); type revolute -> fixed

Commit message: renamed soft_hand_description package to softhand_description

File: robotino_bringup/robots/uibk-robotino2-sh/urdf/robotino.urdf (robot description, URDF)
Before this commit: robot robot, 61 links, 60 joints
Links:
- link hand_base_link: geometry collision mesh filename=package://softhand_description/meshes/robotino_softhand_ada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; visual mesh filename=package://softhand_description/meshes/robotino_softhand_ada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
- link hand_clamp: geometry collision box size=0.066 0.0725 0.0256; visual mesh filename=package://softhand_description/meshes/accesories/clamp.stl
- link hand_index_distal_link: geometry collision mesh filename=package://softhand_description/meshes/fingertip_collision.s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 scale=.001 .001 .001; visual mesh filename=package://softhand_description/meshes/fingertip.stl scale=.001 .001 .001
- link hand_index_knuckle_link: geometry collision mesh filename=package://softhand_description/meshes/knuckle_collision.stl scale=.001 .001 .001; visual mesh filename=package://softhand_description/meshes/knuckle.stl scale=.001 .001 .001
- link hand_index_middle_link: geometry collision mesh filename=package://softhand_description/meshes/phalanx_collision.stl scale=.001 .001 .001; visual mesh filename=package://softhand_description/meshes/phalanx.stl scale=.001 .001 .001
- link hand_index_proximal_link: geometry collision mesh filename=package://softhand_description/meshes/phalanx_collision.stl scale=.001 .001 .001; visual mesh filename=package://softhand_description/meshes/phalanx.stl scale=.001 .001 .001
- link hand_little_distal_link: geometry collision mesh filename=package://softhand_description/meshes/fingertip_collision.s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 scale=.001 .001 .001; visual mesh filename=package://softhand_description/meshes/fingertip.stl scale=.001 .001 .001
- link hand_little_knuckle_link: geometry collision mesh filename=package://softhand_description/meshes/knuckle_collision.stl scale=.001 .001 .001; visual mesh filename=package://softhand_description/meshes/knuckle.stl scale=.001 .001 .001
- link hand_little_middle_link: geometry collision mesh filename=package://softhand_description/meshes/phalanx_collision.stl scale=.001 .001 .001; visual mesh filename=package://softhand_description/meshes/phalanx.stl scale=.001 .001 .001
- link hand_little_proximal_link: geometry collision mesh filename=package://softhand_description/meshes/phalanx_collision.stl scale=.001 .001 .001; visual mesh filename=package://softhand_description/meshes/phalanx.stl scale=.001 .001 .001
- link hand_middle_distal_link: geometry collision mesh filename=package://softhand_description/meshes/fingertip_collision.s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 scale=.001 .001 .001; visual mesh filename=package://softhand_description/meshes/fingertip.stl scale=.001 .001 .001
- link hand_middle_knuckle_link: geometry collision mesh filename=package://softhand_description/meshes/knuckle_collision.stl scale=.001 .001 .001; visual mesh filename=package://softhand_description/meshes/knuckle.stl scale=.001 .001 .001
- link hand_middle_middle_link: geometry collision mesh filename=package://softhand_description/meshes/phalanx_collision.stl scale=.001 .001 .001; visual mesh filename=package://softhand_description/meshes/phalanx.stl scale=.001 .001 .001
- link hand_middle_proximal_link: geometry collision mesh filename=package://softhand_description/meshes/phalanx_collision.stl scale=.001 .001 .001; visual mesh filename=package://softhand_description/meshes/phalanx.stl scale=.001 .001 .001
- link hand_palm_link: geometry collision mesh filename=package://softhand_description/meshes/palm_right_collision.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 scale=.001 .001 .001; visual mesh filename=package://softhand_description/meshes/palm_right.stl scale=.001 .001 .001
- link hand_ring_distal_link: geometry collision mesh filename=package://softhand_description/meshes/fingertip_collision.s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 scale=.001 .001 .001; visual mesh filename=package://softhand_description/meshes/fingertip.stl scale=.001 .001 .001
- link hand_ring_knuckle_link: geometry collision mesh filename=package://softhand_description/meshes/knuckle_collision.stl scale=.001 .001 .001; visual mesh filename=package://softhand_description/meshes/knuckle.stl scale=.001 .001 .001
- link hand_ring_middle_link: geometry collision mesh filename=package://softhand_description/meshes/phalanx_collision.stl scale=.001 .001 .001; visual mesh filename=package://softhand_description/meshes/phalanx.stl scale=.001 .001 .001
- link hand_ring_proximal_link: geometry collision mesh filename=package://softhand_description/meshes/phalanx_collision.stl scale=.001 .001 .001; visual mesh filename=package://softhand_description/meshes/phalanx.stl scale=.001 .001 .001
- link hand_softhand_base: geometry collision box size=0.066 0.066 0.062; visual mesh filename=package://softhand_description/meshes/accesories/softhand_b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
- link hand_thumb_distal_link: geometry collision mesh filename=package://softhand_description/meshes/fingertip_collision.s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 scale=.001 .001 .001; visual mesh filename=package://softhand_description/meshes/fingertip.stl scale=.001 .001 .001
- link hand_thumb_knuckle_link: geometry collision mesh filename=package://softhand_description/meshes/thumb_knuckle_right_c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 scale=.001 .001 .001; visual mesh filename=package://softhand_description/meshes/thumb_knuckle_right.s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 scale=.001 .001 .001
- link hand_thumb_proximal_link: geometry collision mesh filename=package://softhand_description/meshes/phalanx_collision.stl scale=.001 .001 .001; visual mesh filename=package://softhand_description/meshes/phalanx.stl scale=.001 .001 .001
- link hand_wrist_link: geometry collision mesh filename=package://softhand_description/meshes/wrist.stl; visual mesh filename=package://softhand_description/meshes/wrist.stl

File: robotino_bringup/robots/uibk-robotino2-sh/urdf/robotino.urdf.xacro (robot description, xacro)
@@ -8,5 +8,5 @@
   <xacro:include filename="$(find robotino_description)/urdf/pan_tilt_axis.urdf.xacro" />
   <xacro:include filename="$(find robotino_description)/urdf/arm.urdf.xacro" />
-  <xacro:include filename="$(find soft_hand_description)/model/softhand_withCableCanal.urdf.xacro" />
+  <xacro:include filename="$(find softhand_description)/model/softhand_withCableCanal.urdf.xacro" />
   <xacro:base name="base" has_8dof="false"/>
   <gazebo>

File: robotino_bringup/robots/uibk-robotino2-sh/urdf/robotino_base_plan.urdf.xacro (robot description, xacro)
@@ -8,5 +8,5 @@
   <xacro:include filename="$(find robotino_description)/urdf/pan_tilt_axis.urdf.xacro" />
   <xacro:include filename="$(find robotino_description)/urdf/arm.urdf.xacro" />
-  <xacro:include filename="$(find soft_hand_description)/model/softhand_withCableCanal.urdf.xacro" />
+  <xacro:include filename="$(find softhand_description)/model/softhand_withCableCanal.urdf.xacro" />
   <xacro:base name="base" has_8dof="true"/>
   <gazebo>

Commit message: added shell

File: robotino_bringup/robots/uibk-robotino2-sh/urdf/robotino.urdf (robot description, URDF)
Before this commit: robot robot, 61 links, 60 joints
Links:
- added link base_shell_link, mass 4; collision mesh filename=package://robotino_description/meshes/base_shell_collision.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; visual mesh filename=package://robotino_description/meshes/squirrel_assembly.stl
Joints:
- added joint base_shell_joint: type fixed, parent base_link, child base_shell_link, origin xyz=0 0 0 rpy=0 0 0
- joint base_pan_joint: origin xyz=0.257201 0.0587815 0.637117 rpy=0.012045 -0.0565489 0.0113182 -> xyz=0.319612 -0.0356507 0.687939 rpy=0.037253 0.0665136 0.0628319
- joint hokuyo_joint: origin xyz=0.208610627 0.0 0.095 rpy=0.0 0.0 0.0 -> xyz=0.208610627 0.0 0.14 rpy=0.0 0.0 0.0
- joint kinect_joint: origin xyz=0.0772857 0.117459 -0.0273189 rpy=1.57297 -3.11833 3.10173 -> xyz=-0.0221115 0.0645073 -0.065954 rpy=-1.57413 -0.00632857 0.0520659

File: robotino_bringup/robots/uibk-robotino2-sh/urdf/robotino.urdf.xacro (robot description, xacro)
@@ -6,4 +6,5 @@
   <xacro:include filename="$(find robotino_description)/urdf/hokuyo.urdf.xacro" />
   <xacro:include filename="$(find robotino_description)/urdf/kinect.urdf.xacro" />
+  <xacro:include filename="$(find robotino_description)/urdf/base_shell.urdf.xacro" />
   <xacro:include filename="$(find robotino_description)/urdf/pan_tilt_axis.urdf.xacro" />
   <xacro:include filename="$(find robotino_description)/urdf/arm.urdf.xacro" />
@@ -16,4 +17,7 @@
     </plugin>
   </gazebo>
+  <xacro:shell name="base_shell" parent="base_link">
+    <origin xyz="0 0 0" rpy="0 0 0"/>
+  </xacro:shell>
   <hokuyo name="hokuyo" parent="base_link">
     <origin xyz="${hokuyo_x} ${hokuyo_y} ${hokuyo_z}" rpy="${hokuyo_roll} ${hokuyo_pitch} ${hokuyo_yaw}"/>

File: robotino_bringup/robots/uibk-robotino2-sh/urdf/robotino_base_plan.urdf.xacro (robot description, xacro)
@@ -5,4 +5,5 @@
   <xacro:include filename="$(find robotino_description)/urdf/base.urdf.xacro" />
   <xacro:include filename="$(find robotino_description)/urdf/hokuyo.urdf.xacro" />
+  <xacro:include filename="$(find robotino_description)/urdf/base_shell.urdf.xacro" />
   <xacro:include filename="$(find robotino_description)/urdf/kinect.urdf.xacro" />
   <xacro:include filename="$(find robotino_description)/urdf/pan_tilt_axis.urdf.xacro" />
@@ -16,4 +17,7 @@
     </plugin>
   </gazebo>
+  <xacro:shell name="base_shell" parent="base_link">
+    <origin xyz="0 0 0" rpy="0 0 0"/>
+  </xacro:shell>
   <hokuyo name="hokuyo" parent="base_linkz">
     <origin xyz="${hokuyo_x} ${hokuyo_y} ${hokuyo_z}" rpy="${hokuyo_roll} ${hokuyo_pitch} ${hokuyo_yaw}"/>

Commit message: fixed model according to Nadia's comment

File: robotino_bringup/robots/uibk-robotino2-sh/urdf/robotino.urdf (robot description, URDF)
Before this commit: robot robot, 62 links, 61 joints
Links:
- removed link base_shell_link
Joints:
- removed joint base_shell_joint

File: robotino_bringup/robots/uibk-robotino2-sh/urdf/robotino.urdf.xacro (robot description, xacro)
@@ -6,9 +6,8 @@
   <xacro:include filename="$(find robotino_description)/urdf/hokuyo.urdf.xacro" />
   <xacro:include filename="$(find robotino_description)/urdf/kinect.urdf.xacro" />
-  <xacro:include filename="$(find robotino_description)/urdf/base_shell.urdf.xacro" />
   <xacro:include filename="$(find robotino_description)/urdf/pan_tilt_axis.urdf.xacro" />
   <xacro:include filename="$(find robotino_description)/urdf/arm.urdf.xacro" />
   <xacro:include filename="$(find softhand_description)/model/softhand_withCableCanal.urdf.xacro" />
-  <xacro:base name="base" has_8dof="true"/>
+  <xacro:base name="base" has_8dof="false"/>
   <gazebo>
     <plugin name="ros_control" filename="libhwi_switch_gazebo_ros_control.so">

File: robotino_bringup/robots/uibk-robotino2-sh/urdf/robotino_base_plan.urdf.xacro (robot description, xacro)
@@ -17,7 +17,4 @@
     </plugin>
   </gazebo>
-  <xacro:shell name="base_shell" parent="base_link">
-    <origin xyz="0 0 0" rpy="0 0 0"/>
-  </xacro:shell>
   <hokuyo name="hokuyo" parent="base_linkz">
     <origin xyz="${hokuyo_x} ${hokuyo_y} ${hokuyo_z}" rpy="${hokuyo_roll} ${hokuyo_pitch} ${hokuyo_yaw}"/>
