Commit message: now uses robotino.urdf from correct robotino_base_link.urdf.xacro

File: robotino_bringup/robots/tuw-robotino2/urdf/robotino.urdf (robot description, URDF)
Before this commit: robot robot, 35 links, 34 joints
Links:
- link profile_link: geometry collision mesh filename=package://robotino_description/meshes/pan_tilt.stl; visual mesh filename=package://robotino_description/meshes/pan_tilt.stl
Joints:
- joint arm_base_joint: parent base_link -> base_linkz
- joint hokuyo_joint: parent base_link -> base_linkz
- joint profile_joint: parent base_link -> base_linkz

Commit message: update squirrel_robots to the new kclhand structure

File: robotino_bringup/robots/tuw-robotino2/urdf/robotino.urdf (robot description, URDF)
Before this commit: robot robot, 35 links, 34 joints
Links:
- link hand_base_link: geometry collision mesh filename=package://robotino_description/meshes/kclhand/base_link.STL; visual mesh filename=package://robotino_description/meshes/kclhand/base_link.STL
- link hand_cableCanal_link: geometry collision mesh filename=package://robotino_description/meshes/kclhand/cableCanalCol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; visual box size=0.0 0.0 0.0
- link hand_left_coupler: geometry collision mesh filename=package://robotino_description/meshes/kclhand/left_coupler.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; visual mesh filename=package://robotino_description/meshes/kclhand/left_coupler.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
- link hand_left_crank: geometry collision mesh filename=package://robotino_description/meshes/kclhand/left_crank.STL; visual mesh filename=package://robotino_description/meshes/kclhand/left_crank.STL
- link hand_left_finger_lower_link: geometry collision mesh filename=package://robotino_description/meshes/kclhand/left_finger_l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; visual mesh filename=package://robotino_description/meshes/kclhand/left_finger_l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
- link hand_left_finger_upper_link: geometry collision mesh filename=package://robotino_description/meshes/kclhand/left_finger_u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; visual mesh filename=package://robotino_description/meshes/kclhand/left_finger_u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
- link hand_middle_finger_lower_link: geometry collision mesh filename=package://robotino_description/meshes/kclhand/middle_finger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; visual mesh filename=package://robotino_description/meshes/kclhand/middle_finger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
- link hand_middle_finger_upper_link: geometry collision mesh filename=package://robotino_description/meshes/kclhand/middle_finger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; visual mesh filename=package://robotino_description/meshes/kclhand/middle_finger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
- link hand_right_coupler: geometry collision mesh filename=package://robotino_description/meshes/kclhand/right_coupler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; visual mesh filename=package://robotino_description/meshes/kclhand/right_coupler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
- link hand_right_crank: geometry collision mesh filename=package://robotino_description/meshes/kclhand/right_crank.S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; visual mesh filename=package://robotino_description/meshes/kclhand/right_crank.S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
- link hand_right_finger_lower_link: geometry collision mesh filename=package://robotino_description/meshes/kclhand/right_finger_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; visual mesh filename=package://robotino_description/meshes/kclhand/right_finger_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
- link hand_right_finger_upper_link: geometry collision mesh filename=package://robotino_description/meshes/kclhand/right_finger_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; visual mesh filename=package://robotino_description/meshes/kclhand/right_finger_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
- link hand_wrist_link: geometry collision mesh filename=package://robotino_description/meshes/kclhand/wrist.stl; visual mesh filename=package://robotino_description/meshes/kclhand/wrist.stl

File: robotino_bringup/robots/uibk-robotino2/urdf/robotino.urdf (robot description, URDF)
Before this commit: robot robot, 35 links, 34 joints
Links:
- link hand_base_link: geometry collision mesh filename=package://robotino_description/meshes/kclhand/base_link.STL; visual mesh filename=package://robotino_description/meshes/kclhand/base_link.STL
- link hand_cableCanal_link: geometry collision mesh filename=package://robotino_description/meshes/kclhand/cableCanalCol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; visual box size=0.0 0.0 0.0
- link hand_left_coupler: geometry collision mesh filename=package://robotino_description/meshes/kclhand/left_coupler.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; visual mesh filename=package://robotino_description/meshes/kclhand/left_coupler.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
- link hand_left_crank: geometry collision mesh filename=package://robotino_description/meshes/kclhand/left_crank.STL; visual mesh filename=package://robotino_description/meshes/kclhand/left_crank.STL
- link hand_left_finger_lower_link: geometry collision mesh filename=package://robotino_description/meshes/kclhand/left_finger_l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; visual mesh filename=package://robotino_description/meshes/kclhand/left_finger_l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
- link hand_left_finger_upper_link: geometry collision mesh filename=package://robotino_description/meshes/kclhand/left_finger_u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; visual mesh filename=package://robotino_description/meshes/kclhand/left_finger_u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
- link hand_middle_finger_lower_link: geometry collision mesh filename=package://robotino_description/meshes/kclhand/middle_finger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; visual mesh filename=package://robotino_description/meshes/kclhand/middle_finger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
- link hand_middle_finger_upper_link: geometry collision mesh filename=package://robotino_description/meshes/kclhand/middle_finger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; visual mesh filename=package://robotino_description/meshes/kclhand/middle_finger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
- link hand_right_coupler: geometry collision mesh filename=package://robotino_description/meshes/kclhand/right_coupler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; visual mesh filename=package://robotino_description/meshes/kclhand/right_coupler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
- link hand_right_crank: geometry collision mesh filename=package://robotino_description/meshes/kclhand/right_crank.S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; visual mesh filename=package://robotino_description/meshes/kclhand/right_crank.S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
- link hand_right_finger_lower_link: geometry collision mesh filename=package://robotino_description/meshes/kclhand/right_finger_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; visual mesh filename=package://robotino_description/meshes/kclhand/right_finger_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
- link hand_right_finger_upper_link: geometry collision mesh filename=package://robotino_description/meshes/kclhand/right_finger_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; visual mesh filename=package://robotino_description/meshes/kclhand/right_finger_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
- link hand_wrist_link: geometry collision mesh filename=package://robotino_description/meshes/kclhand/wrist.stl; visual mesh filename=package://robotino_description/meshes/kclhand/wrist.stl

Commit message: changed back, I have no idea what I am doing.

File: robotino_bringup/robots/tuw-robotino2/urdf/robotino.urdf (robot description, URDF)
Before this commit: robot robot, 35 links, 34 joints
Links:
- link profile_link: geometry collision mesh filename=package://robotino_description/meshes/pan_tilt_tuw.stl; visual mesh filename=package://robotino_description/meshes/pan_tilt_tuw.stl
Joints:
- joint arm_base_joint: parent base_linkz -> base_link
- joint hokuyo_joint: parent base_linkz -> base_link
- joint profile_joint: parent base_linkz -> base_link

Commit message: restore the base_linkz tree for moveit

File: robotino_bringup/robots/tuw-robotino2/urdf/robotino.urdf (robot description, URDF)
Before this commit: robot robot, 35 links, 34 joints
Joints:
- joint arm_base_joint: parent base_link -> base_linkz
- joint hokuyo_joint: parent base_link -> base_linkz
- joint profile_joint: parent base_link -> base_linkz

Commit message: removed soft limits in tuw robotino. tested. working

File: robotino_bringup/robots/tuw-robotino2/urdf/robotino.urdf (robot description, URDF)
Before this commit: robot robot, 35 links, 34 joints
Joints:
- joint arm_joint1: limit lower=-1.9 upper=1.9 effort=190 velocity=30 -> lower=-1.2 upper=1.5 effort=190 velocity=30
- joint arm_joint2: limit lower=-1.9 upper=1.9 effort=190 velocity=30 -> lower=-1.7 upper=2.3 effort=190 velocity=30
- joint arm_joint3: limit lower=-1.7 upper=1.7 effort=190 velocity=30 -> lower=-1.8 upper=1.8 effort=190 velocity=30
- joint arm_joint4: limit lower=-1.7 upper=1.7 effort=160 velocity=30 -> lower=-1.9 upper=1.9 effort=160 velocity=30
- joint arm_joint5: limit lower=-1.7 upper=1.7 effort=160 velocity=30 -> lower=-2.9 upper=2.9 effort=160 velocity=30
- joint base_jointx: limit lower=-10 upper=10 effort=0 velocity=0 -> lower=-20 upper=20 effort=0 velocity=0
- joint base_jointy: limit lower=-10 upper=10 effort=0 velocity=0 -> lower=-20 upper=20 effort=0 velocity=0
- joint origin_joint: limit lower=-10 upper=10 effort=190 velocity=30 -> lower=-20 upper=20 effort=190 velocity=30
