Commit message: added a collision case

File: robotino_bringup/robots/tuw-robotino2/urdf/robotino.urdf.xacro (robot description, xacro)
@@ -5,4 +5,5 @@
   <xacro:include filename="$(find robotino_description)/urdf/gazebo.urdf.xacro" />
   <xacro:include filename="$(find robotino_description)/urdf/robotino_body.urdf.xacro" />
+  <xacro:include filename="$(find robotino_description)/urdf/base_case.urdf.xacro" />
   <xacro:include filename="$(find robotino_description)/urdf/rotatory.urdf.xacro" />
   <xacro:include filename="$(find robotino_description)/urdf/hokuyo.urdf.xacro" />
@@ -27,4 +28,7 @@
     <origin xyz="${hokuyo_x} ${hokuyo_y} ${hokuyo_z}" rpy="${hokuyo_roll} ${hokuyo_pitch} ${hokuyo_yaw}"/>
   </hokuyo>
+  <case name="case" parent="base_link">
+    <origin xyz="0 0 0" rpy="0 0 0"/>
+  </case>
   <xacro:rotatory />
   <gazebo>

File: robotino_bringup/robots/uibk-robotino2/urdf/robotino.urdf.xacro (robot description, xacro)
@@ -5,4 +5,5 @@
   <xacro:include filename="$(find robotino_description)/urdf/gazebo.urdf.xacro" />
   <xacro:include filename="$(find robotino_description)/urdf/robotino_body.urdf.xacro" />
+  <xacro:include filename="$(find robotino_description)/urdf/base_case.urdf.xacro" />
   <xacro:include filename="$(find robotino_description)/urdf/rotatory.urdf.xacro" />
   <xacro:include filename="$(find robotino_description)/urdf/hokuyo.urdf.xacro" />
@@ -18,7 +19,16 @@
     </plugin>
   </gazebo>
+  <gazebo>
+    <plugin name="ros_control" filename="libhwi_switch_gazebo_ros_control.so">
+      <robotNamespace>base_controller</robotNamespace>
+      <filterJointsParam>joint_names</filterJointsParam>
+    </plugin>
+  </gazebo>
   <hokuyo name="hokuyo" parent="base_link">
     <origin xyz="${hokuyo_x} ${hokuyo_y} ${hokuyo_z}" rpy="${hokuyo_roll} ${hokuyo_pitch} ${hokuyo_yaw}"/>
   </hokuyo>
+  <case name="case" parent="base_link">
+    <origin xyz="0 0 0" rpy="0 0 0"/>
+  </case>
   <xacro:rotatory />
   <gazebo>

Commit message: case

File: robotino_bringup/robots/tuw-robotino2/urdf/robotino.urdf.xacro (robot description, xacro)
@@ -28,7 +28,7 @@
     <origin xyz="${hokuyo_x} ${hokuyo_y} ${hokuyo_z}" rpy="${hokuyo_roll} ${hokuyo_pitch} ${hokuyo_yaw}"/>
   </hokuyo>
-  <case name="case" parent="base_link">
-    <origin xyz="0 0 0" rpy="0 0 0"/>
-  </case>
+  <!--case name="case" parent="base_link">
+    <origin xyz="0 0 0" rpy="0 0 -0.5"/>
+  </case-->
   <xacro:rotatory />
   <gazebo>

File: robotino_bringup/robots/uibk-robotino2/urdf/robotino.urdf.xacro (robot description, xacro)
@@ -28,7 +28,7 @@
     <origin xyz="${hokuyo_x} ${hokuyo_y} ${hokuyo_z}" rpy="${hokuyo_roll} ${hokuyo_pitch} ${hokuyo_yaw}"/>
   </hokuyo>
-  <case name="case" parent="base_link">
+  <!--case name="case" parent="base_link">
     <origin xyz="0 0 0" rpy="0 0 -0.5"/>
-  </case>
+  </case-->
   <xacro:rotatory />
   <gazebo>

Commit message: added shell model to tuw-robotino-2

File: robotino_bringup/robots/tuw-robotino2/urdf/robotino.urdf.xacro (robot description, xacro)
@@ -4,4 +4,5 @@
   <xacro:include filename="$(find robotino_bringup)/robots/tuw-robotino2/urdf/properties.urdf.xacro" />
   <xacro:include filename="$(find robotino_description)/urdf/base.urdf.xacro" />
+  <xacro:include filename="$(find robotino_description)/urdf/base_shell.urdf.xacro" />
   <xacro:include filename="$(find robotino_description)/urdf/hokuyo.urdf.xacro" />
   <xacro:include filename="$(find robotino_description)/urdf/kinect.urdf.xacro" />
@@ -9,5 +10,5 @@
   <xacro:include filename="$(find robotino_description)/urdf/arm.urdf.xacro" />
   <xacro:include filename="$(find robotino_description)/urdf/kclhand_withCableCanal.urdf.xacro" />
-  <xacro:base name="base" has_8dof="true"/>
+  <xacro:base name="base" has_8dof="false"/>
   <gazebo>
     <plugin name="ros_control" filename="libhwi_switch_gazebo_ros_control.so">
@@ -16,4 +17,7 @@
     </plugin>
   </gazebo>
+  <xacro:shell name="base_shell" parent="base_link">
+    <origin xyz="0 0 0" rpy="0 0 0"/>
+  </xacro:shell>
   <hokuyo name="hokuyo" parent="base_link">
     <origin xyz="${hokuyo_x} ${hokuyo_y} ${hokuyo_z}" rpy="${hokuyo_roll} ${hokuyo_pitch} ${hokuyo_yaw}"/>

Commit message: the position of the shell should depend on the position of the scan

File: robotino_bringup/robots/tuw-robotino2/urdf/robotino.urdf.xacro (robot description, xacro)
@@ -18,5 +18,5 @@
   </gazebo>
   <xacro:shell name="base_shell" parent="base_link">
-    <origin xyz="0 0 0" rpy="0 0 0"/>
+    <origin xyz="0 0 ${hokuyo_z-0.13}" rpy="0 0 0"/>
   </xacro:shell>
   <hokuyo name="hokuyo" parent="base_link">
