Commit message: updated model

File: robotino_bringup/robots/tuw-robotino2/urdf/properties.urdf.xacro (robot description, xacro)
@@ -29,10 +29,10 @@
   <property name="hokuyo_yaw" value="0.0"/>
    <!-- pan_tilt mount positions | handeye calibration | relative to base_link -->
-  <property name="pan_tilt_x" value="0.25"/>
-  <property name="pan_tilt_y" value="0.0"/>
+  <property name="pan_tilt_x" value="0.203"/>
+  <property name="pan_tilt_y" value="0.003"/>
   <property name="pan_tilt_z" value="0.55"/>
   <property name="pan_tilt_roll" value="0"/>
   <property name="pan_tilt_pitch" value="0"/> <!--${M_PI/2}"/> -->
-  <property name="pan_tilt_yaw" value="0"/>
+  <property name="pan_tilt_yaw" value="0.0"/>
   <!-- kinect mount positions | handeye calibration | relative to pan_tilt_link -->
   <property name="kinect_x" value="0.0"/>

File: robotino_description/urdf/pan_tilt_axis.urdf.xacro (robot description, xacro)
@@ -2,7 +2,33 @@
 <root xmlns:xacro="http://www.ros.org/wiki/xacro">
   <xacro:macro name="pan_tilt_axis" params="parent *origin">
-    <joint name="pan_joint" type="revolute">
+    <joint name="base_pan_joint" type="fixed">
       <insert_block name="origin" />
       <parent link="${parent}"/>
+      <child link="base_pan_link" />
+    </joint>
+    <link name="base_pan_link">
+      <inertial>
+        <mass value="0.00001" />
+        <origin xyz="0 0 0" />
+        <inertia ixx="1.0" ixy="0.0" ixz="0.0"
+          iyy="1.0" iyz="0.0"
+          izz="1.0" />
+      </inertial>
+      <visual>
+        <origin xyz="0 0 0" rpy="0 0 0" />
+        <geometry>
+          <mesh filename="package://robotino_description/meshes/pan_tilt.stl"/>
+        </geometry>
+      </visual>
+      <collision>
+        <origin xyz="0 0 0" rpy="0 0 0" />
+        <geometry>
+          <mesh filename="package://robotino_description/meshes/pan_tilt.stl"/>
+        </geometry>
+      </collision>
+    </link>
+    <joint name="pan_joint" type="revolute">
+			<origin xyz="0 0 0" rpy="0 0 0"/>
+      <parent link="base_pan_link"/>
       <child link="pan_link" />
       <axis xyz="0 0 1" />

Commit message: addapted simulation to new arm driver

File: robotino_bringup/robots/tuw-robotino2/urdf/properties.urdf.xacro (robot description, xacro)
@@ -44,6 +44,6 @@
    <!-- arm mount positions | handeye calibration | relative to base_link -->
   <property name="arm_x" value="0.0"/>
-  <property name="arm_y" value="0.0"/>
-  <property name="arm_z" value="0.35"/>
+  <property name="arm_y" value="-0.01591"/>
+  <property name="arm_z" value="0.32"/>
   <property name="arm_roll" value="0.0"/>
   <property name="arm_pitch" value="0.0"/>

File: robotino_bringup/robots/tuw-robotino2/urdf/robotino.urdf.xacro (robot description, xacro)
@@ -10,13 +10,7 @@
   <xacro:include filename="$(find robotino_description)/urdf/kinect.urdf.xacro" />
   <xacro:include filename="$(find robotino_description)/urdf/pan_tilt_tuw_axis.urdf.xacro" />
-  <xacro:include filename="$(find robotino_arm_description)/xacro/arm_model.urdf.xacro" />
+  <xacro:include filename="$(find robotino_description)/urdf/arm.urdf.xacro" />
   <xacro:include filename="$(find kclhand_description)/urdf/kclhand_withCableCanal.urdf.xacro" />
   <xacro:body name="base"/>
-  <gazebo>
-    <plugin name="ros_control" filename="libhwi_switch_gazebo_ros_control.so">
-      <robotNamespace>base_controller</robotNamespace>
-      <filterJointsParam>joint_names</filterJointsParam>
-    </plugin>
-  </gazebo>
   <gazebo>
     <plugin name="ros_control" filename="libhwi_switch_gazebo_ros_control.so">
@@ -28,15 +22,7 @@
     <origin xyz="${hokuyo_x} ${hokuyo_y} ${hokuyo_z}" rpy="${hokuyo_roll} ${hokuyo_pitch} ${hokuyo_yaw}"/>
   </hokuyo>
-  <!--case name="case" parent="base_link">
-    <origin xyz="0 0 0" rpy="0 0 -0.5"/>
-  </case-->
-  <xacro:rotatory />
-  <gazebo>
-    <plugin name="ros_control" filename="libhwi_switch_gazebo_ros_control.so">
-      <robotNamespace>rotatory_controller</robotNamespace>
-      <filterJointsParam>joint_names</filterJointsParam>
-    </plugin>
-  </gazebo>
-  <xacro:arm />
+  <xacro:arm name="arm_" parent="base_link">
+    <origin xyz="${arm_x} ${arm_y} ${arm_z}" rpy="${arm_roll} ${arm_pitch} ${arm_yaw}"/>
+  </xacro:arm>
   <gazebo>
     <plugin name="ros_control" filename="libhwi_switch_gazebo_ros_control.so">
@@ -45,5 +31,5 @@
     </plugin>
   </gazebo>
-  <xacro:kclhand name="hand" parent="link5">
+  <xacro:kclhand name="hand" parent="arm_link5">
     <origin xyz="0 0 0" rpy="1.5707963 0 0" />
   </xacro:kclhand>

File: robotino_bringup/robots/uibk-robotino2/urdf/properties.urdf.xacro (robot description, xacro)
@@ -44,6 +44,6 @@
    <!-- arm mount positions | handeye calibration | relative to base_link -->
   <property name="arm_x" value="0.0"/>
-  <property name="arm_y" value="0.0"/>
-  <property name="arm_z" value="0.35"/>
+  <property name="arm_y" value="-0.01591"/>
+  <property name="arm_z" value="0.32"/>
   <property name="arm_roll" value="0.0"/>
   <property name="arm_pitch" value="0.0"/>

File: robotino_bringup/robots/uibk-robotino2/urdf/robotino.urdf.xacro (robot description, xacro)
@@ -10,13 +10,7 @@
   <xacro:include filename="$(find robotino_description)/urdf/kinect.urdf.xacro" />
   <xacro:include filename="$(find robotino_description)/urdf/pan_tilt_axis.urdf.xacro" />
-  <xacro:include filename="$(find robotino_arm_description)/xacro/arm_model.urdf.xacro" />
+  <xacro:include filename="$(find robotino_description)/urdf/arm.urdf.xacro" />
   <xacro:include filename="$(find kclhand_description)/urdf/kclhand_withCableCanal.urdf.xacro" />
   <xacro:body name="base"/>
-  <gazebo>
-    <plugin name="ros_control" filename="libhwi_switch_gazebo_ros_control.so">
-      <robotNamespace>base_controller</robotNamespace>
-      <filterJointsParam>joint_names</filterJointsParam>
-    </plugin>
-  </gazebo>
   <gazebo>
     <plugin name="ros_control" filename="libhwi_switch_gazebo_ros_control.so">
@@ -28,15 +22,7 @@
     <origin xyz="${hokuyo_x} ${hokuyo_y} ${hokuyo_z}" rpy="${hokuyo_roll} ${hokuyo_pitch} ${hokuyo_yaw}"/>
   </hokuyo>
-  <!--case name="case" parent="base_link">
-    <origin xyz="0 0 0" rpy="0 0 -0.5"/>
-  </case-->
-  <xacro:rotatory />
-  <gazebo>
-    <plugin name="ros_control" filename="libhwi_switch_gazebo_ros_control.so">
-      <robotNamespace>rotatory_controller</robotNamespace>
-      <filterJointsParam>joint_names</filterJointsParam>
-    </plugin>
-  </gazebo>
-  <xacro:arm />
+  <xacro:arm name="arm_" parent="base_link">
+    <origin xyz="${arm_x} ${arm_y} ${arm_z}" rpy="${arm_roll} ${arm_pitch} ${arm_yaw}"/>
+  </xacro:arm>
   <gazebo>
     <plugin name="ros_control" filename="libhwi_switch_gazebo_ros_control.so">
@@ -45,5 +31,5 @@
     </plugin>
   </gazebo>
-  <xacro:kclhand name="hand" parent="link5">
+  <xacro:kclhand name="hand" parent="arm_link5">
     <origin xyz="0 0 0" rpy="1.5707963 0 0" />
   </xacro:kclhand>

Commit message: launch file can not work, motors are running on raspberry

File: robotino_bringup/robots/tuw-robotino2/urdf/properties.urdf.xacro (robot description, xacro)
@@ -21,18 +21,11 @@
   <property name="hokuyo_pitch" value="0.0"/>
   <property name="hokuyo_yaw" value="-0.015"/>
-  <!-- pan_tilt mount positions | handeye calibration | relative to base_link -->
-  <property name="pan_tilt_x" value="0.258758"/>
-  <property name="pan_tilt_y" value="-0.0038856"/>
-  <property name="pan_tilt_z" value="0.655646"/>
-  <property name="pan_tilt_roll" value="0.0233953"/>
-  <property name="pan_tilt_pitch" value="-0.0360962"/>
-  <property name="pan_tilt_yaw" value="0.00901179"/>
   <!-- kinect mount positions | handeye calibration | relative to pan_tilt_link -->
-  <property name="kinect_x" value="-0.0300317"/>
-  <property name="kinect_y" value="0.0603655"/>
-  <property name="kinect_z" value="-0.0649396"/>
-  <property name="kinect_roll" value="1.582"/>
-  <property name="kinect_pitch" value="3.11972"/>
-  <property name="kinect_yaw" value="3.12919"/>
+  <property name="kinect_x" value="0.0"/>
+  <property name="kinect_y" value="0.0"/>
+  <property name="kinect_z" value="0.0"/>
+  <property name="kinect_roll" value="-1.57"/>
+  <property name="kinect_pitch" value="0"/>
+  <property name="kinect_yaw" value="0"/>
   <!-- arm mount positions | handeye calibration | relative to base_link -->
   <property name="arm_x" value="0.0"/>

File: robotino_bringup/robots/tuw-robotino2/urdf/robotino.urdf.xacro (robot description, xacro)
@@ -4,8 +4,7 @@
   <xacro:include filename="$(find robotino_bringup)/robots/tuw-robotino2/urdf/properties.urdf.xacro" />
   <xacro:include filename="$(find robotino_description)/urdf/base.urdf.xacro" />
-  <xacro:include filename="$(find robotino_description)/urdf/base_shell.urdf.xacro" />
+  <xacro:include filename="$(find robotino_description)/urdf/shell.urdf.xacro" />
   <xacro:include filename="$(find robotino_description)/urdf/hokuyo.urdf.xacro" />
   <xacro:include filename="$(find robotino_description)/urdf/kinect.urdf.xacro" />
-  <xacro:include filename="$(find robotino_description)/urdf/pan_tilt_tuw_axis.urdf.xacro" />
   <xacro:include filename="$(find robotino_description)/urdf/arm.urdf.xacro" />
   <xacro:include filename="$(find robotino_description)/urdf/kclhand_withCableCanal.urdf.xacro" />
@@ -17,7 +16,4 @@
     </plugin>
   </gazebo>
-  <xacro:shell name="base_shell" parent="base_link">
-    <origin xyz="0 0 ${hokuyo_z-0.13}" rpy="0 0 0"/>
-  </xacro:shell>
   <hokuyo name="hokuyo" parent="base_linkz">
     <origin xyz="${hokuyo_x} ${hokuyo_y} ${hokuyo_z}" rpy="${hokuyo_roll} ${hokuyo_pitch} ${hokuyo_yaw}"/>
@@ -41,15 +37,9 @@
     </plugin>
   </gazebo>
-  <pan_tilt_axis parent="base_linkz">
-    <origin xyz="${pan_tilt_x} ${pan_tilt_y} ${pan_tilt_z}" rpy="${pan_tilt_roll} ${pan_tilt_pitch} ${pan_tilt_yaw}"/>
-  </pan_tilt_axis>
-  <kinect name="kinect" parent="tilt_link">
+  <xacro:shell name="shell" parent="base_linkz">
+    <origin xyz="0 0 ${hokuyo_z-0.13}" rpy="0 0 0"/>
+  </xacro:shell>
+  <kinect name="kinect" parent="neck_tilt_link">
     <origin xyz="${kinect_x} ${kinect_y} ${kinect_z}" rpy="${kinect_roll} ${kinect_pitch} ${kinect_yaw}"/>
   </kinect>
-  <gazebo>
-    <plugin name="ros_control" filename="libhwi_switch_gazebo_ros_control.so">
-      <robotNamespace>pan_tilt_controller</robotNamespace>
-      <filterJointsParam>joint_names</filterJointsParam>
-    </plugin>
-  </gazebo>
 </robot>

Commit message: update tuw robotino model

File: robotino_bringup/robots/tuw-robotino2/urdf/properties.urdf.xacro (robot description, xacro)
@@ -21,18 +21,18 @@
   <property name="hokuyo_pitch" value="0.0"/>
   <property name="hokuyo_yaw" value="-0.015"/>
-  <!-- pan_tilt mount positions | handeye calibration | relative to base_link -->
-  <property name="pan_tilt_x" value="0.258758"/>
-  <property name="pan_tilt_y" value="-0.0038856"/>
-  <property name="pan_tilt_z" value="0.655646"/>
-  <property name="pan_tilt_roll" value="0.0233953"/>
-  <property name="pan_tilt_pitch" value="-0.0360962"/>
-  <property name="pan_tilt_yaw" value="0.00901179"/>
-  <!-- kinect mount positions | handeye calibration | relative to pan_tilt_link -->
-  <property name="kinect_x" value="-0.0300317"/>
-  <property name="kinect_y" value="0.0603655"/>
-  <property name="kinect_z" value="-0.0649396"/>
-  <property name="kinect_roll" value="1.582"/>
-  <property name="kinect_pitch" value="3.11972"/>
-  <property name="kinect_yaw" value="3.12919"/>
+  <!-- base_neck_link mount positions | camera base calibration | relative to base_link -->
+  <property name="shell_x" value="0.0"/>
+  <property name="shell_y" value="0.0"/>
+  <property name="shell_z" value="0.0"/>
+  <property name="shell_roll" value="0.0"/>
+  <property name="shell_pitch" value="0.0"/>
+  <property name="shell_yaw" value="0.0"/>
+  <!-- kinect mount positions | camera base calibration | relative to neck_tilt_link -->
+  <property name="kinect_x" value="0.0"/>
+  <property name="kinect_y" value="0.0"/>
+  <property name="kinect_z" value="0.0"/>
+  <property name="kinect_roll" value="-1.57"/>
+  <property name="kinect_pitch" value="0"/>
+  <property name="kinect_yaw" value="0"/>
   <!-- arm mount positions | handeye calibration | relative to base_link -->
   <property name="arm_x" value="0.0"/>

File: robotino_bringup/robots/tuw-robotino2/urdf/robotino.urdf.xacro (robot description, xacro)
@@ -4,8 +4,7 @@
   <xacro:include filename="$(find robotino_bringup)/robots/tuw-robotino2/urdf/properties.urdf.xacro" />
   <xacro:include filename="$(find robotino_description)/urdf/base.urdf.xacro" />
-  <xacro:include filename="$(find robotino_description)/urdf/base_shell.urdf.xacro" />
+  <xacro:include filename="$(find robotino_description)/urdf/shell.urdf.xacro" />
   <xacro:include filename="$(find robotino_description)/urdf/hokuyo.urdf.xacro" />
   <xacro:include filename="$(find robotino_description)/urdf/kinect.urdf.xacro" />
-  <xacro:include filename="$(find robotino_description)/urdf/pan_tilt_tuw_axis.urdf.xacro" />
   <xacro:include filename="$(find robotino_description)/urdf/arm.urdf.xacro" />
   <xacro:include filename="$(find robotino_description)/urdf/kclhand_withCableCanal.urdf.xacro" />
@@ -17,6 +16,6 @@
     </plugin>
   </gazebo>
-  <xacro:shell name="base_shell" parent="base_link">
-    <origin xyz="0 0 ${hokuyo_z-0.13}" rpy="0 0 0"/>
+  <xacro:shell name="shell" parent="base_linkz">
+    <origin xyz="${shell_x} ${shell_y} ${shell_z}" rpy="${shell_roll} ${shell_pitch} ${shell_yaw}"/>
   </xacro:shell>
   <hokuyo name="hokuyo" parent="base_linkz">
@@ -41,15 +40,6 @@
     </plugin>
   </gazebo>
-  <pan_tilt_axis parent="base_linkz">
-    <origin xyz="${pan_tilt_x} ${pan_tilt_y} ${pan_tilt_z}" rpy="${pan_tilt_roll} ${pan_tilt_pitch} ${pan_tilt_yaw}"/>
-  </pan_tilt_axis>
-  <kinect name="kinect" parent="tilt_link">
+  <kinect name="kinect" parent="neck_tilt_link">
     <origin xyz="${kinect_x} ${kinect_y} ${kinect_z}" rpy="${kinect_roll} ${kinect_pitch} ${kinect_yaw}"/>
   </kinect>
-  <gazebo>
-    <plugin name="ros_control" filename="libhwi_switch_gazebo_ros_control.so">
-      <robotNamespace>pan_tilt_controller</robotNamespace>
-      <filterJointsParam>joint_names</filterJointsParam>
-    </plugin>
-  </gazebo>
 </robot>
