Commit message: update shell robot model

File: robotino_bringup/robots/idmind-robotino/urdf/properties.urdf.xacro (robot description, xacro)
@@ -6,7 +6,4 @@
   <property name="M_PI" value="3.14159"/>
   <property name="M_SCALE" value="0.01"/>
-  <property name="BASE_RADIUS" value="0.18"/>
-  <property name="BASE_HEIGHT" value="0.05"/>
-  <property name="BASE_MASS" value="20"/>
   <property name="HOKUYO_RADIUS" value="0.02"/>
   <property name="HOKUYO_LENGTH" value="0.07"/>
@@ -21,31 +18,10 @@
   <property name="hokuyo_pitch" value="0.0"/>
   <property name="hokuyo_yaw" value="-0.015"/>
-  <!-- pan_tilt mount positions | handeye calibration | relative to base_link -->
-  <property name="pan_tilt_x" value="0.258758"/>
-  <property name="pan_tilt_y" value="-0.0038856"/>
-  <property name="pan_tilt_z" value="0.655646"/>
-  <property name="pan_tilt_roll" value="0.0233953"/>
-  <property name="pan_tilt_pitch" value="-0.0360962"/>
-  <property name="pan_tilt_yaw" value="0.00901179"/>
   <!-- kinect mount positions | handeye calibration | relative to pan_tilt_link -->
-  <property name="kinect_x" value="-0.0300317"/>
-  <property name="kinect_y" value="0.0603655"/>
-  <property name="kinect_z" value="-0.0649396"/>
-  <property name="kinect_roll" value="1.582"/>
-  <property name="kinect_pitch" value="3.11972"/>
-  <property name="kinect_yaw" value="3.12919"/>
-  <!-- arm mount positions | handeye calibration | relative to base_link -->
-  <property name="arm_x" value="0.0"/>
-  <property name="arm_y" value="-0.01591"/>
-  <property name="arm_z" value="0.32"/>
-  <property name="arm_roll" value="0.0"/>
-  <property name="arm_pitch" value="0.0"/>
-  <property name="arm_yaw" value="-1"/>
-   <!-- arm calibration-->
-  <property name="arm_1_ref" value="0.0"/>
-  <property name="arm_2_ref" value="0.0"/>
-  <property name="arm_3_ref" value="0.0"/>
-  <property name="arm_4_ref" value="0.0"/>
-  <property name="arm_5_ref" value="0.0"/>
-  <property name="arm_6_ref" value="0.0"/>
+  <property name="kinect_x" value="0.0"/>
+  <property name="kinect_y" value="0.0"/>
+  <property name="kinect_z" value="0.0"/>
+  <property name="kinect_roll" value="-1.57"/>
+  <property name="kinect_pitch" value="0"/>
+  <property name="kinect_yaw" value="0"/>
 </robot>

File: robotino_bringup/robots/idmind-robotino/urdf/robotino.urdf.xacro (robot description, xacro)
@@ -6,4 +6,5 @@
   <xacro:include filename="$(find robotino_description)/urdf/shell.urdf.xacro" />
   <xacro:include filename="$(find robotino_description)/urdf/hokuyo.urdf.xacro" />
+  <xacro:include filename="$(find robotino_description)/urdf/kinect.urdf.xacro" />
   <xacro:base name="base"/>
   <gazebo>
@@ -19,3 +20,6 @@
     <origin xyz="${hokuyo_x} ${hokuyo_y} ${hokuyo_z}" rpy="${hokuyo_roll} ${hokuyo_pitch} ${hokuyo_yaw}"/>
   </hokuyo>
+  <kinect name="kinect" parent="neck_tilt_link">
+    <origin xyz="${kinect_x} ${kinect_y} ${kinect_z}" rpy="${kinect_roll} ${kinect_pitch} ${kinect_yaw}"/>
+  </kinect>
 </robot>

Commit message: update urdf to support calibration

File: robotino_bringup/robots/idmind-robotino/urdf/properties.urdf.xacro (robot description, xacro)
@@ -18,5 +18,5 @@
   <property name="hokuyo_pitch" value="0.0"/>
   <property name="hokuyo_yaw" value="-0.015"/>
-  <!-- kinect mount positions | handeye calibration | relative to pan_tilt_link -->
+  <!-- kinect mount positions | camera base calibration | relative to neck_tilt_link -->
   <property name="kinect_x" value="0.0"/>
   <property name="kinect_y" value="0.0"/>
@@ -25,3 +25,10 @@
   <property name="kinect_pitch" value="0"/>
   <property name="kinect_yaw" value="0"/>
+  <!-- base_neck_link mount positions | camera base calibration | relative to base_link -->
+  <property name="shell_x" value="0.0"/>
+  <property name="shell_y" value="0.0"/>
+  <property name="shell_z" value="0.0"/>
+  <property name="shell_roll" value="0.0"/>
+  <property name="shell_pitch" value="0.0"/>
+  <property name="shell_yaw" value="0.0"/>
 </robot>

File: robotino_bringup/robots/idmind-robotino/urdf/robotino.urdf.xacro (robot description, xacro)
@@ -15,5 +15,5 @@
   </gazebo>
   <xacro:shell name="shell" parent="base_linkz">
-    <origin xyz="0 0 0" rpy="0 0 0"/>
+    <origin xyz="${shell_x} ${shell_y} ${shell_z}" rpy="${shell_roll} ${shell_pitch} ${shell_yaw}"/>
   </xacro:shell>
   <hokuyo name="hokuyo" parent="base_linkz">
